Commit message: new plato urdf with united joint R direction

File: optimo_description/urdf/plato.urdf.xacro (robot description, xacro)
@@ -1,602 +1,325 @@
 <?xml version="1.0"?>
 <robot name="plato" xmlns:xacro="http://www.ros.org/wiki/xacro">
-<link name="base_link">
-</link>
-<joint name = "base_link_to_palm" type="fixed">
-    <origin xyz="0 0 0" rpy="0 0 0"/>
-    <parent link="base_link"/>
-    <child link="base"/>
+<link name="base_link"></link>
+<joint name="base_link_to_base" type="fixed">
+<parent link="base_link"/>
+<child link="base" />
+<origin rpy="0.0 0 0" xyz="0 0 0"/>
 </joint>
 <link name="base">
 <visual>
-<origin xyz="3.4694469519536141888e-18 0 -0.016000000000000000333" rpy="9.0205620750793734716e-17 2.7644301800592740999e-17 -6.8593115106840873102e-16" />
+<origin xyz="0 0 0" rpy="0 -0 0" />
 <geometry>
-<mesh filename="package://optimo_description/meshes/plato/wrist.stl"/>
+<mesh filename="package://optimo_description/meshes/plato/base_visual.stl"/>
 </geometry>
-<material name="wrist_material">
-<color rgba="0.91764705882352937127 0.91764705882352937127 0.91764705882352937127 1.0"/>
+<material name="base_material">
+<color rgba="0.89999999999999991118 0.89999999999999991118 0.89999999999999991118 1.0"/>
 </material>
 </visual>
 <collision>
-<origin xyz="3.4694469519536141888e-18 0 -0.016000000000000000333" rpy="9.0205620750793734716e-17 2.7644301800592740999e-17 -6.8593115106840873102e-16" />
+<origin xyz="0 0 0" rpy="0 -0 0" />
 <geometry>
-<mesh filename="package://optimo_description/meshes/plato/wrist.stl"/>
-</geometry>
-</collision>
-<visual>
-<origin xyz="3.4694469519536141888e-18 0 -0.016000000000000000333" rpy="9.0205620750793734716e-17 2.7644301800592740999e-17 -6.8593115106840873102e-16" />
-<geometry>
-<mesh filename="package://optimo_description/meshes/plato/palm.stl"/>
-</geometry>
-<material name="palm_material">
-<color rgba="0.90196078431372550543 0.90196078431372550543 0.90196078431372550543 1.0"/>
-</material>
-</visual>
-<collision>
-<origin xyz="3.4694469519536141888e-18 0 -0.016000000000000000333" rpy="9.0205620750793734716e-17 2.7644301800592740999e-17 -6.8593115106840873102e-16" />
-<geometry>
-<mesh filename="package://optimo_description/meshes/plato/palm.stl"/>
-</geometry>
-</collision>
-<visual>
-<origin xyz="-1.3788241001829422089e-16 -2.7755575615628913511e-17 -0.016000000000000028089" rpy="1.6653345369377128704e-16 -6.1550287343936601898e-16 -4.3977943457854727703e-15" />
-<geometry>
-<mesh filename="package://optimo_description/meshes/plato/thumb_roll.stl"/>
-</geometry>
-<material name="thumb_roll_material">
-<color rgba="0.61568627450980395466 0.81176470588235294379 0.92941176470588238168 1.0"/>
-</material>
-</visual>
-<collision>
-<origin xyz="-1.3788241001829422089e-16 -2.7755575615628913511e-17 -0.016000000000000028089" rpy="1.6653345369377128704e-16 -6.1550287343936601898e-16 -4.3977943457854727703e-15" />
-<geometry>
-<mesh filename="package://optimo_description/meshes/plato/thumb_roll.stl"/>
+<mesh filename="package://optimo_description/meshes/plato/base_collision.stl"/>
 </geometry>
 </collision>
 <inertial>
-<origin xyz="-0.0007588504329184387687 0.045493179467456477949 -0.0068276731996390008922" rpy="0 0 0"/>
-<mass value="0.1728032154969740275" />
-<inertia ixx="0.00022114103876778821718" ixy="2.1184002504335696667e-06"  ixz="-2.4145885068302762577e-06" iyy="0.000124447216717875575" iyz="-5.2375390643356322257e-06" izz="0.00030593848378724351235" />
+<origin xyz="0.045493179467456464071 0.00075885043291842098779 -0.00682767319963901477" rpy="0 0 0"/>
+<mass value="0.17280321549697399974" />
+<inertia ixx="0.000124447216717875575" ixy="-2.1184002504334913161e-06"  ixz="-5.2375390643355526047e-06" iyy="0.00022114103876778816297" iyz="2.4145885068302643992e-06" izz="0.00030593848378724351235" />
 </inertial>
 </link>
-<link name="mcp_yaw">
-<visual>
-<origin xyz="3.4694469519536141888e-18 1.3877787807814456755e-17 -0.0098999999999999990785" rpy="3.141592653589793116 -1.8219420127185215539e-33 -1.0018951972865276753e-32" />
-<geometry>
-<mesh filename="package://optimo_description/meshes/plato/motor.stl"/>
-</geometry>
-<material name="motor_material">
-<color rgba="0.90196078431372550543 0.90196078431372550543 0.90196078431372550543 1.0"/>
-</material>
-</visual>
-<collision>
-<origin xyz="3.4694469519536141888e-18 1.3877787807814456755e-17 -0.0098999999999999990785" rpy="3.141592653589793116 -1.8219420127185215539e-33 -1.0018951972865276753e-32" />
-<geometry>
-<mesh filename="package://optimo_description/meshes/plato/motor.stl"/>
-</geometry>
-</collision>
-<visual>
-<origin xyz="-0.014900000000000123215 0.028149999999999508749 -0.0099000000000003078593" rpy="-3.9443456428854888764e-30 1.5707963267948943376 0" />
-<geometry>
-<mesh filename="package://optimo_description/meshes/plato/motor.stl"/>
-</geometry>
-<material name="motor_material">
-<color rgba="0.90196078431372550543 0.90196078431372550543 0.90196078431372550543 1.0"/>
-</material>
-</visual>
-<collision>
-<origin xyz="-0.014900000000000123215 0.028149999999999508749 -0.0099000000000003078593" rpy="-3.9443456428854888764e-30 1.5707963267948943376 0" />
-<geometry>
-<mesh filename="package://optimo_description/meshes/plato/motor.stl"/>
-</geometry>
-</collision>
-<visual>
-<origin xyz="-6.9388939039072283776e-18 1.3877787807814456755e-17 -0.019799999999999998157" rpy="-3.1415926535897922278 -1.6363862086693127369e-16 -3.141592653589793116" />
-<geometry>
-<mesh filename="package://optimo_description/meshes/plato/mcp_yaw_connect.stl"/>
-</geometry>
-<material name="mcp_yaw_connect_material">
-<color rgba="0.90196078431372550543 0.90196078431372550543 0.90196078431372550543 1.0"/>
-</material>
-</visual>
-<collision>
-<origin xyz="-6.9388939039072283776e-18 1.3877787807814456755e-17 -0.019799999999999998157" rpy="-3.1415926535897922278 -1.6363862086693127369e-16 -3.141592653589793116" />
-<geometry>
-<mesh filename="package://optimo_description/meshes/plato/mcp_yaw_connect.stl"/>
-</geometry>
-</collision>
-<inertial>
-<origin xyz="-0.0079504685553140486826 0.013983661603933850506 -0.010286902688940493741" rpy="0 0 0"/>
-<mass value="0.12656081824380860379" />
-<inertia ixx="3.5117165939881067604e-05" ixy="1.3052140141476160172e-05"  ixz="-1.995751982634699314e-07" iyy="1.7537495218030352186e-05" iyz="-4.9180486622802420018e-07" izz="4.2451494821236167819e-05" />
-</inertial>
-</link>
-<link name="mcp_pitch">
-<visual>
-<origin xyz="0 -2.6020852139652106416e-18 -0.016399999999999633621" rpy="1.0325074129013607149e-14 -4.2751324234174125628e-15 -1.570796326794896558" />
-<geometry>
-<mesh filename="package://optimo_description/meshes/plato/motor.stl"/>
-</geometry>
-<material name="motor_material">
-<color rgba="0.90196078431372550543 0.90196078431372550543 0.90196078431372550543 1.0"/>
-</material>
-</visual>
-<collision>
-<origin xyz="0 -2.6020852139652106416e-18 -0.016399999999999633621" rpy="1.0325074129013607149e-14 -4.2751324234174125628e-15 -1.570796326794896558" />
-<geometry>
-<mesh filename="package://optimo_description/meshes/plato/motor.stl"/>
-</geometry>
-</collision>
-<visual>
-<origin xyz="0.019999999999999906741 -8.6736173798840354721e-19 -0.0049999999999999940326" rpy="1.570796326794896558 -1.570796326794896558 0" />
-<geometry>
-<mesh filename="package://optimo_description/meshes/plato/phlange.stl"/>
-</geometry>
-<material name="phlange_material">
-<color rgba="0.90196078431372550543 0.90196078431372550543 0.90196078431372550543 1.0"/>
-</material>
-</visual>
-<collision>
-<origin xyz="0.019999999999999906741 -8.6736173798840354721e-19 -0.0049999999999999940326" rpy="1.570796326794896558 -1.570796326794896558 0" />
-<geometry>
-<mesh filename="package://optimo_description/meshes/plato/phlange.stl"/>
-</geometry>
-</collision>
-<visual>
-<origin xyz="0 -8.6736173798840354721e-19 0" rpy="1.570796326794896558 1.570796326794896558 0" />
-<geometry>
-<mesh filename="package://optimo_description/meshes/plato/mcp_pitch_connect.stl"/>
-</geometry>
-<material name="mcp_pitch_connect_material">
-<color rgba="0.90196078431372550543 0.90196078431372550543 0.90196078431372550543 1.0"/>
-</material>
-</visual>
-<collision>
-<origin xyz="0 -8.6736173798840354721e-19 0" rpy="1.570796326794896558 1.570796326794896558 0" />
-<geometry>
-<mesh filename="package://optimo_description/meshes/plato/mcp_pitch_connect.stl"/>
-</geometry>
-</collision>
-<inertial>
-<origin xyz="0.0020817714488827365922 3.9659157887021715613e-10 -0.015795112278832897784" rpy="0 0 0"/>
-<mass value="0.069114549940711825227" />
-<inertia ixx="5.8883565545031231453e-06" ixy="-9.2074790703350845863e-09"  ixz="-1.1640174651109904652e-06" iyy="9.6829622072777303483e-06" iyz="-9.4322549796764935789e-14" izz="9.2871592762527697414e-06" />
-</inertial>
-</link>
-<link name="pip">
-<visual>
-<origin xyz="0 0 -0.0022999999999999999611" rpy="1.570796326794896558 1.570796326794896558 0" />
-<geometry>
-<mesh filename="package://optimo_description/meshes/plato/pip_connect.stl"/>
-</geometry>
-<material name="pip_connect_material">
-<color rgba="0.90196078431372550543 0.90196078431372550543 0.90196078431372550543 1.0"/>
-</material>
-</visual>
-<collision>
-<origin xyz="0 0 -0.0022999999999999999611" rpy="1.570796326794896558 1.570796326794896558 0" />
-<geometry>
-<mesh filename="package://optimo_description/meshes/plato/pip_connect.stl"/>
-</geometry>
-</collision>
-<visual>
-<origin xyz="0.029600000000000431521 -2.6801477703841669609e-16 -0.0023000000000002185363" rpy="1.57079632679489678 -1.570796326794896558 0" />
-<geometry>
-<mesh filename="package://optimo_description/meshes/plato/fingertip.stl"/>
-</geometry>
-<material name="fingertip_material">
-<color rgba="0.90196078431372550543 0.90196078431372550543 0.90196078431372550543 1.0"/>
-</material>
-</visual>
-<collision>
-<origin xyz="0.029600000000000431521 -2.6801477703841669609e-16 -0.0023000000000002185363" rpy="1.57079632679489678 -1.570796326794896558 0" />
-<geometry>
-<mesh filename="package://optimo_description/meshes/plato/fingertip.stl"/>
-</geometry>
-</collision>
-<visual>
-<origin xyz="0.024000241812767941774 -0.030174068124402677465 -0.072096228994413036339" rpy="-3.8455702303801434139e-17 1.570796326794896558 0" />
-<geometry>
-<mesh filename="package://optimo_description/meshes/plato/ft_sensor.stl"/>
-</geometry>
-<material name="ft_sensor_material">
-<color rgba="0.90196078431372550543 0.90196078431372550543 0.90196078431372550543 1.0"/>
-</material>
-</visual>
-<collision>
-<origin xyz="0.024000241812767941774 -0.030174068124402677465 -0.072096228994413036339" rpy="-3.8455702303801434139e-17 1.570796326794896558 0" />
-<geometry>
-<mesh filename="package://optimo_description/meshes/plato/ft_sensor.stl"/>
-</geometry>
-</collision>
-<inertial>
-<origin xyz="0.020839063326584635755 -0.00066661768468522094536 -0.0023008505382950436395" rpy="0 0 0"/>
-<mass value="0.0080671501064400203546" />
-<inertia ixx="2.1185571765449787875e-07" ixy="3.6426243959718411587e-08"  ixz="-1.3233834118458726401e-10" iyy="1.2852102149793485867e-06" iyz="-3.108419012789066537e-11" izz="1.3237276294093304559e-06" />
-</inertial>
-</link>
-<joint name="f2_pip" type="revolute">
-<origin xyz="0.047999999999998710365 0 -0.0027000000000000877465" rpy="8.6736173795253712333e-17 -1.1333526709686569771e-16 9.7660980066365267833e-26" />
-<parent link="mcp_pitch" />
-<child link="pip" />
-<axis xyz="0 0 1"/>
-<limit effort="1" velocity="20" lower="-2.0943951023931952626" upper="2.0943951023931952626"/>
-<joint_properties friction="0.0"/>
-</joint>
-<joint name="f2_mcp_pitch" type="revolute">
-<origin xyz="-0.0050000000000001397493 0.028149999999999536504 -0.0099000000000003061246" rpy="-1.57079632679489678 -2.7077043760675503572e-14 1.5707963267948823471" />
-<parent link="mcp_yaw" />
-<child link="mcp_pitch" />
-<axis xyz="0 0 1"/>
-<limit effort="1" velocity="20" lower="-1.570796326794896558" upper="1.570796326794896558"/>
-<joint_properties friction="0.0"/>
-</joint>
-<joint name="f2_mcp_yaw" type="revolute">
-<origin xyz="0.029999999999999912154 0.10000000000000003331 0.0050000000000003270995" rpy="5.8606965434539231359e-16 1.9351011260415344561e-16 -7.1054273576010255245e-15" />
-<parent link="base" />
-<child link="mcp_yaw" />
-<axis xyz="0 0 1"/>
-<limit effort="1" velocity="20" lower="-0.52359877559829881566" upper="0.26179938779914940783"/>
-<joint_properties friction="0.0"/>
-</joint>
-<link name="mcp_yaw_2">
-<visual>
-<origin xyz="-3.4694469519536141888e-18 0 -0.0099000000000000008132" rpy="3.141592653589793116 -1.1374534524689678013e-32 1.389378947316507434e-31" />
-<geometry>
-<mesh filename="package://optimo_description/meshes/plato/motor.stl"/>
-</geometry>
-<material name="motor_material">
-<color rgba="0.90196078431372550543 0.90196078431372550543 0.90196078431372550543 1.0"/>
-</material>
-</visual>
-<collision>
-<origin xyz="-3.4694469519536141888e-18 0 -0.0099000000000000008132" rpy="3.141592653589793116 -1.1374534524689678013e-32 1.389378947316507434e-31" />
-<geometry>
-<mesh filename="package://optimo_description/meshes/plato/motor.stl"/>
-</geometry>
-</collision>
-<visual>
-<origin xyz="-0.014899999999999899436 0.028149999999999578137 -0.0099000000000004015344" rpy="2.6040940641035082432e-31 1.570796326794896336 0" />
-<geometry>
-<mesh filename="package://optimo_description/meshes/plato/motor.stl"/>
-</geometry>
-<material name="motor_material">
-<color rgba="0.90196078431372550543 0.90196078431372550543 0.90196078431372550543 1.0"/>
-</material>
-</visual>
-<collision>
-<origin xyz="-0.014899999999999899436 0.028149999999999578137 -0.0099000000000004015344" rpy="2.6040940641035082432e-31 1.570796326794896336 0" />
-<geometry>
-<mesh filename="package://optimo_description/meshes/plato/motor.stl"/>
-</geometry>
-</collision>
-<visual>
-<origin xyz="-3.4694469519536141888e-18 0 -0.019800000000000001626" rpy="-3.1415926535897926719 3.1762611116722443688e-16 3.141592653589793116" />
-<geometry>
-<mesh filename="package://optimo_description/meshes/plato/mcp_yaw_connect.stl"/>
-</geometry>
-<material name="mcp_yaw_connect_material">
-<color rgba="0.90196078431372550543 0.90196078431372550543 0.90196078431372550543 1.0"/>
-</material>
-</visual>
-<collision>
-<origin xyz="-3.4694469519536141888e-18 0 -0.019800000000000001626" rpy="-3.1415926535897926719 3.1762611116722443688e-16 3.141592653589793116" />
-<geometry>
-<mesh filename="package://optimo_description/meshes/plato/mcp_yaw_connect.stl"/>
-</geometry>
-</collision>
-<inertial>
-<origin xyz="-0.0079504685553139359255 0.013983661603933878262 -0.010286902688940540579" rpy="0 0 0"/>
-<mass value="0.12656081824380860379" />
-<inertia ixx="3.5117165939881223459e-05" ixy="1.3052140141475956884e-05"  ixz="-1.9957519826351961518e-07" iyy="1.7537495218030094688e-05" iyz="-4.9180486622795326117e-07" izz="4.2451494821235971307e-05" />
-</inertial>
-</link>
-<link name="mcp_pitch_2">
-<visual>
-<origin xyz="0 0 -6.9388939039072283776e-18" rpy="1.570796326794896558 1.570796326794896558 0" />
-<geometry>
-<mesh filename="package://optimo_description/meshes/plato/mcp_pitch_connect.stl"/>
-</geometry>
-<material name="mcp_pitch_connect_material">
-<color rgba="0.90196078431372550543 0.90196078431372550543 0.90196078431372550543 1.0"/>
-</material>
-</visual>
-<collision>
-<origin xyz="0 0 -6.9388939039072283776e-18" rpy="1.570796326794896558 1.570796326794896558 0" />
-<geometry>
-<mesh filename="package://optimo_description/meshes/plato/mcp_pitch_connect.stl"/>
-</geometry>
-</collision>
-<visual>
-<origin xyz="0 1.7347234759768070944e-18 -0.016399999999999980566" rpy="-5.991802860914466036e-16 1.7451588453829230951e-16 -1.570796326794896558" />
-<geometry>
-<mesh filename="package://optimo_description/meshes/plato/motor.stl"/>
-</geometry>
-<material name="motor_material">
-<color rgba="0.90196078431372550543 0.90196078431372550543 0.90196078431372550543 1.0"/>
-</material>
-</visual>
-<collision>
-<origin xyz="0 1.7347234759768070944e-18 -0.016399999999999980566" rpy="-5.991802860914466036e-16 1.7451588453829230951e-16 -1.570796326794896558" />
-<geometry>
-<mesh filename="package://optimo_description/meshes/plato/motor.stl"/>
-</geometry>
-</collision>
-<visual>
-<origin xyz="0.020000000000000017764 2.6020852139652106416e-18 -0.0050000000000000009714" rpy="1.570796326794896558 -1.570796326794896558 0" />
-<geometry>
-<mesh filename="package://optimo_description/meshes/plato/phlange.stl"/>
-</geometry>
-<material name="phlange_material">
-<color rgba="0.90196078431372550543 0.90196078431372550543 0.90196078431372550543 1.0"/>
-</material>
-</visual>
-<collision>
-<origin xyz="0.020000000000000017764 2.6020852139652106416e-18 -0.0050000000000000009714" rpy="1.570796326794896558 -1.570796326794896558 0" />
-<geometry>
-<mesh filename="package://optimo_description/meshes/plato/phlange.stl"/>
-</geometry>
-</collision>
-<inertial>
-<origin xyz="0.0020817714488827595773 3.9659158286529116865e-10 -0.015795112278833196157" rpy="0 0 0"/>
-<mass value="0.069114549940711839104" />
-<inertia ixx="5.8883565545031163691e-06" ixy="-9.2074790702916195538e-09"  ixz="-1.1640174651111035441e-06" iyy="9.6829622072775829646e-06" iyz="-9.4322528370318213712e-14" izz="9.2871592762525291841e-06" />
-</inertial>
-</link>
-<link name="pip_2">
-<visual>
-<origin xyz="0.02400024181276727564 -0.030174068124402667057 -0.072096228994410066493" rpy="-3.8455702303801045871e-17 1.570796326794896558 0" />
-<geometry>
-<mesh filename="package://optimo_description/meshes/plato/ft_sensor.stl"/>
-</geometry>
-<material name="ft_sensor_material">
-<color rgba="0.90196078431372550543 0.90196078431372550543 0.90196078431372550543 1.0"/>
-</material>
-</visual>
-<collision>
-<origin xyz="0.02400024181276727564 -0.030174068124402667057 -0.072096228994410066493" rpy="-3.8455702303801045871e-17 1.570796326794896558 0" />
-<geometry>
-<mesh filename="package://optimo_description/meshes/plato/ft_sensor.stl"/>
-</geometry>
-</collision>
-<visual>
-<origin xyz="2.7755575615628913511e-17 0 -0.0023000000000000034306" rpy="1.570796326794896558 1.570796326794896558 0" />
-<geometry>
-<mesh filename="package://optimo_description/meshes/plato/pip_connect.stl"/>
-</geometry>
-<material name="pip_connect_material">
-<color rgba="0.90196078431372550543 0.90196078431372550543 0.90196078431372550543 1.0"/>
-</material>
-</visual>
-<collision>
-<origin xyz="2.7755575615628913511e-17 0 -0.0023000000000000034306" rpy="1.570796326794896558 1.570796326794896558 0" />
-<geometry>
-<mesh filename="package://optimo_description/meshes/plato/pip_connect.stl"/>
-</geometry>
-</collision>
-<visual>
-<origin xyz="0.029600000000000403766 -2.6714741530042829254e-16 -0.0023000000000000624112" rpy="1.57079632679489678 -1.5707963267948885644 0" />
-<geometry>
-<mesh filename="package://optimo_description/meshes/plato/fingertip.stl"/>
-</geometry>
-<material name="fingertip_material">
-<color rgba="0.90196078431372550543 0.90196078431372550543 0.90196078431372550543 1.0"/>
-</material>
-</visual>
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