Commit message: add geomtry to base link

File: optimo_description/urdf/optimo_arm.xacro (robot description, xacro)
@@ -39,5 +39,14 @@
         </inertial>
     </link>
-    <link name="link1"/>
+    <link name="link1">
+        <visual>
+            <geometry>
+                <sphere radius="0.01"/>
+            </geometry>
+            <material name="LightGrey">
+                <color rgba="0.999 0.999 0.999 1.0"/>
+            </material>
+        </visual>
+    </link>
     <link name="link1_passive">
         <visual>
