Commit message: urdf+xacro folder organized

File: optimo_description/urdf/optimo.urdf.xacro (robot description, xacro)
@@ -1,5 +1,6 @@
 <?xml version="1.0"?>
 <robot name="optimo" xmlns:xacro="http://www.ros.org/wiki/xacro">
-    <xacro:include filename="optimo_arm.xacro"/>
-    <xacro:include filename="optimo.gazebo.xacro" />
+    <xacro:include filename="optimo_property/optimo_arm.xacro"/>
+    <xacro:include filename="optimo_property/optimo.gazebo.xacro" />
+    <xacro:include filename="optimo_property/optimo.control.xacro" />
 </robot>

File: optimo_description/urdf/optimo_property/optimo.control.xacro (robot description, xacro)
@@ -1,18 +1,3 @@
-<?xml version="1.0"?>
-<robot xmlns:xacro="http://www.ros.org/wiki/xacro">
-    <!-- Joint State Publisher -->
-    <gazebo>
-        <plugin name="gazebo_ros_joint_state_publisher" filename="libgazebo_ros_joint_state_publisher.so">
-            <update_rate>1000</update_rate>
-            <joint_name>joint1</joint_name>
-            <joint_name>joint2</joint_name>
-            <joint_name>joint3</joint_name>
-            <joint_name>joint4</joint_name>
-            <joint_name>joint5</joint_name>
-            <joint_name>joint6</joint_name>
-            <joint_name>joint7</joint_name>
-        </plugin>
-    </gazebo>
-    <gazebo>
+<gazebo>
         <plugin filename="libgazebo_ros2_control.so" name="gazebo_ros2_control">
             <parameters>$(find plato_gazebo)/config/optimo_controller.yaml</parameters>
@@ -27,5 +12,7 @@
             <command_interface name="position">
             </command_interface>
-            <state_interface name="position" />
+            <state_interface name="position">
+                <param name="initial_value">0.0</param>
+            </state_interface>
             <state_interface name="velocity" />
             <state_interface name="effort" />
@@ -36,5 +23,7 @@
                 <!-- <param name="max">1.7628</param> -->
             </command_interface>
-            <state_interface name="position" />
+            <state_interface name="position">
+                <param name="initial_value">3.141592</param>
+            </state_interface>
             <state_interface name="velocity" />
             <state_interface name="effort" />
@@ -45,5 +34,7 @@
                 <!-- <param name="max">2.8973</param> -->
             </command_interface>
-            <state_interface name="position" />
+            <state_interface name="position">
+                <param name="initial_value">0.0</param>
+            </state_interface>
             <state_interface name="velocity" />
             <state_interface name="effort" />
@@ -54,5 +45,7 @@
                 <!-- <param name="max">-0.0698</param> -->
             </command_interface>
-            <state_interface name="position" />
+            <state_interface name="position">
+                <param name="initial_value">0.0</param>
+            </state_interface>
             <state_interface name="velocity" />
             <state_interface name="effort" />
@@ -63,5 +56,7 @@
                 <!-- <param name="max">2.8973</param> -->
             </command_interface>
-            <state_interface name="position" />
+            <state_interface name="position">
+                <param name="initial_value">0.0</param>
+            </state_interface>
             <state_interface name="velocity" />
             <state_interface name="effort" />
@@ -72,5 +67,7 @@
                 <!-- <param name="max">3.7525</param> -->
             </command_interface>
-            <state_interface name="position" />
+            <state_interface name="position">
+                <param name="initial_value">0.0</param>
+            </state_interface>
             <state_interface name="velocity" />
             <state_interface name="effort" />
@@ -81,8 +78,9 @@
                 <!-- <param name="max">3.7525</param> -->
             </command_interface>
-            <state_interface name="position" />
+            <state_interface name="position">
+                <param name="initial_value">0.0</param>
+            </state_interface>
             <state_interface name="velocity" />
             <state_interface name="effort" />
         </joint>
     </ros2_control>
-</robot>

File: optimo_description/urdf/optimo_property/optimo_arm.xacro (robot description, xacro)
@@ -22,13 +22,13 @@
         <visual>
             <geometry>
-                <mesh filename="$(find optimo_description)/meshes/link0.stl"/>
-            </geometry>
-            <material name="LightGrey">
-                <color rgba="0.999 0.999 0.999 1.0"/>
-            </material>
-        </visual>
-        <collision>
-            <geometry>
-                <mesh filename="$(find optimo_description)/meshes/col0.stl"/>
+                <mesh filename="file://$(find optimo_description)/meshes/link0.stl"/>
+            </geometry>
+            <material name="LightGrey">
+                <color rgba="0.999 0.999 0.999 1.0"/>
+            </material>
+        </visual>
+        <collision>
+            <geometry>
+                <mesh filename="file://$(find optimo_description)/meshes/col0.stl"/>
             </geometry>
         </collision>
@@ -52,13 +52,13 @@
         <visual>
             <geometry>
-                <mesh filename="$(find optimo_description)/meshes/link1.stl"/>
-            </geometry>
-            <material name="LightGrey">
-                <color rgba="0.999 0.999 0.999 1.0"/>
-            </material>
-        </visual>
-        <collision>
-            <geometry>
-                <mesh filename="$(find optimo_description)/meshes/col1.stl"/>
+                <mesh filename="file://$(find optimo_description)/meshes/link1.stl"/>
+            </geometry>
+            <material name="LightGrey">
+                <color rgba="0.999 0.999 0.999 1.0"/>
+            </material>
+        </visual>
+        <collision>
+            <geometry>
+                <mesh filename="file://$(find optimo_description)/meshes/col1.stl"/>
             </geometry>
         </collision>
@@ -73,13 +73,13 @@
         <visual>
             <geometry>
-                <mesh filename="$(find optimo_description)/meshes/link2.stl"/>
-            </geometry>
-            <material name="LightGrey">
-                <color rgba="0.999 0.999 0.999 1.0"/>
-            </material>
-        </visual>
-        <collision>
-            <geometry>
-                <mesh filename="$(find optimo_description)/meshes/col2.stl"/>
+                <mesh filename="file://$(find optimo_description)/meshes/link2.stl"/>
+            </geometry>
+            <material name="LightGrey">
+                <color rgba="0.999 0.999 0.999 1.0"/>
+            </material>
+        </visual>
+        <collision>
+            <geometry>
+                <mesh filename="file://$(find optimo_description)/meshes/col2.stl"/>
             </geometry>
         </collision>
@@ -94,13 +94,13 @@
         <visual>
             <geometry>
-                <mesh filename="$(find optimo_description)/meshes/link3.stl"/>
-            </geometry>
-            <material name="LightGrey">
-                <color rgba="0.999 0.999 0.999 1.0"/>
-            </material>
-        </visual>
-        <collision>
-            <geometry>
-                <mesh filename="$(find optimo_description)/meshes/col3.stl"/>
+                <mesh filename="file://$(find optimo_description)/meshes/link3.stl"/>
+            </geometry>
+            <material name="LightGrey">
+                <color rgba="0.999 0.999 0.999 1.0"/>
+            </material>
+        </visual>
+        <collision>
+            <geometry>
+                <mesh filename="file://$(find optimo_description)/meshes/col3.stl"/>
             </geometry>
         </collision>
@@ -115,13 +115,13 @@
         <visual>
             <geometry>
-                <mesh filename="$(find optimo_description)/meshes/link4.stl"/>
-            </geometry>
-            <material name="LightGrey">
-                <color rgba="0.999 0.999 0.999 1.0"/>
-            </material>
-        </visual>
-        <collision>
-            <geometry>
-                <mesh filename="$(find optimo_description)/meshes/col4.stl"/>
+                <mesh filename="file://$(find optimo_description)/meshes/link4.stl"/>
+            </geometry>
+            <material name="LightGrey">
+                <color rgba="0.999 0.999 0.999 1.0"/>
+            </material>
+        </visual>
+        <collision>
+            <geometry>
+                <mesh filename="file://$(find optimo_description)/meshes/col4.stl"/>
             </geometry>
         </collision>
@@ -136,13 +136,13 @@
         <visual>
             <geometry>
-                <mesh filename="$(find optimo_description)/meshes/link5.stl"/>
-            </geometry>
-            <material name="LightGrey">
-                <color rgba="0.999 0.999 0.999 1.0"/>
-            </material>
-        </visual>
-        <collision>
-            <geometry>
-                <mesh filename="$(find optimo_description)/meshes/col5.stl"/>
+                <mesh filename="file://$(find optimo_description)/meshes/link5.stl"/>
+            </geometry>
+            <material name="LightGrey">
+                <color rgba="0.999 0.999 0.999 1.0"/>
+            </material>
+        </visual>
+        <collision>
+            <geometry>
+                <mesh filename="file://$(find optimo_description)/meshes/col5.stl"/>
             </geometry>
         </collision>
@@ -157,13 +157,13 @@
         <visual>
             <geometry>
-                <mesh filename="$(find optimo_description)/meshes/link6.stl"/>
-            </geometry>
-            <material name="LightGrey">
-                <color rgba="0.999 0.999 0.999 1.0"/>
-            </material>
-        </visual>
-        <collision>
-            <geometry>
-                <mesh filename="$(find optimo_description)/meshes/col6.stl"/>
+                <mesh filename="file://$(find optimo_description)/meshes/link6.stl"/>
+            </geometry>
+            <material name="LightGrey">
+                <color rgba="0.999 0.999 0.999 1.0"/>
+            </material>
+        </visual>
+        <collision>
+            <geometry>
+                <mesh filename="file://$(find optimo_description)/meshes/col6.stl"/>
             </geometry>
         </collision>
@@ -178,13 +178,13 @@
         <visual>
             <geometry>
-                <mesh filename="$(find optimo_description)/meshes/link7.stl"/>
-            </geometry>
-            <material name="LightGrey">
-                <color rgba="0.999 0.999 0.999 1.0"/>
-            </material>
-        </visual>
-        <collision>
-            <geometry>
-                <mesh filename="$(find optimo_description)/meshes/col7.stl"/>
+                <mesh filename="file://$(find optimo_description)/meshes/link7.stl"/>
+            </geometry>
+            <material name="LightGrey">
+                <color rgba="0.999 0.999 0.999 1.0"/>
+            </material>
+        </visual>
+        <collision>
+            <geometry>
+                <mesh filename="file://$(find optimo_description)/meshes/col7.stl"/>
             </geometry>
         </collision>
@@ -221,6 +221,5 @@
         <child link="link1"/>
         <axis xyz="0 0 1"/>
-        <!-- <limit lower="${DtR*-164}" upper="${DtR*167}" effort="79" velocity="10"/> -->
-        <limit lower="-2.8624" upper="2.9147" effort="79" velocity="10"/>
+        <limit lower="${DtR*-164}" upper="${DtR*167}" effort="79" velocity="10"/>
     </joint>
     <joint name="joint1_passive" type="fixed">
@@ -235,5 +234,4 @@
         <axis xyz="0 0 1"/>
         <limit lower="${DtR*60}" upper="${DtR*250}" effort="95" velocity="10"/>
-        <!-- <limit lower="0" upper="${DtR*250}" effort="95" velocity="10"/> -->
     </joint>
     <joint name="joint2_passive" type="fixed">

File: optimo_description/urdf/plato.urdf.xacro (robot description, xacro)
@@ -11,5 +11,5 @@
 <origin xyz="0 0 0" rpy="0 -0 0" />
 <geometry>
-<mesh filename="package://optimo_description/meshes/plato/base_visual.stl"/>
+<mesh filename="file://$(find optimo_description)/meshes/plato/base_visual.stl"/>
 </geometry>
 <material name="base_material">
@@ -20,5 +20,5 @@
 <origin xyz="0 0 0" rpy="0 -0 0" />
 <geometry>
-<mesh filename="package://optimo_description/meshes/plato/base_collision.stl"/>
+<mesh filename="file://$(find optimo_description)/meshes/plato/base_collision.stl"/>
 </geometry>
 </collision>
@@ -34,5 +34,5 @@
     <origin xyz="0 0 0" rpy="0 -0 0" />
     <geometry>
-    <mesh filename="package://optimo_description/meshes/plato/proxbracket_visual.stl"/>
+    <mesh filename="file://$(find optimo_description)/meshes/plato/proxbracket_visual.stl"/>
     </geometry>
     <material name="proxbracket_material">
@@ -43,5 +43,5 @@
     <origin xyz="0 0 0" rpy="0 -0 0" />
     <geometry>
-    <mesh filename="package://optimo_description/meshes/plato/proxbracket_collision.stl"/>
+    <mesh filename="file://$(find optimo_description)/meshes/plato/proxbracket_collision.stl"/>
     </geometry>
     </collision>
@@ -56,5 +56,5 @@
     <origin xyz="0 0 0" rpy="0 -0 0" />
     <geometry>
-    <mesh filename="package://optimo_description/meshes/plato/prox_visual.stl"/>
+    <mesh filename="file://$(find optimo_description)/meshes/plato/prox_visual.stl"/>
     </geometry>
     <material name="prox_material">
@@ -65,5 +65,5 @@
     <origin xyz="0 0 0" rpy="0 -0 0" />
     <geometry>
-    <mesh filename="package://optimo_description/meshes/plato/prox_collision.stl"/>
+    <mesh filename="file://$(find optimo_description)/meshes/plato/prox_collision.stl"/>
     </geometry>
     </collision>
@@ -78,5 +78,5 @@
     <origin xyz="0 0 0" rpy="0 -0 0" />
     <geometry>
-    <mesh filename="package://optimo_description/meshes/plato/mid_visual.stl"/>
+    <mesh filename="file://$(find optimo_description)/meshes/plato/mid_visual.stl"/>
     </geometry>
     <material name="mid_material">
@@ -87,5 +87,5 @@
     <origin xyz="0 0 0" rpy="0 -0 0" />
     <geometry>
-    <mesh filename="package://optimo_description/meshes/plato/mid_collision.stl"/>
+    <mesh filename="file://$(find optimo_description)/meshes/plato/mid_collision.stl"/>
     </geometry>
     </collision>
@@ -132,5 +132,5 @@
     <origin xyz="0 0 0" rpy="0 -0 0" />
     <geometry>
-    <mesh filename="package://optimo_description/meshes/plato/proxbracket_2_visual.stl"/>
+    <mesh filename="file://$(find optimo_description)/meshes/plato/proxbracket_2_visual.stl"/>
     </geometry>
     <material name="proxbracket_2_material">
@@ -141,5 +141,5 @@
     <origin xyz="0 0 0" rpy="0 -0 0" />
     <geometry>
-    <mesh filename="package://optimo_description/meshes/plato/proxbracket_2_collision.stl"/>
+    <mesh filename="file://$(find optimo_description)/meshes/plato/proxbracket_2_collision.stl"/>
     </geometry>
     </collision>
@@ -154,5 +154,5 @@
     <origin xyz="0 0 0" rpy="0 -0 0" />
     <geometry>
-    <mesh filename="package://optimo_description/meshes/plato/prox_2_visual.stl"/>
+    <mesh filename="file://$(find optimo_description)/meshes/plato/prox_2_visual.stl"/>
     </geometry>
     <material name="prox_2_material">
@@ -163,5 +163,5 @@
     <origin xyz="0 0 0" rpy="0 -0 0" />
     <geometry>
-    <mesh filename="package://optimo_description/meshes/plato/prox_2_collision.stl"/>
+    <mesh filename="file://$(find optimo_description)/meshes/plato/prox_2_collision.stl"/>
     </geometry>
     </collision>
@@ -176,5 +176,5 @@
     <origin xyz="0 0 0" rpy="0 -0 0" />
     <geometry>
-    <mesh filename="package://optimo_description/meshes/plato/mid_2_visual.stl"/>
+    <mesh filename="file://$(find optimo_description)/meshes/plato/mid_2_visual.stl"/>
     </geometry>
     <material name="mid_2_material">
@@ -185,5 +185,5 @@
     <origin xyz="0 0 0" rpy="0 -0 0" />
     <geometry>
-    <mesh filename="package://optimo_description/meshes/plato/mid_2_collision.stl"/>
+    <mesh filename="file://$(find optimo_description)/meshes/plato/mid_2_collision.stl"/>
     </geometry>
     </collision>
@@ -230,5 +230,5 @@
     <origin xyz="0 0 0" rpy="0 -0 0" />
     <geometry>
-    <mesh filename="package://optimo_description/meshes/plato/proxbracket_3_visual.stl"/>
+    <mesh filename="file://$(find optimo_description)/meshes/plato/proxbracket_3_visual.stl"/>
     </geometry>
     <material name="proxbracket_3_material">
@@ -239,5 +239,5 @@
     <origin xyz="0 0 0" rpy="0 -0 0" />
     <geometry>
-    <mesh filename="package://optimo_description/meshes/plato/proxbracket_3_collision.stl"/>
+    <mesh filename="file://$(find optimo_description)/meshes/plato/proxbracket_3_collision.stl"/>
     </geometry>
     </collision>
@@ -252,5 +252,5 @@
         <origin xyz="0 0 0" rpy="0 -0 0" />
         <geometry>
-        <mesh filename="package://optimo_description/meshes/plato/prox_3_visual.stl"/>
+        <mesh filename="file://$(find optimo_description)/meshes/plato/prox_3_visual.stl"/>
         </geometry>
         <material name="prox_3_material">
@@ -261,5 +261,5 @@
         <origin xyz="0 0 0" rpy="0 -0 0" />
         <geometry>
-        <mesh filename="package://optimo_description/meshes/plato/prox_3_collision.stl"/>
+        <mesh filename="file://$(find optimo_description)/meshes/plato/prox_3_collision.stl"/>
         </geometry>
         </collision>
@@ -274,5 +274,5 @@
         <origin xyz="0 0 0" rpy="0 -0 0" />
         <geometry>
-        <mesh filename="package://optimo_description/meshes/plato/mid_3_visual.stl"/>
+        <mesh filename="file://$(find optimo_description)/meshes/plato/mid_3_visual.stl"/>
         </geometry>
         <material name="mid_3_material">
@@ -283,5 +283,5 @@
         <origin xyz="0 0 0" rpy="0 -0 0" />
         <geometry>
-        <mesh filename="package://optimo_description/meshes/plato/mid_3_collision.stl"/>
+        <mesh filename="file://$(find optimo_description)/meshes/plato/mid_3_collision.stl"/>
         </geometry>
         </collision>
