Commit message: namespace added for optimo

File: optimo_description/urdf/optimo.urdf.xacro (robot description, xacro)
@@ -4,3 +4,14 @@
     <xacro:include filename="optimo_xacro/optimo.gazebo.xacro" />
     <xacro:include filename="optimo_xacro/optimo.control.xacro" />
+    <!-- Set Namespace for the Optimo Arm -->
+    <xacro:property name="robot_name" value="optimo" />
+    <xacro:optimo_arm ns = "${robot_name}"/>
+    <!-- Put World for Gazebo -->
+    <link name="world"/>
+    <!-- Connect to base_link of Optimo -->
+    <joint name="world_joint" type="fixed">
+        <parent link="world"/>
+        <child link="${robot_name}_base_link"/>
+        <origin xyz="0 0 0" rpy="0 0 0"/>
+    </joint>
 </robot>

File: optimo_description/urdf/optimo_xacro/optimo_arm.xacro (robot description, xacro)
@@ -3,300 +3,294 @@
     <xacro:property name="PI" value="3.1415926535897931"/>
     <xacro:property name="DtR" value=".01745329251"/>
-    <!-- Used for fixing robot to Gazebo 'base_link' -->
-    <link name="world"/>
-    <joint name="w2bl_joint" type="fixed">
-        <parent link="world"/>
-        <child link="base_link"/>
-        <origin xyz="0 0 0" rpy="0 0 0"/>
-    </joint>
-    <!-- Base Link -->
-    <link name="base_link">
-    </link>
-    <joint name="base_joint" type="fixed">
-        <parent link="base_link"/>
-        <child link="link0"/>
-        <origin xyz="0 0 0.27" rpy="0 0 0"/>
-    </joint>
-    <!-- Robot Links -->
-    <link name="link0">
-        <visual>
-            <geometry>
-                <mesh filename="file://$(find optimo_description)/meshes/link0.stl"/>
-            </geometry>
-            <material name="LightGrey">
-                <color rgba="0.999 0.999 0.999 1.0"/>
-            </material>
-        </visual>
-        <collision>
-            <geometry>
-                <mesh filename="file://$(find optimo_description)/meshes/col0.stl"/>
-            </geometry>
-        </collision>
-        <inertial>            <!-- Doesn't matter, just placeholder values -->
-            <origin xyz="0 0 0" />
-            <mass value="1"/>
-            <inertia ixx="0" ixy="0.0" ixz="0.0" iyy="0" iyz="0.0" izz="0"/>
-        </inertial>
-    </link>
-    <link name="link1">
-        <visual>
-            <geometry>
-                <sphere radius="0.01"/>
-            </geometry>
-            <material name="LightGrey">
-                <color rgba="0.999 0.999 0.999 1.0"/>
-            </material>
-        </visual>
-    </link>
-    <link name="link1_passive">
-        <visual>
-            <geometry>
-                <mesh filename="file://$(find optimo_description)/meshes/link1.stl"/>
-            </geometry>
-            <material name="LightGrey">
-                <color rgba="0.999 0.999 0.999 1.0"/>
-            </material>
-        </visual>
-        <collision>
-            <geometry>
-                <mesh filename="file://$(find optimo_description)/meshes/col1.stl"/>
-            </geometry>
-        </collision>
-        <inertial>
-            <origin xyz="0 -0.01635 0.01549" />
-            <mass value="4.152"/>
-            <inertia ixx="0.01" ixy="0.000017" ixz="-.00001" iyy="0.007494" iyz="0.0000213" izz="0.009939"/>
-        </inertial>
-    </link>
-    <link name="link2"/>
-    <link name="link2_passive">
-        <visual>
-            <geometry>
-                <mesh filename="file://$(find optimo_description)/meshes/link2.stl"/>
-            </geometry>
-            <material name="LightGrey">
-                <color rgba="0.999 0.999 0.999 1.0"/>
-            </material>
-        </visual>
-        <collision>
-            <geometry>
-                <mesh filename="file://$(find optimo_description)/meshes/col2.stl"/>
-            </geometry>
-        </collision>
-        <inertial>
-            <origin xyz="0 -0.05063 0.05677" />
-            <mass value="1.72"/>
-            <inertia ixx="0.005694" ixy="0" ixz="0" iyy="0.005902" iyz="0.001353" izz="0.002415"/>
-        </inertial>
-    </link>
-    <link name="link3"/>
-    <link name="link3_passive">
-        <visual>
-            <geometry>
-                <mesh filename="file://$(find optimo_description)/meshes/link3.stl"/>
-            </geometry>
-            <material name="LightGrey">
-                <color rgba="0.999 0.999 0.999 1.0"/>
-            </material>
-        </visual>
-        <collision>
-            <geometry>
-                <mesh filename="file://$(find optimo_description)/meshes/col3.stl"/>
-            </geometry>
-        </collision>
-        <inertial>            <!-- Inertia values taken from yaml, but these seem like they cannot be accurate...-->
-            <origin xyz="-0.000039 .098 0" />
-            <mass value="4.310"/>
-            <inertia ixx="0.012989" ixy="-0.000015" ixz="-.000003" iyy="0.002584" iyz="0.000632" izz="0.01305"/>
-        </inertial>
-    </link>
-    <link name="link4"/>
-    <link name="link4_passive">
-        <visual>
-            <geometry>
-                <mesh filename="file://$(find optimo_description)/meshes/link4.stl"/>
-            </geometry>
-            <material name="LightGrey">
-                <color rgba="0.999 0.999 0.999 1.0"/>
-            </material>
-        </visual>
-        <collision>
-            <geometry>
-                <mesh filename="file://$(find optimo_description)/meshes/col4.stl"/>
-            </geometry>
-        </collision>
-        <inertial>
-            <origin xyz="-.00001 0.048852 0.0688" />
-            <mass value="1.09"/>
-            <inertia ixx="0.033673" ixy="-.00046473" ixz="0" iyy="0.001089" iyz="0.000095" izz="0.033877"/>
-        </inertial>
-    </link>
-    <link name="link5"/>
-    <link name="link5_passive">
-        <visual>
-            <geometry>
-                <mesh filename="file://$(find optimo_description)/meshes/link5.stl"/>
-            </geometry>
-            <material name="LightGrey">
-                <color rgba="0.999 0.999 0.999 1.0"/>
-            </material>
-        </visual>
-        <collision>
-            <geometry>
-                <mesh filename="file://$(find optimo_description)/meshes/col5.stl"/>
-            </geometry>
-        </collision>
-        <inertial>
-            <origin xyz=".001262 0.085 0.008" />
-            <mass value="2.23"/>
-            <inertia ixx="0.000932" ixy="0" ixz="0" iyy="0.000802" iyz="-0.000030" izz="0.000733"/>
-        </inertial>
-    </link>
-    <link name="link6"/>
-    <link name="link6_passive">
-        <visual>
-            <geometry>
-                <mesh filename="file://$(find optimo_description)/meshes/link6.stl"/>
-            </geometry>
-            <material name="LightGrey">
-                <color rgba="0.999 0.999 0.999 1.0"/>
-            </material>
-        </visual>
-        <collision>
-            <geometry>
-                <mesh filename="file://$(find optimo_description)/meshes/col6.stl"/>
-            </geometry>
-        </collision>
-        <inertial>
-            <origin xyz="0 -0.00007 0.010855" />
-            <mass value="1.138"/>
-            <inertia ixx="0.000932" ixy="0" ixz="0" iyy="0.000802" iyz="-0.000030" izz="0.0007325"/>
-        </inertial>
-    </link>
-    <link name="link7"/>
-    <link name="link7_passive">
-        <visual>
-            <geometry>
-                <mesh filename="file://$(find optimo_description)/meshes/link7.stl"/>
-            </geometry>
-            <material name="LightGrey">
-                <color rgba="0.999 0.999 0.999 1.0"/>
-            </material>
-        </visual>
-        <collision>
-            <geometry>
-                <mesh filename="file://$(find optimo_description)/meshes/col7.stl"/>
-            </geometry>
-        </collision>
-        <inertial>
-            <origin xyz="-.015 0 0.14" />
-            <mass value="1"/>
-            <inertia ixx="0.005541" ixy=".000045" ixz="0.000077" iyy="0.004779" iyz="0.000043" izz="0.001723"/>
-        </inertial>
-    </link>
-    <!-- <joint name='jN' type='revolute'>
-      <child>LINK NAME</child>
-      <parent>LINK NAME</parent>
-      <axis>
-        <xyz>AXIS OF ROTATION, IN JOINT FRAME</xyz>
-        <limit>
-          <lower>RADIANS FOR REVOLUTE/ METERS FOR PRISMATIC</lower>
-          <upper></upper>
-          <effort></effort>
-          <velocity></velocity>
-        </limit>
-        <dynamics>
-          <damping>VISCOUS DAMPING COEFFICIENT</damping>
-          <friction>PHYSICAL STATIC FRICTION</friction>
-          <spring_reference>SPRING REF POSITION FOR THIS JOINT AXIS</spring_reference>
-          <spring_stiffness>SPRING STIFFNESS FOR THIS JOINT AXIS</spring_stiffness>
-        </dynamics>
-        <use_parent_model_frame>1</use_parent_model_frame>
-      </axis>
-    </joint> -->
-    <!-- Joints -->
-    <joint name="joint1" type="revolute">
-        <origin xyz="0 0 0" rpy="0 0 0"/>
-        <parent link="link0"/>
-        <child link="link1"/>
-        <axis xyz="0 0 1"/>
-        <limit lower="${DtR*-164}" upper="${DtR*167}" effort="79" velocity="10"/>
-    </joint>
-    <joint name="joint1_passive" type="fixed">
-        <origin xyz="0 0 0" rpy="${PI/2} 0 0"/>
-        <parent link="link1"/>
-        <child link="link1_passive"/>
-    </joint>
-    <joint name="joint2" type="revolute">
-        <origin xyz="0 0 0" rpy="0 0 0"/>
-        <parent link="link1_passive"/>
-        <child link="link2"/>
-        <axis xyz="0 0 1"/>
-        <limit lower="${DtR*60}" upper="${DtR*250}" effort="95" velocity="10"/>
-    </joint>
-    <joint name="joint2_passive" type="fixed">
-        <origin xyz="0 0 0" rpy="${PI/2} 0 0"/>
-        <parent link="link2"/>
-        <child link="link2_passive"/>
-    </joint>
-    <joint name="joint3" type="revolute">
-        <origin xyz="0 0 0.4" rpy="0 0 0"/>
-        <parent link="link2_passive"/>
-        <child link="link3"/>
-        <axis xyz="0 0 1"/>
-        <limit lower="${DtR*-167}" upper="${DtR*163}" effort="32" velocity="10"/>
-    </joint>
-    <joint name="joint3_passive" type="fixed">
-        <origin xyz="0 0 0" rpy="-${PI/2} 0 0"/>
-        <parent link="link3"/>
-        <child link="link3_passive"/>
-    </joint>
-    <joint name="joint4" type="revolute">
-        <origin xyz="0 0 0" rpy="0 0 0"/>
-        <parent link="link3_passive"/>
-        <child link="link4"/>
-        <axis xyz="0 0 1"/>
-        <limit lower="${DtR*-145}" upper="${DtR*145}" effort="40" velocity="10"/>
-    </joint>
-    <joint name="joint4_passive" type="fixed">
-        <origin xyz="0 0 0" rpy="${PI/2} 0 0"/>
-        <parent link="link4"/>
-        <child link="link4_passive"/>
-    </joint>
-    <joint name="joint5" type="revolute">
-        <origin xyz="0 0 0.4" rpy="0 0 0"/>
-        <parent link="link4_passive"/>
-        <child link="link5"/>
-        <axis xyz="0 0 1"/>
-        <limit lower="${DtR*-170}" upper="${DtR*170}" effort="15" velocity="10"/>
-    </joint>
-    <joint name="joint5_passive" type="fixed">
-        <origin xyz="0 0 0" rpy="-${PI/2} 0 0"/>
-        <parent link="link5"/>
-        <child link="link5_passive"/>
-    </joint>
-    <joint name="joint6" type="revolute">
-        <origin xyz="0 0 0" rpy="0 0 0"/>
-        <parent link="link5_passive"/>
-        <child link="link6"/>
-        <axis xyz="0 0 1"/>
-        <limit lower="${DtR*-120}" upper="${DtR*120}" effort="15" velocity="10"/>
-    </joint>
-    <joint name="joint6_passive" type="fixed">
-        <origin xyz="0 0 0" rpy="${PI/2} 0 0"/>
-        <parent link="link6"/>
-        <child link="link6_passive"/>
-    </joint>
-     <joint name="joint7" type="revolute">
-        <origin xyz="0 0 0" rpy="0 0 0"/>
-        <parent link="link6_passive"/>
-        <child link="link7"/>
-        <axis xyz="0 0 1"/>
-        <limit lower="${DtR*-152}" upper="${DtR*188}" effort="15" velocity="10"/>
-    </joint>
-    <joint name="joint7_passive" type="fixed">
-        <origin xyz="0 0 0" rpy="${PI/2} 0 0"/>
-        <parent link="link7"/>
-        <child link="link7_passive"/>
-    </joint>
+    <xacro:macro name="optimo_arm" params="ns:='optimo'">
+        <link name="${ns}_base_link">
+        </link>
+        <joint name="${ns}_base_joint" type="fixed">
+            <parent link="${ns}_base_link"/>
+            <child link="${ns}_link0"/>
+            <origin xyz="0 0 0.27" rpy="0 0 0"/>
+        </joint>
+        <!-- Robot Links -->
+        <link name="${ns}_link0">
+            <visual>
+                <geometry>
+                    <mesh filename="file://$(find optimo_description)/meshes/link0.stl"/>
+                </geometry>
+                <material name="LightGrey">
+                    <color rgba="0.999 0.999 0.999 1.0"/>
+                </material>
+            </visual>
+            <collision>
+                <geometry>
+                    <mesh filename="file://$(find optimo_description)/meshes/col0.stl"/>
+                </geometry>
+            </collision>
+            <inertial>            <!-- Doesn't matter, just placeholder values -->
+                <origin xyz="0 0 0" />
+                <mass value="1"/>
+                <inertia ixx="0" ixy="0.0" ixz="0.0" iyy="0" iyz="0.0" izz="0"/>
+            </inertial>
+        </link>
+        <link name="${ns}_link1">
+            <visual>
+                <geometry>
+                    <sphere radius="0.01"/>
+                </geometry>
+                <material name="LightGrey">
+                    <color rgba="0.999 0.999 0.999 1.0"/>
+                </material>
+            </visual>
+        </link>
+        <link name="${ns}_link1_passive">
+            <visual>
+                <geometry>
+                    <mesh filename="file://$(find optimo_description)/meshes/link1.stl"/>
+                </geometry>
+                <material name="LightGrey">
+                    <color rgba="0.999 0.999 0.999 1.0"/>
+                </material>
+            </visual>
+            <collision>
+                <geometry>
+                    <mesh filename="file://$(find optimo_description)/meshes/col1.stl"/>
+                </geometry>
+            </collision>
+            <inertial>
+                <origin xyz="0 -0.01635 0.01549" />
+                <mass value="4.152"/>
+                <inertia ixx="0.01" ixy="0.000017" ixz="-.00001" iyy="0.007494" iyz="0.0000213" izz="0.009939"/>
+            </inertial>
+        </link>
+        <link name="${ns}_link2"/>
+        <link name="${ns}_link2_passive">
+            <visual>
+                <geometry>
+                    <mesh filename="file://$(find optimo_description)/meshes/link2.stl"/>
+                </geometry>
+                <material name="LightGrey">
+                    <color rgba="0.999 0.999 0.999 1.0"/>
+                </material>
+            </visual>
+            <collision>
+                <geometry>
+                    <mesh filename="file://$(find optimo_description)/meshes/col2.stl"/>
+                </geometry>
+            </collision>
+            <inertial>
+                <origin xyz="0 -0.05063 0.05677" />
+                <mass value="1.72"/>
+                <inertia ixx="0.005694" ixy="0" ixz="0" iyy="0.005902" iyz="0.001353" izz="0.002415"/>
+            </inertial>
+        </link>
+        <link name="${ns}_link3"/>
+        <link name="${ns}_link3_passive">
+            <visual>
+                <geometry>
+                    <mesh filename="file://$(find optimo_description)/meshes/link3.stl"/>
+                </geometry>
+                <material name="LightGrey">
+                    <color rgba="0.999 0.999 0.999 1.0"/>
+                </material>
+            </visual>
+            <collision>
+                <geometry>
+                    <mesh filename="file://$(find optimo_description)/meshes/col3.stl"/>
+                </geometry>
+            </collision>
+            <inertial>            <!-- Inertia values taken from yaml, but these seem like they cannot be accurate...-->
+                <origin xyz="-0.000039 .098 0" />
+                <mass value="4.310"/>
+                <inertia ixx="0.012989" ixy="-0.000015" ixz="-.000003" iyy="0.002584" iyz="0.000632" izz="0.01305"/>
+            </inertial>
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
Commit message: torque_controller tuning start

File: optimo_description/urdf/optimo.urdf.xacro (robot description, xacro)
@@ -3,16 +3,15 @@
     <!-- Bring xacro files -->
     <xacro:include filename="optimo_xacro/optimo_arm.xacro"/>
-    <xacro:include filename="optimo_xacro/optimo.gazebo.xacro" />
-    <xacro:include filename="optimo_xacro/optimo.control.xacro" />
     <!-- Set Namespace for the Optimo Arm -->
-    <xacro:property name="robot_name" value="optimo" />
-    <xacro:optimo_arm ns = "${robot_name}"/>
+    <xacro:property name="arm_ns" value="optimo" />
+    <xacro:optimo_arm ns ="${arm_ns}"/>
     <!-- Put World for Gazebo -->
     <link name="world"/>
-    <!-- Connect to base_link of Optimo -->
     <joint name="world_joint" type="fixed">
         <parent link="world"/>
-        <child link="${robot_name}_base_link"/>
+        <child link="${arm_ns}_base_link"/>
         <origin xyz="0 0 0" rpy="0 0 0"/>
     </joint>
+    <xacro:include filename="optimo_xacro/optimo.gazebo.xacro" />
+    <xacro:include filename="optimo_xacro/optimo.effort_control.xacro" />
 </robot>

File: optimo_description/urdf/optimo_xacro/optimo.effort_control.xacro (robot description, xacro)
@@ -13,5 +13,5 @@
             </hardware>
             <joint name="optimo_joint1">
-                <command_interface name="position">
+                <command_interface name="effort">
                 </command_interface>
                 <state_interface name="position">
@@ -21,13 +21,13 @@
             </joint>
             <joint name="optimo_joint2">
-                 <command_interface name="position">
+                <command_interface name="effort">
                 </command_interface>
                 <state_interface name="position">
-                    <param name="initial_value">2.74</param>
+                    <param name="initial_value">2.768</param>
                 </state_interface>
                 <state_interface name="velocity" />
             </joint>
             <joint name="optimo_joint3">
-                <command_interface name="position">
+                <command_interface name="effort">
                 </command_interface>
                 <state_interface name="position">
@@ -37,5 +37,5 @@
             </joint>
             <joint name="optimo_joint4">
-                <command_interface name="position">
+                <command_interface name="effort">
                 </command_interface>
                 <state_interface name="position">
@@ -45,5 +45,5 @@
             </joint>
             <joint name="optimo_joint5">
-                <command_interface name="position">
+                <command_interface name="effort">
                 </command_interface>
                 <state_interface name="position">
@@ -53,5 +53,5 @@
             </joint>
             <joint name="optimo_joint6">
-                <command_interface name="position">
+                <command_interface name="effort">
                 </command_interface>
                 <state_interface name="position">
@@ -61,5 +61,5 @@
             </joint>
             <joint name="optimo_joint7">
-                <command_interface name="position">
+                <command_interface name="effort">
                 </command_interface>
                 <state_interface name="position">

File: optimo_description/urdf/optimo_xacro/optimo.gazebo.xacro (robot description, xacro)
@@ -4,30 +4,30 @@
     <xacro:property name="DtR" value=".01745329251"/>
     <gazebo reference="base_link"/>
-    <gazebo reference="link0"/>
-    <gazebo reference="link1"/>
-    <gazebo reference="link1_passive"/>
-    <gazebo reference="link2"/>
-    <gazebo reference="link2_passive"/>
-    <gazebo reference="link3"/>
-    <gazebo reference="link3_passive"/>
-    <gazebo reference="link4"/>
-    <gazebo reference="link4_passive"/>
-    <gazebo reference="link5"/>
-    <gazebo reference="link5_passive"/>
-    <gazebo reference="link6"/>
-    <gazebo reference="link6_passive"/>
-    <gazebo reference="link7"/>
-    <gazebo reference="link7_passive"/>
+    <gazebo reference="optimo_link0"/>
+    <gazebo reference="optimo_link1"/>
+    <gazebo reference="optimo_link1_passive"/>
+    <gazebo reference="optimo_link2"/>
+    <gazebo reference="optimo_link2_passive"/>
+    <gazebo reference="optimo_link3"/>
+    <gazebo reference="optimo_link3_passive"/>
+    <gazebo reference="optimo_link4"/>
+    <gazebo reference="optimo_link4_passive"/>
+    <gazebo reference="optimo_link5"/>
+    <gazebo reference="optimo_link5_passive"/>
+    <gazebo reference="optimo_link6"/>
+    <gazebo reference="optimo_link6_passive"/>
+    <gazebo reference="optimo_link7"/>
+    <gazebo reference="optimo_link7_passive"/>
     <!-- Joint State Publisher -->
     <gazebo>
         <plugin name="gazebo_ros_joint_state_publisher" filename="libgazebo_ros_joint_state_publisher.so">
             <update_rate>1000</update_rate>
-            <joint_name>joint1</joint_name>
-            <joint_name>joint2</joint_name>
-            <joint_name>joint3</joint_name>
-            <joint_name>joint4</joint_name>
-            <joint_name>joint5</joint_name>
-            <joint_name>joint6</joint_name>
-            <joint_name>joint7</joint_name>
+            <joint_name>optimo_joint1</joint_name>
+            <joint_name>optimo_joint2</joint_name>
+            <joint_name>optimo_joint3</joint_name>
+            <joint_name>optimo_joint4</joint_name>
+            <joint_name>optimo_joint5</joint_name>
+            <joint_name>optimo_joint6</joint_name>
+            <joint_name>optimo_joint7</joint_name>
         </plugin>
     </gazebo>

File: plato_description/urdf/plato_manipulator.urdf.xacro (robot description, xacro)
@@ -24,3 +24,7 @@
         <origin xyz="0 0.16 0" rpy="1.5707 0 1.5707"/>
     </joint>
+    <!-- Make sure to include the controllers after all joints are defined -->
+    <!-- Optimo Gazebo Parameters and ros2_controller -->
+    <xacro:include filename="$(find optimo_description)/urdf/optimo_xacro/optimo.gazebo.xacro"/>
+    <xacro:include filename="$(find optimo_description)/urdf/optimo_xacro/optimo.control.xacro"/>
 </robot>
