Commit message: changed back to position controller

File: optimo_description/urdf/optimo.urdf.xacro (robot description, xacro)
@@ -13,5 +13,8 @@
         <origin xyz="0 0 0" rpy="0 0 0"/>
     </joint>
+    <!-- Include Physics Parameters in Gazebo -->
     <xacro:include filename="optimo_xacro/optimo.gazebo.xacro" />
-    <xacro:include filename="optimo_xacro/optimo.effort_control.xacro" />
+    <!-- Include ros2_control -->
+    <xacro:include filename="optimo_xacro/optimo.control.xacro" />
+    <xacro:optimo_ros2_control ns="${arm_ns}"/>
 </robot>

File: optimo_description/urdf/optimo_xacro/optimo.control.xacro (robot description, xacro)
@@ -1,71 +1,32 @@
-<?xml version="1.0"?>
+<?xml version="1.0" encoding="utf-8"?>
 <robot xmlns:xacro="http://www.ros.org/wiki/xacro">
-        <!-- Optimo ROS 2 Controller -->
-        <gazebo>
-            <plugin filename="libgazebo_ros2_control.so" name="gazebo_ros2_control">
-                <parameters>$(find plato_moveit)/config/optimo_controller.yaml</parameters>
-            </plugin>
-        </gazebo>
-        <!--  ROS 2 Controller for Gazebo -->
+    <gazebo>
+        <plugin filename="libgazebo_ros2_control.so" name="gazebo_ros2_control">
+            <parameters>$(find plato_bringup)/config/optimo_controllers.yaml</parameters>
+        </plugin>
+    </gazebo>
+    <xacro:macro name="optimo_ros2_control" params="ns">
         <ros2_control name="GazeboSystem" type="system">
             <hardware>
                 <plugin>gazebo_ros2_control/GazeboSystem</plugin>
             </hardware>
-            <joint name="optimo_joint1">
-                <command_interface name="position">
-                </command_interface>
-                <state_interface name="position">
-                    <param name="initial_value">0.0</param>
-                </state_interface>
-                <state_interface name="velocity" />
-            </joint>
-            <joint name="optimo_joint2">
-                 <command_interface name="position">
-                </command_interface>
-                <state_interface name="position">
-                    <param name="initial_value">2.74</param>
-                </state_interface>
-                <state_interface name="velocity" />
-            </joint>
-            <joint name="optimo_joint3">
-                <command_interface name="position">
-                </command_interface>
-                <state_interface name="position">
-                    <param name="initial_value">0.0</param>
-                </state_interface>
-                <state_interface name="velocity" />
-            </joint>
-            <joint name="optimo_joint4">
-                <command_interface name="position">
-                </command_interface>
-                <state_interface name="position">
-                    <param name="initial_value">-1.847</param>
-                </state_interface>
-                <state_interface name="velocity" />
-            </joint>
-            <joint name="optimo_joint5">
-                <command_interface name="position">
-                </command_interface>
-                <state_interface name="position">
-                    <param name="initial_value">0.0</param>
-                </state_interface>
-                <state_interface name="velocity" />
-            </joint>
-            <joint name="optimo_joint6">
-                <command_interface name="position">
-                </command_interface>
-                <state_interface name="position">
-                    <param name="initial_value">0.713</param>
-                </state_interface>
-                <state_interface name="velocity" />
-            </joint>
-            <joint name="optimo_joint7">
-                <command_interface name="position">
-                </command_interface>
-                <state_interface name="position">
-                    <param name="initial_value">0.0</param>
-                </state_interface>
-                <state_interface name="velocity" />
-            </joint>
+            <xacro:macro name="configure_joint" params="joint_name initial_position">
+                <joint name="${joint_name}">
+                    <command_interface name="position" />
+                    <state_interface name="position">
+                        <param name="initial_value">${initial_position}</param>
+                    </state_interface>
+                    <state_interface name="velocity" />
+                    <state_interface name="effort" />
+                </joint>
+            </xacro:macro>
+            <xacro:configure_joint joint_name="${ns}_joint1" initial_position="$0" />
+            <xacro:configure_joint joint_name="${ns}_joint2" initial_position="${160*DtR}" />
+            <xacro:configure_joint joint_name="${ns}_joint3" initial_position="0.0" />
+            <xacro:configure_joint joint_name="${ns}_joint4" initial_position="${-60*DtR}" />
+            <xacro:configure_joint joint_name="${ns}_joint5" initial_position="0.0" />
+            <xacro:configure_joint joint_name="${ns}_joint6" initial_position="${-30*DtR}" />
+            <xacro:configure_joint joint_name="${ns}_joint7" initial_position="0.0" />
         </ros2_control>
+    </xacro:macro>
 </robot>

File: optimo_description/urdf/optimo_xacro/optimo_arm.xacro (robot description, xacro)
@@ -3,4 +3,13 @@
     <xacro:property name="PI" value="3.1415926535897931"/>
     <xacro:property name="DtR" value=".01745329251"/>
+    <xacro:property name="mass_link0" value="3.06357" />
+    <xacro:property name="mass_link1" value="2.34471" />
+    <xacro:property name="mass_link2" value="2.36414" />
+    <xacro:property name="mass_link3" value="2.38050" />
+    <xacro:property name="mass_link4" value="2.42754" />
+    <xacro:property name="mass_link5" value="3.49611" />
+    <xacro:property name="mass_link6" value="1.46736" />
+    <xacro:property name="mass_link7" value="0.45606" />
+    <xacro:property name="mass_link8" value="0.001" />
     <xacro:macro name="optimo_arm" params="ns:='optimo'">
         <link name="${ns}_base_link">
@@ -78,7 +87,9 @@
             </collision>
             <inertial>
-                <origin xyz="0 -0.05063 0.05677" />
+                <origin xyz="0 -0.05063 0.05677"  rpy="0 0 ${180*DtR}"/>
                 <mass value="1.72"/>
-                <inertia ixx="0.005694" ixy="0" ixz="0" iyy="0.005902" iyz="0.001353" izz="0.002415"/>
+                 <!-- <inertia ixx="0.005902" ixy="0" ixz="-0.001353" iyy="0.005694" iyz="0" izz="0.002415"/> -->
+                 <!-- <inertia ixx="0.005694" ixy="0" ixz="0" iyy="0.005902" iyz="0.001353" izz="0.002415"/> -->
+                  <inertia ixx="0.005694" ixy="0" ixz="0" iyy="0.005902" iyz="-0.001353" izz="0.002415"/>
             </inertial>
         </link>
@@ -99,5 +110,5 @@
             </collision>
             <inertial>            <!-- Inertia values taken from yaml, but these seem like they cannot be accurate...-->
-                <origin xyz="-0.000039 .098 0" />
+                <origin xyz="-0.000039 .098 0"/>
                 <mass value="4.310"/>
                 <inertia ixx="0.012989" ixy="-0.000015" ixz="-.000003" iyy="0.002584" iyz="0.000632" izz="0.01305"/>
@@ -106,4 +117,5 @@
         <link name="${ns}_link4"/>
         <link name="${ns}_link4_passive">
+            <origin xyz="0 0 0" rpy="0 0 0"/>
             <visual>
                 <geometry>
@@ -120,7 +132,8 @@
             </collision>
             <inertial>
-                <origin xyz="-.00001 0.048852 0.0688" />
+                <origin xyz="-.00001 0.048852 0.0688" rpy="0 0 0"/>
                 <mass value="1.09"/>
-                <inertia ixx="0.033673" ixy="-.00046473" ixz="0" iyy="0.001089" iyz="0.000095" izz="0.033877"/>
+                 <!-- <inertia ixx="0.007" ixy="-3.989e-7" ixz="0.002" iyy="0.007" iyz="-1.061e-6" izz="0.002"/> -->
+                <inertia ixx="0.007" ixy="3.989e-7" ixz="-0.002" iyy="0.007" iyz="-1.061e-6" izz="0.002"/>
             </inertial>
         </link>
@@ -183,5 +196,5 @@
             </collision>
             <inertial>
-                <origin xyz="-.015 0 0.14" />
+                <origin xyz="0 0 0" />
                 <mass value="1"/>
                 <inertia ixx="0.005541" ixy=".000045" ixz="0.000077" iyy="0.004779" iyz="0.000043" izz="0.001723"/>

Commit message: gazeo does not spawn with controller

File: optimo_description/urdf/optimo.urdf.xacro (robot description, xacro)
@@ -17,4 +17,4 @@
     <!-- Include ros2_control -->
     <xacro:include filename="optimo_xacro/optimo.control.xacro" />
-    <xacro:optimo_ros2_control ns="${arm_ns}"/>
+    <!-- <xacro:optimo_ros2_control ns="${arm_ns}"/> -->
 </robot>

File: optimo_description/urdf/optimo_xacro/optimo.control.xacro (robot description, xacro)
@@ -3,8 +3,9 @@
     <gazebo>
         <plugin filename="libgazebo_ros2_control.so" name="gazebo_ros2_control">
-            <parameters>$(find plato_bringup)/config/optimo_controllers.yaml</parameters>
+            <parameters>$(find plato_gazebo)/config/optimo_controllers.yaml</parameters>
         </plugin>
     </gazebo>
-    <xacro:macro name="optimo_ros2_control" params="ns">
+    <xacro:property name="ns" value="optimo" />
+    <!-- <xacro:macro name="optimo_ros2_control" params="ns:=optimo"> -->
         <ros2_control name="GazeboSystem" type="system">
             <hardware>
@@ -18,5 +19,4 @@
                     </state_interface>
                     <state_interface name="velocity" />
-                    <state_interface name="effort" />
                 </joint>
             </xacro:macro>
@@ -29,4 +29,4 @@
             <xacro:configure_joint joint_name="${ns}_joint7" initial_position="0.0" />
         </ros2_control>
-    </xacro:macro>
+    <!-- </xacro:macro> -->
 </robot>

File: optimo_description/urdf/optimo_xacro/optimo_arm.xacro (robot description, xacro)
@@ -68,5 +68,6 @@
                 <origin xyz="0 -0.01635 0.01549" />
                 <mass value="4.152"/>
-                <inertia ixx="0.01" ixy="0.000017" ixz="-.00001" iyy="0.007494" iyz="0.0000213" izz="0.009939"/>
+                <!-- <inertia ixx="0.01" ixy="0.000017" ixz="-.00001" iyy="0.007494" iyz="0.0000213" izz="0.009939"/> -->
+                <inertia ixx="0" ixy="0.0" ixz="0.0" iyy="0" iyz="0.0" izz="0"/>
             </inertial>
         </link>
@@ -89,7 +90,6 @@
                 <origin xyz="0 -0.05063 0.05677"  rpy="0 0 ${180*DtR}"/>
                 <mass value="1.72"/>
-                 <!-- <inertia ixx="0.005902" ixy="0" ixz="-0.001353" iyy="0.005694" iyz="0" izz="0.002415"/> -->
-                 <!-- <inertia ixx="0.005694" ixy="0" ixz="0" iyy="0.005902" iyz="0.001353" izz="0.002415"/> -->
-                  <inertia ixx="0.005694" ixy="0" ixz="0" iyy="0.005902" iyz="-0.001353" izz="0.002415"/>
+                  <!-- <inertia ixx="0.005694" ixy="0" ixz="0" iyy="0.005902" iyz="-0.001353" izz="0.002415"/> -->
+                  <inertia ixx="0" ixy="0.0" ixz="0.0" iyy="0" iyz="0.0" izz="0"/>
             </inertial>
         </link>
@@ -112,5 +112,6 @@
                 <origin xyz="-0.000039 .098 0"/>
                 <mass value="4.310"/>
-                <inertia ixx="0.012989" ixy="-0.000015" ixz="-.000003" iyy="0.002584" iyz="0.000632" izz="0.01305"/>
+                <!-- <inertia ixx="0.012989" ixy="-0.000015" ixz="-.000003" iyy="0.002584" iyz="0.000632" izz="0.01305"/> -->
+                <inertia ixx="0" ixy="0.0" ixz="0.0" iyy="0" iyz="0.0" izz="0"/>
             </inertial>
         </link>
@@ -135,5 +136,6 @@
                 <mass value="1.09"/>
                  <!-- <inertia ixx="0.007" ixy="-3.989e-7" ixz="0.002" iyy="0.007" iyz="-1.061e-6" izz="0.002"/> -->
-                <inertia ixx="0.007" ixy="3.989e-7" ixz="-0.002" iyy="0.007" iyz="-1.061e-6" izz="0.002"/>
+                <!-- <inertia ixx="0.007" ixy="3.989e-7" ixz="-0.002" iyy="0.007" iyz="-1.061e-6" izz="0.002"/> -->
+                <inertia ixx="0" ixy="0.0" ixz="0.0" iyy="0" iyz="0.0" izz="0"/>
             </inertial>
         </link>
@@ -156,5 +158,6 @@
                 <origin xyz=".001262 0.085 0.008" />
                 <mass value="2.23"/>
-                <inertia ixx="0.000932" ixy="0" ixz="0" iyy="0.000802" iyz="-0.000030" izz="0.000733"/>
+                <!-- <inertia ixx="0.000932" ixy="0" ixz="0" iyy="0.000802" iyz="-0.000030" izz="0.000733"/> -->
+                <inertia ixx="0" ixy="0.0" ixz="0.0" iyy="0" iyz="0.0" izz="0"/>
             </inertial>
         </link>
@@ -177,5 +180,6 @@
                 <origin xyz="0 -0.00007 0.010855" />
                 <mass value="1.138"/>
-                <inertia ixx="0.000932" ixy="0" ixz="0" iyy="0.000802" iyz="-0.000030" izz="0.0007325"/>
+                <!-- <inertia ixx="0.000932" ixy="0" ixz="0" iyy="0.000802" iyz="-0.000030" izz="0.0007325"/> -->
+                <inertia ixx="0" ixy="0.0" ixz="0.0" iyy="0" iyz="0.0" izz="0"/>
             </inertial>
         </link>
@@ -198,5 +202,6 @@
                 <origin xyz="0 0 0" />
                 <mass value="1"/>
-                <inertia ixx="0.005541" ixy=".000045" ixz="0.000077" iyy="0.004779" iyz="0.000043" izz="0.001723"/>
+                <!-- <inertia ixx="0.005541" ixy=".000045" ixz="0.000077" iyy="0.004779" iyz="0.000043" izz="0.001723"/> -->
+                <inertia ixx="0" ixy="0.0" ixz="0.0" iyy="0" iyz="0.0" izz="0"/>
             </inertial>
         </link>

Commit message: pos controller fixed

File: optimo_description/urdf/optimo.urdf.xacro (robot description, xacro)
@@ -17,4 +17,4 @@
     <!-- Include ros2_control -->
     <xacro:include filename="optimo_xacro/optimo.control.xacro" />
-    <!-- <xacro:optimo_ros2_control ns="${arm_ns}"/> -->
+    <xacro:optimo_ros2_control ns="${arm_ns}"/>
 </robot>

File: optimo_description/urdf/optimo_xacro/optimo.control.xacro (robot description, xacro)
@@ -1,12 +1,12 @@
-<?xml version="1.0" encoding="utf-8"?>
+<?xml version="1.0"?>
 <robot xmlns:xacro="http://www.ros.org/wiki/xacro">
+    <!-- Optimo ROS 2 Controller -->
     <gazebo>
         <plugin filename="libgazebo_ros2_control.so" name="gazebo_ros2_control">
-            <parameters>$(find plato_gazebo)/config/optimo_controllers.yaml</parameters>
+            <parameters>$(find plato_bringup)/config/optimo_controllers.yaml</parameters>
         </plugin>
     </gazebo>
-    <xacro:property name="ns" value="optimo" />
-    <!-- <xacro:macro name="optimo_ros2_control" params="ns:=optimo"> -->
-        <ros2_control name="GazeboSystem" type="system">
+    <xacro:macro name="optimo_ros2_control" params="ns">
+        <ros2_control name="OptimoGazebo" type="system">
             <hardware>
                 <plugin>gazebo_ros2_control/GazeboSystem</plugin>
@@ -14,19 +14,19 @@
             <xacro:macro name="configure_joint" params="joint_name initial_position">
                 <joint name="${joint_name}">
-                    <command_interface name="position" />
+                    <command_interface name="position"/>
                     <state_interface name="position">
                         <param name="initial_value">${initial_position}</param>
                     </state_interface>
-                    <state_interface name="velocity" />
+                    <state_interface name="velocity"/>
                 </joint>
             </xacro:macro>
-            <xacro:configure_joint joint_name="${ns}_joint1" initial_position="$0" />
-            <xacro:configure_joint joint_name="${ns}_joint2" initial_position="${160*DtR}" />
-            <xacro:configure_joint joint_name="${ns}_joint3" initial_position="0.0" />
-            <xacro:configure_joint joint_name="${ns}_joint4" initial_position="${-60*DtR}" />
-            <xacro:configure_joint joint_name="${ns}_joint5" initial_position="0.0" />
-            <xacro:configure_joint joint_name="${ns}_joint6" initial_position="${-30*DtR}" />
-            <xacro:configure_joint joint_name="${ns}_joint7" initial_position="0.0" />
+            <xacro:configure_joint joint_name="${ns}_joint1" initial_position="0.0"/>
+            <xacro:configure_joint joint_name="${ns}_joint2" initial_position="3.14"/>
+            <xacro:configure_joint joint_name="${ns}_joint3" initial_position="0.0"/>
+            <xacro:configure_joint joint_name="${ns}_joint4" initial_position="0.0"/>
+            <xacro:configure_joint joint_name="${ns}_joint5" initial_position="0.0"/>
+            <xacro:configure_joint joint_name="${ns}_joint6" initial_position="0.0"/>
+            <xacro:configure_joint joint_name="${ns}_joint7" initial_position="0.0"/>
         </ros2_control>
-    <!-- </xacro:macro> -->
+  </xacro:macro>
 </robot>
