Commit message: arm+hand gazebo working

File: plato_description/urdf/plato_xacro/plato_hand.xacro (robot description, xacro)
@@ -1,12 +1,11 @@
 <?xml version="1.0"?>
 <robot xmlns:xacro="http://www.ros.org/wiki/xacro">
-<xacro:macro name="plato_hand" params="ns:='plato'">
-    <link name="${ns}_base_link"></link>
-    <joint name="${ns}_base_link_to_palm" type="fixed">
-        <parent link="${ns}_base_link"/>
-        <child link="${ns}_palm" />
+    <link name="plato_base_link"></link>
+    <joint name="plato_base_link_to_palm" type="fixed">
+        <parent link="plato_base_link"/>
+        <child link="plato_palm" />
         <origin rpy="0.0 0 0" xyz="0 0 0"/>
     </joint>
-    <link name="${ns}_palm">
+    <link name="plato_palm">
         <visual>
         <origin xyz="0 0 0" rpy="0 -0 0" />
@@ -31,5 +30,5 @@
     </link>
     <!-- Finger 1 (Thumb) -->
-        <link name="${ns}_f1_proxbracket">
+        <link name="plato_f1_proxbracket">
             <visual>
             <origin xyz="0 0 0" rpy="0 -0 0" />
@@ -53,5 +52,5 @@
             </inertial>
         </link>
-        <link name="${ns}_f1_prox">
+        <link name="plato_f1_prox">
             <visual>
             <origin xyz="0 0 0" rpy="0 -0 0" />
@@ -75,5 +74,5 @@
             </inertial>
         </link>
-        <link name="${ns}_f1_mid">
+        <link name="plato_f1_mid">
             <visual>
             <origin xyz="0 0 0" rpy="0 -0 0" />
@@ -97,37 +96,37 @@
             </inertial>
         </link>
-        <link name="${ns}_f1_ee_frame">
-        </link>
-        <joint name="${ns}_f1_pip_pitch" type="revolute">
+        <link name="plato_f1_ee_frame">
+        </link>
+        <joint name="plato_f1_pip_pitch" type="revolute">
             <origin xyz="0.048000000000000028755 6.9388939039072283776e-18 -0.0026999999999999871325" rpy="6.6672023420374162248e-16 1.5291665303066472343e-16 3.3306690741059185714e-16" />
-            <parent link="${ns}_f1_prox" />
-            <child link="${ns}_f1_mid" />
+            <parent link="plato_f1_prox" />
+            <child link="plato_f1_mid" />
             <axis xyz="0 0 1"/>
             <limit effort="1" velocity="20" lower="-2.0944" upper="2.0944"/>
             <joint_properties friction="0.0"/>
         </joint>
-        <joint name="${ns}_f1_mcp_pitch" type="revolute">
+        <joint name="plato_f1_mcp_pitch" type="revolute">
             <origin xyz="-0.0049999999999999697464 -0.028150000000000133249 -0.0098999999999999366285" rpy="-2.8657554781383847745e-16 -1.5707963267948961139 0" />
-            <parent link="${ns}_f1_proxbracket" />
-            <child link="${ns}_f1_prox" />
+            <parent link="plato_f1_proxbracket" />
+            <child link="plato_f1_prox" />
             <axis xyz="0 0 1"/>
             <limit effort="1" velocity="20" lower="-2.0943951023931952626" upper="0.52359877559829881566"/>
             <joint_properties friction="0.0"/>
         </joint>
-        <joint name="${ns}_f1_mcp_roll" type="revolute">
+        <joint name="plato_f1_mcp_roll" type="revolute">
             <origin xyz="0.084500000000000047296 0.029999999999999988481 -0.033000000000000008493" rpy="1.5707963267948958919 -2.5535129566378612263e-15 1.5707963267948938935" />
-            <parent link="${ns}_palm" />
-            <child link="${ns}_f1_proxbracket" />
+            <parent link="plato_palm" />
+            <child link="plato_f1_proxbracket" />
             <axis xyz="0 0 1"/>
             <limit effort="1" velocity="20" lower="-0.52359877559829881566" upper="1.0471975511965976313"/>
             <joint_properties friction="0.0"/>
         </joint>
-        <joint name="${ns}_f1_ee_joint" type="fixed">
+        <joint name="plato_f1_ee_joint" type="fixed">
             <origin xyz="0.05060 0.0 0.0" rpy="-1.5707 0.0 0.0"/>
-            <parent link="${ns}_f1_mid"/>
-            <child link="${ns}_f1_ee_frame"/>
+            <parent link="plato_f1_mid"/>
+            <child link="plato_f1_ee_frame"/>
         </joint>
     <!-- Finger 2 (Index) -->
-        <link name="${ns}_f2_proxbracket">
+        <link name="plato_f2_proxbracket">
             <visual>
             <origin xyz="0 0 0" rpy="0 -0 0" />
@@ -151,5 +150,5 @@
             </inertial>
         </link>
-        <link name="${ns}_f2_prox">
+        <link name="plato_f2_prox">
             <visual>
             <origin xyz="0 0 0" rpy="0 -0 0" />
@@ -173,5 +172,5 @@
             </inertial>
         </link>
-        <link name="${ns}_f2_mid">
+        <link name="plato_f2_mid">
             <visual>
             <origin xyz="0 0 0" rpy="0 -0 0" />
@@ -195,37 +194,37 @@
             </inertial>
         </link>
-        <link name="${ns}_f2_ee_frame">
-        </link>
-        <joint name="${ns}_f2_pip_pitch" type="revolute">
+        <link name="plato_f2_ee_frame">
+        </link>
+        <joint name="plato_f2_pip_pitch" type="revolute">
             <origin xyz="0.047999999999999792832 0 0.0047999999999999813649" rpy="8.673617379890070258e-17 5.7824115865889863811e-17 -1.5021026917775434348e-15" />
-            <parent link="${ns}_f2_prox" />
-            <child link="${ns}_f2_mid" />
+            <parent link="plato_f2_prox" />
+            <child link="plato_f2_mid" />
             <axis xyz="0 0 1"/>
             <limit effort="1" velocity="20" lower="-2.0944" upper="2.0944"/>
             <joint_properties friction="0.0"/>
         </joint>
-        <joint name="${ns}_f2_mcp_pitch" type="revolute">
+        <joint name="plato_f2_mcp_pitch" type="revolute">
             <origin xyz="-0.0024999999999990307753 -0.028150000000000355294 -0.0099000000000003564316" rpy="-1.570796326794896558 6.9017807609091964755e-16 -1.5707963267948907848" />
-            <parent link="${ns}_f2_proxbracket" />
-            <child link="${ns}_f2_prox" />
+            <parent link="plato_f2_proxbracket" />
+            <child link="plato_f2_prox" />
             <axis xyz="0 0 1"/>
             <limit effort="1" velocity="20" lower="-1.570796326794896558" upper="0.785398163397448279"/>
             <joint_properties friction="0.0"/>
         </joint>
-        <joint name="${ns}_f2_mcp_yaw" type="revolute">
+        <joint name="plato_f2_mcp_yaw" type="revolute">
             <origin xyz="0.1000000000000001027 0.029999999999999974604 -0.015000000000000013323" rpy="3.141592653589793116 -1.1714553645825245089e-15 -1.5707963267948998887" />
-            <parent link="${ns}_palm" />
-            <child link="${ns}_f2_proxbracket" />
+            <parent link="plato_palm" />
+            <child link="plato_f2_proxbracket" />
             <axis xyz="0 0 1"/>
             <limit effort="1" velocity="20" lower="-1.570796326794896558" upper="0.26179938779914940783"/>
             <joint_properties friction="0.0"/>
         </joint>
-        <joint name="${ns}_f2_ee_joint" type="fixed">
+        <joint name="plato_f2_ee_joint" type="fixed">
             <origin xyz="0.05060 0.0 0.0" rpy="-1.5707 0.0 0.0"/>
-            <parent link="${ns}_f2_mid"/>
-            <child link="${ns}_f2_ee_frame"/>
+            <parent link="plato_f2_mid"/>
+            <child link="plato_f2_ee_frame"/>
         </joint>
     <!-- Finger 3: Middle -->
-        <link name="${ns}_f3_proxbracket">
+        <link name="plato_f3_proxbracket">
             <visual>
             <origin xyz="0 0 0" rpy="0 -0 0" />
@@ -249,5 +248,5 @@
             </inertial>
         </link>
-        <link name="${ns}_f3_prox">
+        <link name="plato_f3_prox">
             <visual>
             <origin xyz="0 0 0" rpy="0 -0 0" />
@@ -271,5 +270,5 @@
             </inertial>
         </link>
-        <link name="${ns}_f3_mid">
+        <link name="plato_f3_mid">
             <visual>
             <origin xyz="0 0 0" rpy="0 -0 0" />
@@ -293,35 +292,34 @@
             </inertial>
         </link>
-        <link name="${ns}_f3_ee_frame">
-        </link>
-        <joint name="${ns}_f3_pip_pitch" type="revolute">
+        <link name="plato_f3_ee_frame">
+        </link>
+        <joint name="plato_f3_pip_pitch" type="revolute">
             <origin xyz="0.047999999999998654854 2.0122792321330962295e-16 0.0047999999999999917732" rpy="-1.9081958235950694314e-16 5.7824115816011125546e-17 1.7763568393717672612e-15" />
-            <parent link="${ns}_f3_prox" />
-            <child link="${ns}_f3_mid" />
+            <parent link="plato_f3_prox" />
+            <child link="plato_f3_mid" />
             <axis xyz="0 0 1"/>
             <limit effort="1" velocity="20" lower="-2.0944" upper="2.0944"/>
             <joint_properties friction="0.0"/>
         </joint>
-        <joint name="${ns}_f3_mcp_pitch" type="revolute">
+        <joint name="plato_f3_mcp_pitch" type="revolute">
             <origin xyz="-0.002500000000000099365 -0.028150000000000077738 -0.0099000000000001291828" rpy="-1.570796326794896558 -3.7816971775725042188e-15 -1.5707963267948943376" />
-            <parent link="${ns}_f3_proxbracket" />
-            <child link="${ns}_f3_prox" />
+            <parent link="plato_f3_proxbracket" />
+            <child link="plato_f3_prox" />
             <axis xyz="0 0 1"/>
             <limit effort="1" velocity="20" lower="-1.570796326794896558" upper="0.785398163397448279"/>
             <joint_properties friction="0.0"/>
         </joint>
-        <joint name="${ns}_f3_mcp_yaw" type="revolute">
+        <joint name="plato_f3_mcp_yaw" type="revolute">
             <origin xyz="0.10000000000000000555 -0.029999999999999964195 -0.015000000000000048017" rpy="-3.1415926535897926719 1.1057720720235713428e-16 -1.5707963267948983344" />
-            <parent link="${ns}_palm" />
-            <child link="${ns}_f3_proxbracket" />
+            <parent link="plato_palm" />
+            <child link="plato_f3_proxbracket" />
             <axis xyz="0 0 1"/>
             <limit effort="1" velocity="20" lower="-0.26179938779914940783" upper="0.785398163397448279"/>
             <joint_properties friction="0.0"/>
         </joint>
-        <joint name="${ns}_f3_ee_joint" type="fixed">
+        <joint name="plato_f3_ee_joint" type="fixed">
             <origin xyz="0.05060 0.0 0.0" rpy="-1.5707 0.0 0.0"/>
-            <parent link="${ns}_f3_mid"/>
-            <child link="${ns}_f3_ee_frame"/>
-        </joint>
-    </xacro:macro>
+            <parent link="plato_f3_mid"/>
+            <child link="plato_f3_ee_frame"/>
+        </joint>
 </robot>

Commit message: hand_moveit_works wo ee

File: optimo_description/urdf/optimo.urdf.xacro (robot description, xacro)
@@ -1,12 +1,6 @@
 <?xml version="1.0"?>
 <robot name="optimo" xmlns:xacro="http://www.ros.org/wiki/xacro">
-    <!-- Bring xacro files -->
-    <xacro:include filename="optimo_xacro/optimo_arm.xacro"/>
-    <link name="world"/>
-    <joint name="world_joint" type="fixed">
-        <parent link="world"/>
-        <child link="optimo_base_link"/>
-        <origin xyz="0 0 0" rpy="0 0 0"/>
-    </joint>
+    <!-- Include the URDF of the base -->
+    <xacro:include filename="optimo_xacro/optimo_arm.xacro" />
     <!-- Include Physics Parameters in Gazebo -->
     <xacro:include filename="optimo_xacro/optimo.gazebo.xacro" />

File: optimo_description/urdf/optimo_xacro/optimo.gazebo.xacro (robot description, xacro)
@@ -1,22 +1,17 @@
 <?xml version="1.0"?>
 <robot xmlns:xacro="http://www.ros.org/wiki/xacro">
-    <xacro:property name="PI" value="3.1415926535897931"/>
-    <xacro:property name="DtR" value=".01745329251"/>
-    <gazebo reference="base_link"/>
-    <gazebo reference="optimo_link0"/>
+    <!-- <material name="Grey">
+        <color rgba="0.8 0.8 0.8 1"/>
+    </material> -->
+    <gazebo reference="optimo_base_link">
+        <material>Gazebo/Grey</material>
+    </gazebo>
     <gazebo reference="optimo_link1"/>
-    <gazebo reference="optimo_link1_passive"/>
     <gazebo reference="optimo_link2"/>
-    <gazebo reference="optimo_link2_passive"/>
     <gazebo reference="optimo_link3"/>
-    <gazebo reference="optimo_link3_passive"/>
     <gazebo reference="optimo_link4"/>
-    <gazebo reference="optimo_link4_passive"/>
     <gazebo reference="optimo_link5"/>
-    <gazebo reference="optimo_link5_passive"/>
     <gazebo reference="optimo_link6"/>
-    <gazebo reference="optimo_link6_passive"/>
     <gazebo reference="optimo_link7"/>
-    <gazebo reference="optimo_link7_passive"/>
     <!-- Joint State Publisher -->
     <gazebo>

File: optimo_description/urdf/optimo_xacro/optimo_arm.xacro (robot description, xacro)
@@ -3,13 +3,4 @@
     <xacro:property name="PI" value="3.1415926535897931"/>
     <xacro:property name="DtR" value=".01745329251"/>
-    <xacro:property name="mass_link0" value="3.06357" />
-    <xacro:property name="mass_link1" value="2.34471" />
-    <xacro:property name="mass_link2" value="2.36414" />
-    <xacro:property name="mass_link3" value="2.38050" />
-    <xacro:property name="mass_link4" value="2.42754" />
-    <xacro:property name="mass_link5" value="3.49611" />
-    <xacro:property name="mass_link6" value="1.46736" />
-    <xacro:property name="mass_link7" value="0.45606" />
-    <xacro:property name="mass_link8" value="0.001" />
     <link name="optimo_base_link">
     </link>
@@ -205,25 +196,5 @@
         </inertial>
     </link>
-    <!-- <joint name='jN' type='revolute'>
-    <child>LINK NAME</child>
-    <parent>LINK NAME</parent>
-    <axis>
-        <xyz>AXIS OF ROTATION, IN JOINT FRAME</xyz>
-        <limit>
-        <lower>RADIANS FOR REVOLUTE/ METERS FOR PRISMATIC</lower>
-        <upper></upper>
-        <effort></effort>
-        <velocity></velocity>
-        </limit>
-        <dynamics>
-        <damping>VISCOUS DAMPING COEFFICIENT</damping>
-        <friction>PHYSICAL STATIC FRICTION</friction>
-        <spring_reference>SPRING REF POSITION FOR THIS JOINT AXIS</spring_reference>
-        <spring_stiffness>SPRING STIFFNESS FOR THIS JOINT AXIS</spring_stiffness>
-        </dynamics>
-        <use_parent_model_frame>1</use_parent_model_frame>
-    </axis>
-    </joint> -->
-    <!-- Joints -->
+    <!-- Robot Joints -->
     <joint name="optimo_joint1" type="revolute">
         <origin xyz="0 0 0" rpy="0 0 0"/>

File: plato_description/urdf/plato_hand.urdf.xacro (robot description, xacro)
@@ -3,6 +3,3 @@
     <!-- Include Plato Hand Xacro  -->
     <xacro:include filename="$(find plato_description)/urdf/plato_xacro/plato_hand.xacro"/>
-    <!-- Set Namespace for the PLATO Hand -->
-    <xacro:property name="hand_name" value="plato" />
-    <xacro:plato_hand ns = "${hand_name}"/>
 </robot>

File: plato_description/urdf/plato_manipulator.urdf.xacro (robot description, xacro)
@@ -20,4 +20,5 @@
     <!-- Include Gazebo Physics Parameters -->
     <xacro:include filename="$(find optimo_description)/urdf/optimo_xacro/optimo.gazebo.xacro"/>
+    <xacro:include filename="$(find plato_description)/urdf/plato_xacro/plato_hand.gazebo.xacro"/>
     <!-- Make sure to include the controllers after all joints are defined -->
     <!-- Optimo + Plato ros2_controller -->

File: plato_description/urdf/plato_xacro/plato_hand.xacro (robot description, xacro)
@@ -103,5 +103,5 @@
             <child link="plato_f1_mid" />
             <axis xyz="0 0 1"/>
-            <limit effort="1" velocity="20" lower="-2.0944" upper="2.0944"/>
+            <limit effort="0.04" velocity="5" lower="-2.0944" upper="2.0944"/>
             <joint_properties friction="0.0"/>
         </joint>
@@ -111,5 +111,5 @@
             <child link="plato_f1_prox" />
             <axis xyz="0 0 1"/>
-            <limit effort="1" velocity="20" lower="-2.0943951023931952626" upper="0.52359877559829881566"/>
+            <limit effort="0.04" velocity="5" lower="-2.0943951023931952626" upper="0.52359877559829881566"/>
             <joint_properties friction="0.0"/>
         </joint>
@@ -119,5 +119,5 @@
             <child link="plato_f1_proxbracket" />
             <axis xyz="0 0 1"/>
-            <limit effort="1" velocity="20" lower="-0.52359877559829881566" upper="1.0471975511965976313"/>
+            <limit effort="0.04" velocity="5" lower="-0.52359877559829881566" upper="1.0471975511965976313"/>
             <joint_properties friction="0.0"/>
         </joint>
@@ -201,5 +201,5 @@
             <child link="plato_f2_mid" />
             <axis xyz="0 0 1"/>
-            <limit effort="1" velocity="20" lower="-2.0944" upper="2.0944"/>
+            <limit effort="0.04" velocity="5" lower="-2.0944" upper="2.0944"/>
             <joint_properties friction="0.0"/>
         </joint>
@@ -209,5 +209,5 @@
             <child link="plato_f2_prox" />
             <axis xyz="0 0 1"/>
-            <limit effort="1" velocity="20" lower="-1.570796326794896558" upper="0.785398163397448279"/>
+            <limit effort="0.04" velocity="5" lower="-1.570796326794896558" upper="0.785398163397448279"/>
             <joint_properties friction="0.0"/>
         </joint>
@@ -217,5 +217,5 @@
             <child link="plato_f2_proxbracket" />
             <axis xyz="0 0 1"/>
-            <limit effort="1" velocity="20" lower="-1.570796326794896558" upper="0.26179938779914940783"/>
+            <limit effort="0.04" velocity="5" lower="-1.570796326794896558" upper="0.26179938779914940783"/>
             <joint_properties friction="0.0"/>
         </joint>
@@ -299,5 +299,5 @@
             <child link="plato_f3_mid" />
             <axis xyz="0 0 1"/>
-            <limit effort="1" velocity="20" lower="-2.0944" upper="2.0944"/>
+            <limit effort="0.04" velocity="5" lower="-2.0944" upper="2.0944"/>
             <joint_properties friction="0.0"/>
         </joint>
@@ -307,5 +307,5 @@
             <child link="plato_f3_prox" />
             <axis xyz="0 0 1"/>
-            <limit effort="1" velocity="20" lower="-1.570796326794896558" upper="0.785398163397448279"/>
+            <limit effort="0.04" velocity="5" lower="-1.570796326794896558" upper="0.785398163397448279"/>
             <joint_properties friction="0.0"/>
         </joint>
@@ -315,5 +315,5 @@
             <child link="plato_f3_proxbracket" />
             <axis xyz="0 0 1"/>
-            <limit effort="1" velocity="20" lower="-0.26179938779914940783" upper="0.785398163397448279"/>
+            <limit effort="0.04" velocity="5" lower="-0.26179938779914940783" upper="0.785398163397448279"/>
             <joint_properties friction="0.0"/>
         </joint>
