Commit message: optimo_arm xacro joint dynamics and damping added

File: optimo_description/urdf/optimo.urdf.xacro (robot description, xacro)
@@ -1,10 +1,5 @@
 <?xml version="1.0"?>
 <robot name="optimo" xmlns:xacro="http://www.ros.org/wiki/xacro">
-    <!-- Include the URDF of the base -->
+    <!-- Include the URDF of the robot arm -->
     <xacro:include filename="optimo_xacro/optimo_arm.xacro" />
-    <!-- Include Physics Parameters in Gazebo -->
-    <xacro:include filename="optimo_xacro/optimo.gazebo.xacro" />
-    <!-- Include ros2_control -->
-    <xacro:include filename="optimo_xacro/optimo.control.xacro" />
-    <xacro:optimo_ros2_control name="OptimoGazebo"/>
 </robot>

File: optimo_description/urdf/optimo_xacro/optimo.xacro (robot description, xacro)
@@ -337,5 +337,5 @@
         <plugin filename="ign_ros2_control-system" name="ign_ros2_control::IgnitionROS2ControlPlugin">
             <!-- need to make $(find optimo_sim) work again...-->
-            <parameters>$(find optimo_sim)/config/control.yaml</parameters>
+            <parameters>$(find plato_bringup)/config/optimo_effort_controllers.yaml</parameters>
         </plugin>
         <plugin filename="MechanicalStop" name="optimo::MechanicalStop">

File: optimo_description/urdf/optimo_xacro/optimo_arm.xacro (robot description, xacro)
@@ -1,6 +1,15 @@
 <?xml version="1.0"?>
 <robot xmlns:xacro="http://www.ros.org/wiki/xacro">
+    <!-- PI Parameters -->
     <xacro:property name="PI" value="3.1415926535897931"/>
     <xacro:property name="DtR" value=".01745329251"/>
+    <!-- Color Parameters -->
+    <material name="white">
+        <color rgba="1.0 1.0 1.0 1.0"/>
+    </material>
+    <material name="blue">
+        <color rgba="0.5 0.5 1 1.0"/>
+    </material>
+    <!-- Optimo Robot Arm Links -->
     <link name="optimo_base_link">
     </link>
@@ -10,5 +19,4 @@
         <origin xyz="0 0 0.27" rpy="0 0 0"/>
     </joint>
-    <!-- Robot Links -->
     <link name="optimo_link0">
         <visual>
@@ -16,7 +24,5 @@
                 <mesh filename="file://$(find optimo_description)/meshes/link0.stl"/>
             </geometry>
-            <material name="LightGrey">
-                <color rgba="0.999 0.999 0.999 1.0"/>
-            </material>
+            <material name="blue"/>
         </visual>
         <collision>
@@ -31,14 +37,5 @@
         </inertial>
     </link>
-    <link name="optimo_link1">
-        <visual>
-            <geometry>
-                <sphere radius="0.01"/>
-            </geometry>
-            <material name="LightGrey">
-                <color rgba="0.999 0.999 0.999 1.0"/>
-            </material>
-        </visual>
-    </link>
+    <link name="optimo_link1"/>
     <link name="optimo_link1_passive">
         <visual>
@@ -46,7 +43,5 @@
                 <mesh filename="file://$(find optimo_description)/meshes/link1.stl"/>
             </geometry>
-            <material name="LightGrey">
-                <color rgba="0.999 0.999 0.999 1.0"/>
-            </material>
+            <material name="white">
         </visual>
         <collision>
@@ -68,7 +63,5 @@
                 <mesh filename="file://$(find optimo_description)/meshes/link2.stl"/>
             </geometry>
-            <material name="LightGrey">
-                <color rgba="0.999 0.999 0.999 1.0"/>
-            </material>
+            <material name="blue"/>
         </visual>
         <collision>
@@ -90,7 +83,5 @@
                 <mesh filename="file://$(find optimo_description)/meshes/link3.stl"/>
             </geometry>
-            <material name="LightGrey">
-                <color rgba="0.999 0.999 0.999 1.0"/>
-            </material>
+            <material name="white"/>
         </visual>
         <collision>
@@ -113,7 +104,5 @@
                 <mesh filename="file://$(find optimo_description)/meshes/link4.stl"/>
             </geometry>
-            <material name="LightGrey">
-                <color rgba="0.999 0.999 0.999 1.0"/>
-            </material>
+            <material name="blue"/>
         </visual>
         <collision>
@@ -136,7 +125,5 @@
                 <mesh filename="file://$(find optimo_description)/meshes/link5.stl"/>
             </geometry>
-            <material name="LightGrey">
-                <color rgba="0.999 0.999 0.999 1.0"/>
-            </material>
+            <material name="white"/>
         </visual>
         <collision>
@@ -158,7 +145,5 @@
                 <mesh filename="file://$(find optimo_description)/meshes/link6.stl"/>
             </geometry>
-            <material name="LightGrey">
-                <color rgba="0.999 0.999 0.999 1.0"/>
-            </material>
+            <material name="blue"/>
         </visual>
         <collision>
@@ -180,7 +165,5 @@
                 <mesh filename="file://$(find optimo_description)/meshes/link7.stl"/>
             </geometry>
-            <material name="LightGrey">
-                <color rgba="0.999 0.999 0.999 1.0"/>
-            </material>
+            <material name="white"/>
         </visual>
         <collision>
@@ -196,5 +179,5 @@
         </inertial>
     </link>
-    <!-- Robot Joints -->
+    <!-- Optimo Robot Joints -->
     <joint name="optimo_joint1" type="revolute">
         <origin xyz="0 0 0" rpy="0 0 0"/>
@@ -203,4 +186,5 @@
         <axis xyz="0 0 1"/>
         <limit lower="${DtR*-164}" upper="${DtR*167}" effort="79" velocity="10"/>
+        <dynamics damping="1" friction="0.1"/>
     </joint>
     <joint name="optimo_joint1_passive" type="fixed">
@@ -215,4 +199,5 @@
         <axis xyz="0 0 1"/>
         <limit lower="${DtR*60}" upper="${DtR*250}" effort="95" velocity="10"/>
+        <dynamics damping="1" friction="0.1"/>
     </joint>
     <joint name="optimo_joint2_passive" type="fixed">
@@ -227,4 +212,5 @@
         <axis xyz="0 0 1"/>
         <limit lower="${DtR*-167}" upper="${DtR*163}" effort="32" velocity="10"/>
+        <dynamics damping="1" friction="0.1"/>
     </joint>
     <joint name="optimo_joint3_passive" type="fixed">
@@ -239,4 +225,5 @@
         <axis xyz="0 0 1"/>
         <limit lower="${DtR*-145}" upper="${DtR*145}" effort="40" velocity="10"/>
+        <dynamics damping="1" friction="0.1"/>
     </joint>
     <joint name="optimo_joint4_passive" type="fixed">
@@ -251,4 +238,5 @@
         <axis xyz="0 0 1"/>
         <limit lower="${DtR*-170}" upper="${DtR*170}" effort="15" velocity="10"/>
+        <dynamics damping="1" friction="0.1"/>
     </joint>
     <joint name="optimo_joint5_passive" type="fixed">
@@ -263,4 +251,5 @@
         <axis xyz="0 0 1"/>
         <limit lower="${DtR*-120}" upper="${DtR*120}" effort="15" velocity="10"/>
+        <dynamics damping="1" friction="0.1"/>
     </joint>
     <joint name="optimo_joint6_passive" type="fixed">
@@ -275,4 +264,5 @@
         <axis xyz="0 0 1"/>
         <limit lower="${DtR*-152}" upper="${DtR*188}" effort="15" velocity="10"/>
+        <dynamics damping="1" friction="0.1"/>
     </joint>
     <joint name="optimo_joint7_passive" type="fixed">

Commit message: optimo urdf using xacro def and pedestal

File: optimo_description/urdf/optimo.urdf.xacro (robot description, xacro)
@@ -1,7 +1,14 @@
 <?xml version="1.0"?>
 <robot name="optimo" xmlns:xacro="http://www.ros.org/wiki/xacro">
-    <!-- Include the URDF of the robot arm -->
-    <xacro:include filename="optimo_xacro/optimo_arm.xacro" />
+    <!-- Include the Xacro files -->
+    <xacro:include filename="optimo_xacro/optimo_description.xacro" />
+    <xacro:include filename="optimo_xacro/pedestal.xacro" />
     <!-- Include gz configuration -->
     <!-- <xacro:include filename="optimo_xacro/optimo.gz.xacro" /> -->
+    <!-- World Link -->
+    <link name="world"/>
+    <!-- Pedestal -->
+    <xacro:pedestal connector_link="world" />
+    <!-- Optimo Arm -->
+    <xacro:optimo_description connector_link="stand_link"/>
 </robot>
