Commit message: plato description package separated from Optimo

File: optimo_description/urdf/optimo_property/optimo.control.xacro (robot description, xacro)
@@ -1,3 +1,5 @@
-<gazebo>
+<?xml version="1.0"?>
+<robot xmlns:xacro="http://www.ros.org/wiki/xacro">
+    <gazebo>
         <plugin filename="libgazebo_ros2_control.so" name="gazebo_ros2_control">
             <parameters>$(find plato_gazebo)/config/optimo_controller.yaml</parameters>
@@ -85,2 +87,3 @@
         </joint>
     </ros2_control>
+</robot>

File: optimo_description/urdf/optimo_property/optimo.gazebo.xacro (robot description, xacro)
@@ -32,3 +32,5 @@
         </plugin>
     </gazebo>
+    <!-- SEA Spring-Damper -->
+    <!-- <gazebo -->
 </robot>

File: plato_description/urdf/plato_property/plato_hand.xacro (robot description, xacro)
@@ -11,5 +11,5 @@
 <origin xyz="0 0 0" rpy="0 -0 0" />
 <geometry>
-<mesh filename="file://$(find optimo_description)/meshes/plato/base_visual.stl"/>
+<mesh filename="file://$(find plato_description)/meshes/plato/base_visual.stl"/>
 </geometry>
 <material name="base_material">
@@ -20,5 +20,5 @@
 <origin xyz="0 0 0" rpy="0 -0 0" />
 <geometry>
-<mesh filename="file://$(find optimo_description)/meshes/plato/base_collision.stl"/>
+<mesh filename="file://$(find plato_description)/meshes/plato/base_collision.stl"/>
 </geometry>
 </collision>
@@ -34,5 +34,5 @@
     <origin xyz="0 0 0" rpy="0 -0 0" />
     <geometry>
-    <mesh filename="file://$(find optimo_description)/meshes/plato/proxbracket_visual.stl"/>
+    <mesh filename="file://$(find plato_description)/meshes/plato/proxbracket_visual.stl"/>
     </geometry>
     <material name="proxbracket_material">
@@ -43,5 +43,5 @@
     <origin xyz="0 0 0" rpy="0 -0 0" />
     <geometry>
-    <mesh filename="file://$(find optimo_description)/meshes/plato/proxbracket_collision.stl"/>
+    <mesh filename="file://$(find plato_description)/meshes/plato/proxbracket_collision.stl"/>
     </geometry>
     </collision>
@@ -56,5 +56,5 @@
     <origin xyz="0 0 0" rpy="0 -0 0" />
     <geometry>
-    <mesh filename="file://$(find optimo_description)/meshes/plato/prox_visual.stl"/>
+    <mesh filename="file://$(find plato_description)/meshes/plato/prox_visual.stl"/>
     </geometry>
     <material name="prox_material">
@@ -65,5 +65,5 @@
     <origin xyz="0 0 0" rpy="0 -0 0" />
     <geometry>
-    <mesh filename="file://$(find optimo_description)/meshes/plato/prox_collision.stl"/>
+    <mesh filename="file://$(find plato_description)/meshes/plato/prox_collision.stl"/>
     </geometry>
     </collision>
@@ -78,5 +78,5 @@
     <origin xyz="0 0 0" rpy="0 -0 0" />
     <geometry>
-    <mesh filename="file://$(find optimo_description)/meshes/plato/mid_visual.stl"/>
+    <mesh filename="file://$(find plato_description)/meshes/plato/mid_visual.stl"/>
     </geometry>
     <material name="mid_material">
@@ -87,5 +87,5 @@
     <origin xyz="0 0 0" rpy="0 -0 0" />
     <geometry>
-    <mesh filename="file://$(find optimo_description)/meshes/plato/mid_collision.stl"/>
+    <mesh filename="file://$(find plato_description)/meshes/plato/mid_collision.stl"/>
     </geometry>
     </collision>
@@ -132,5 +132,5 @@
     <origin xyz="0 0 0" rpy="0 -0 0" />
     <geometry>
-    <mesh filename="file://$(find optimo_description)/meshes/plato/proxbracket_2_visual.stl"/>
+    <mesh filename="file://$(find plato_description)/meshes/plato/proxbracket_2_visual.stl"/>
     </geometry>
     <material name="proxbracket_2_material">
@@ -141,5 +141,5 @@
     <origin xyz="0 0 0" rpy="0 -0 0" />
     <geometry>
-    <mesh filename="file://$(find optimo_description)/meshes/plato/proxbracket_2_collision.stl"/>
+    <mesh filename="file://$(find plato_description)/meshes/plato/proxbracket_2_collision.stl"/>
     </geometry>
     </collision>
@@ -154,5 +154,5 @@
     <origin xyz="0 0 0" rpy="0 -0 0" />
     <geometry>
-    <mesh filename="file://$(find optimo_description)/meshes/plato/prox_2_visual.stl"/>
+    <mesh filename="file://$(find plato_description)/meshes/plato/prox_2_visual.stl"/>
     </geometry>
     <material name="prox_2_material">
@@ -163,5 +163,5 @@
     <origin xyz="0 0 0" rpy="0 -0 0" />
     <geometry>
-    <mesh filename="file://$(find optimo_description)/meshes/plato/prox_2_collision.stl"/>
+    <mesh filename="file://$(find plato_description)/meshes/plato/prox_2_collision.stl"/>
     </geometry>
     </collision>
@@ -176,5 +176,5 @@
     <origin xyz="0 0 0" rpy="0 -0 0" />
     <geometry>
-    <mesh filename="file://$(find optimo_description)/meshes/plato/mid_2_visual.stl"/>
+    <mesh filename="file://$(find plato_description)/meshes/plato/mid_2_visual.stl"/>
     </geometry>
     <material name="mid_2_material">
@@ -185,5 +185,5 @@
     <origin xyz="0 0 0" rpy="0 -0 0" />
     <geometry>
-    <mesh filename="file://$(find optimo_description)/meshes/plato/mid_2_collision.stl"/>
+    <mesh filename="file://$(find plato_description)/meshes/plato/mid_2_collision.stl"/>
     </geometry>
     </collision>
@@ -230,5 +230,5 @@
     <origin xyz="0 0 0" rpy="0 -0 0" />
     <geometry>
-    <mesh filename="file://$(find optimo_description)/meshes/plato/proxbracket_3_visual.stl"/>
+    <mesh filename="file://$(find plato_description)/meshes/plato/proxbracket_3_visual.stl"/>
     </geometry>
     <material name="proxbracket_3_material">
@@ -239,5 +239,5 @@
     <origin xyz="0 0 0" rpy="0 -0 0" />
     <geometry>
-    <mesh filename="file://$(find optimo_description)/meshes/plato/proxbracket_3_collision.stl"/>
+    <mesh filename="file://$(find plato_description)/meshes/plato/proxbracket_3_collision.stl"/>
     </geometry>
     </collision>
@@ -252,5 +252,5 @@
         <origin xyz="0 0 0" rpy="0 -0 0" />
         <geometry>
-        <mesh filename="file://$(find optimo_description)/meshes/plato/prox_3_visual.stl"/>
+        <mesh filename="file://$(find plato_description)/meshes/plato/prox_3_visual.stl"/>
         </geometry>
         <material name="prox_3_material">
@@ -261,5 +261,5 @@
         <origin xyz="0 0 0" rpy="0 -0 0" />
         <geometry>
-        <mesh filename="file://$(find optimo_description)/meshes/plato/prox_3_collision.stl"/>
+        <mesh filename="file://$(find plato_description)/meshes/plato/prox_3_collision.stl"/>
         </geometry>
         </collision>
@@ -274,5 +274,5 @@
         <origin xyz="0 0 0" rpy="0 -0 0" />
         <geometry>
-        <mesh filename="file://$(find optimo_description)/meshes/plato/mid_3_visual.stl"/>
+        <mesh filename="file://$(find plato_description)/meshes/plato/mid_3_visual.stl"/>
         </geometry>
         <material name="mid_3_material">
@@ -283,5 +283,5 @@
         <origin xyz="0 0 0" rpy="0 -0 0" />
         <geometry>
-        <mesh filename="file://$(find optimo_description)/meshes/plato/mid_3_collision.stl"/>
+        <mesh filename="file://$(find plato_description)/meshes/plato/mid_3_collision.stl"/>
         </geometry>
         </collision>
