Commit message: trying to add ns for controllers

File: optimo_description/urdf/optimo_xacro/optimo.control.xacro (robot description, xacro)
@@ -22,9 +22,9 @@
             </xacro:macro>
             <xacro:configure_joint joint_name="${ns}_joint1" initial_position="0.0"/>
-            <xacro:configure_joint joint_name="${ns}_joint2" initial_position="3.14"/>
+            <xacro:configure_joint joint_name="${ns}_joint2" initial_position="${160*DtR}"/>
             <xacro:configure_joint joint_name="${ns}_joint3" initial_position="0.0"/>
-            <xacro:configure_joint joint_name="${ns}_joint4" initial_position="0.0"/>
+            <xacro:configure_joint joint_name="${ns}_joint4" initial_position="${-60*DtR}"/>
             <xacro:configure_joint joint_name="${ns}_joint5" initial_position="0.0"/>
-            <xacro:configure_joint joint_name="${ns}_joint6" initial_position="0.0"/>
+            <xacro:configure_joint joint_name="${ns}_joint6" initial_position="${-30*DtR}"/>
             <xacro:configure_joint joint_name="${ns}_joint7" initial_position="0.0"/>
         </ros2_control>

File: optimo_description/urdf/optimo_xacro/optimo_arm.xacro (robot description, xacro)
@@ -311,4 +311,4 @@
             <child link="${ns}_link7_passive"/>
         </joint>
-     </xacro:macro>
+    </xacro:macro>
 </robot>

File: plato_description/urdf/plato_manipulator.urdf.xacro (robot description, xacro)
@@ -1,13 +1,14 @@
 <?xml version="1.0"?>
 <robot name="plato" xmlns:xacro="http://www.ros.org/wiki/xacro">
+    <!-- Set Property -->
+    <xacro:property name="hand_ns" default="plato"/>
+    <xacro:property name="arm_ns" default="optimo"/>
     <!-- Include Optimo Arm and PLATO Hand Xacro -->
     <xacro:include filename="$(find optimo_description)/urdf/optimo_xacro/optimo_arm.xacro"/>
+        <xacro:optimo_arm ns = "${arm_ns}"/>
     <xacro:include filename="$(find plato_description)/urdf/plato_xacro/plato_hand.xacro"/>
-    <!-- Set Namespace for the Optimo Arm -->
-    <xacro:property name="arm_ns" value="optimo" />
-    <xacro:optimo_arm ns = "${arm_ns}"/>
-    <!-- Set Namespace for the PLATO Hand -->
-    <xacro:property name="hand_ns" value="plato" />
-    <xacro:plato_hand ns = "${hand_ns}"/>
+        <xacro:plato_hand ns = "${hand_ns}"/>
+    <!-- Include Gazebo Physics Parameters -->
+    <xacro:include filename="$(find optimo_description)/urdf/optimo_xacro/optimo.gazebo.xacro"/>
     <!-- Set World Frame for Gazebo -->
     <link name="world"/>
@@ -26,5 +27,7 @@
     <!-- Make sure to include the controllers after all joints are defined -->
     <!-- Optimo Gazebo Parameters and ros2_controller -->
-    <xacro:include filename="$(find optimo_description)/urdf/optimo_xacro/optimo.gazebo.xacro"/>
     <xacro:include filename="$(find optimo_description)/urdf/optimo_xacro/optimo.control.xacro"/>
+         <xacro:optimo_ros2_control ns="${arm_ns}"/>
+    <!-- <xacro:include filename="$(find plato_description)/urdf/plato_xacro/plato_hand.control.xacro"/> -->
+         <!-- <xacro:plato_ros2_control ns="${hand_ns}"/> -->
 </robot>
