Commit message: plato hand to xacro

File: optimo_description/urdf/optimo_xacro/optimo_description.xacro (robot description, xacro)
@@ -178,5 +178,5 @@
         </inertial>
     </link>
-    <!-- Optimo Robot Joints -->
+    <!-- Optimo Arm Joints -->
     <joint name="optimo_joint1" type="revolute">
         <origin xyz="0 0 0" rpy="0 0 0"/>
@@ -270,4 +270,12 @@
         <child link="optimo_link7_passive"/>
     </joint>
+    <!-- End Effector -->
+    <link name="optimo_ee_link">
+    </link>
+    <joint name="optimo_ee_joint" type="fixed">
+        <parent link="optimo_link7_passive"/>
+        <child link="optimo_ee_link"/>
+        <origin xyz="0 0 0.15" rpy="0 -1.5707 3.14"/>
+    </joint>
 </xacro:macro>
 </robot>

File: optimo_description/urdf/optimo_xacro/pedestal.xacro (robot description, xacro)
@@ -1,4 +1,4 @@
 <?xml version="1.0"?>
-<robot name="optimo" xmlns:xacro="http://www.ros.org/wiki/xacro">
+<robot xmlns:xacro="http://www.ros.org/wiki/xacro">
 <xacro:macro name="pedestal" params="connector_link">
     <link name="stand_link">

File: plato_description/urdf/plato_hand.urdf.xacro (robot description, xacro)
@@ -1,5 +1,9 @@
 <?xml version="1.0"?>
-<robot name="plato" xmlns:xacro="http://www.ros.org/wiki/xacro">
-    <!-- Include Plato Hand Xacro  -->
-    <xacro:include filename="$(find plato_description)/urdf/plato_xacro/plato_hand.xacro"/>
+<robot name="plato_hand" xmlns:xacro="http://www.ros.org/wiki/xacro">
+    <!-- Set World Frame -->
+    <link name="world"/>
+    <!-- Include Xacro -->
+    <xacro:include filename="$(find plato_description)/urdf/plato_xacro/plato_hand_description.xacro"/>
+    <!-- Plato Hand -->
+    <xacro:plato_description connector_link="world"/>
 </robot>

File: plato_description/urdf/plato_manipulator.urdf.xacro (robot description, xacro)
@@ -1,19 +1,15 @@
 <?xml version="1.0"?>
-<robot name="plato" xmlns:xacro="http://www.ros.org/wiki/xacro">
+<robot name="plato_manipulator" xmlns:xacro="http://www.ros.org/wiki/xacro">
     <!-- Set World Frame -->
     <link name="world"/>
-    <!-- Include Optimo Arm and PLATO Hand Xacro -->
+    <!-- Include Xacro -->
     <xacro:include filename="$(find optimo_description)/urdf/optimo_xacro/pedestal.xacro" />
     <xacro:include filename="$(find optimo_description)/urdf/optimo_xacro/optimo_description.xacro"/>
-    <xacro:include filename="$(find plato_description)/urdf/plato_xacro/plato_hand.xacro"/>
+    <xacro:include filename="$(find plato_description)/urdf/plato_xacro/plato_hand_description.xacro"/>
     <!-- Pedestal -->
     <xacro:pedestal connector_link="world" />
     <!-- Optimo Arm -->
     <xacro:optimo_description connector_link="stand_link"/>
-    <!-- Connect PLATO Hand to Optimo Arm -->
-    <joint name="hand_arm_joint" type="fixed">
-        <parent link="optimo_link7_passive"/>
-        <child link="plato_base_link"/>
-        <origin xyz="0 0 0.15" rpy="0 -1.5707 3.14"/>
-    </joint>
+    <!-- Plato Hand -->
+    <xacro:plato_description connector_link="optimo_ee_link"/>
 </robot>

File: plato_description/urdf/plato_xacro/plato_hand_description.xacro (robot description, xacro)
@@ -1,3 +1,11 @@
-<robot name="plato">
+<?xml version="1.0"?>
+<robot xmlns:xacro="http://www.ros.org/wiki/xacro">
+<xacro:macro name="plato_description" params="connector_link">
+    <!-- Connector Joint -->
+    <joint name="plato_connector_joint" type="fixed">
+        <parent link="${connector_link}"/>
+        <child link="plato_base_link"/>
+        <origin xyz="0 0 0" rpy="0 0 0"/>
+    </joint>
     <!-- Base Link -->
     <link name="plato_base_link">
@@ -315,3 +323,4 @@
         <joint_properties friction="0.0"/>
     </joint>
+</xacro:macro>
 </robot>
