Commit message: pedetal xacro name to pedestal_description

File: optimo_description/urdf/optimo_xacro/pedestal.xacro (robot description, xacro)
@@ -1,5 +1,5 @@
 <?xml version="1.0"?>
 <robot xmlns:xacro="http://www.ros.org/wiki/xacro">
-<xacro:macro name="pedestal" params="connector_link">
+<xacro:macro name="pedestal_description" params="connector_link">
     <link name="stand_link">
         <visual>

File: plato_description/urdf/plato_manipulator.urdf.xacro (robot description, xacro)
@@ -8,5 +8,5 @@
     <xacro:include filename="$(find plato_description)/urdf/plato_xacro/plato_hand_description.xacro"/>
     <!-- Pedestal -->
-    <xacro:pedestal connector_link="world" />
+    <xacro:pedestal_description connector_link="world" />
     <!-- Optimo Arm -->
     <xacro:optimo_description connector_link="stand_link"/>
