Commit message: panda_moveit_config deleted

File: plato_moveit_config/config/plato.ros2_control.xacro (robot description, xacro)
@@ -1,16 +1,24 @@
 <?xml version="1.0"?>
 <robot xmlns:xacro="http://www.ros.org/wiki/xacro">
-    <xacro:macro name="plato_ros2_control" params="name initial_positions_file">
+    <xacro:macro name="plato_ros2_control" params="name initial_positions_file sim_type">
         <xacro:property name="initial_positions" value="${load_yaml(initial_positions_file)['initial_positions']}"/>
-      <gazebo>
-          <plugin filename="libgazebo_ros2_control.so" name="gazebo_ros2_control">
-              <parameters>$(find plato_moveit_config)/config/ros2_controllers.yaml</parameters>
-          </plugin>
-      </gazebo>
+        <!-- if Simulation is in Gazebo Classic, use gazebo_ros2_control -->
+        <xacro:if value="${sim_type == 'gazebo'}">
+          <gazebo>
+              <plugin filename="libgazebo_ros2_control.so" name="gazebo_ros2_control">
+                  <parameters>$(find plato_moveit_config)/config/ros2_controllers.yaml</parameters>
+              </plugin>
+          </gazebo>
+        </xacro:if>
         <ros2_control name="${name}" type="system">
             <hardware>
-                <!-- By default, set up controllers for simulation. This won't work on real hardware -->
-                <!-- <plugin>mock_components/GenericSystem</plugin> -->
-                <plugin>gazebo_ros2_control/GazeboSystem</plugin>
+                <!-- Gazebo System -->
+                <xacro:if value="${sim_type == 'gazebo'}">
+                  <plugin>gazebo_ros2_control/GazeboSystem</plugin>
+                </xacro:if>
+                <!-- Fake System -->
+                <xacro:if value="${sim_type == 'fake'}">
+                  <plugin>fake_components/FakeSystem</plugin>
+                </xacro:if>
             </hardware>
             <joint name="optimo_joint1">

File: plato_moveit_config/config/plato.urdf.xacro (robot description, xacro)
@@ -1,9 +1,11 @@
 <?xml version="1.0"?>
 <robot xmlns:xacro="http://www.ros.org/wiki/xacro" name="plato">
+    <!-- Arguments -->
     <xacro:arg name="initial_positions_file" default="initial_positions.yaml" />
+    <xacro:arg name="sim_type" default="gazebo" /> <!-- gazebo | fake | TODO:isaac -->
     <!-- Import plato urdf file -->
     <xacro:include filename="$(find plato_description)/urdf/plato_manipulator.urdf" />
     <!-- Import control_xacro -->
     <xacro:include filename="plato.ros2_control.xacro" />
-    <xacro:plato_ros2_control name="FakeSystem" initial_positions_file="$(arg initial_positions_file)"/>
+    <xacro:plato_ros2_control name="SimSystem" initial_positions_file="$(arg initial_positions_file)" sim_type="$(arg sim_type)"/>
 </robot>

Commit message: gazebo moveit works with world fixed

File: plato_moveit_config/config/plato.ros2_control.xacro (robot description, xacro)
@@ -1,8 +1,8 @@
 <?xml version="1.0"?>
 <robot xmlns:xacro="http://www.ros.org/wiki/xacro">
-    <xacro:macro name="plato_ros2_control" params="name initial_positions_file sim_type">
+    <xacro:macro name="plato_ros2_control" params="name initial_positions_file hardware_type">
         <xacro:property name="initial_positions" value="${load_yaml(initial_positions_file)['initial_positions']}"/>
-        <!-- if Simulation is in Gazebo Classic, use gazebo_ros2_control -->
-        <xacro:if value="${sim_type == 'gazebo'}">
+        <!-- Gazebo ros2_control -->
+        <xacro:if value="${hardware_type == 'gazebo'}">
           <gazebo>
               <plugin filename="libgazebo_ros2_control.so" name="gazebo_ros2_control">
@@ -13,11 +13,9 @@
         <ros2_control name="${name}" type="system">
             <hardware>
-                <!-- Gazebo System -->
-                <xacro:if value="${sim_type == 'gazebo'}">
+                <xacro:if value="${hardware_type == 'gazebo'}">
                   <plugin>gazebo_ros2_control/GazeboSystem</plugin>
                 </xacro:if>
-                <!-- Fake System -->
-                <xacro:if value="${sim_type == 'fake'}">
-                  <plugin>fake_components/FakeSystem</plugin>
+                <xacro:if value="${hardware_type == 'mock'}">
+                  <plugin>mock_components/GenericSystem</plugin>
                 </xacro:if>
             </hardware>

File: plato_moveit_config/config/plato.urdf.xacro (robot description, xacro)
@@ -1,11 +1,17 @@
 <?xml version="1.0"?>
 <robot xmlns:xacro="http://www.ros.org/wiki/xacro" name="plato">
-    <!-- Arguments -->
     <xacro:arg name="initial_positions_file" default="initial_positions.yaml" />
-    <xacro:arg name="sim_type" default="gazebo" /> <!-- gazebo | fake | TODO:isaac -->
+    <xacro:arg name="hardware_type" default="gazebo" /> <!-- gazebo | mock -->
     <!-- Import plato urdf file -->
     <xacro:include filename="$(find plato_description)/urdf/plato_manipulator.urdf" />
     <!-- Import control_xacro -->
     <xacro:include filename="plato.ros2_control.xacro" />
-    <xacro:plato_ros2_control name="SimSystem" initial_positions_file="$(arg initial_positions_file)" sim_type="$(arg sim_type)"/>
+    <xacro:plato_ros2_control name="FakeSystem" initial_positions_file="$(arg initial_positions_file)" hardware_type="$(arg hardware_type)"/>
+    <!-- put world -->
+    <link name="world"/>
+    <joint name="world_joint" type="fixed">
+        <parent link="world"/>
+        <child link="optimo_base_link"/>
+        <origin xyz="0 0 0" rpy="0 0 0"/>
+    </joint>
 </robot>
