Commit message: effort adjsuted to 0.04 Nm

File: plato_description/urdf/plato_xacro/plato_hand.xacro (robot description, xacro)
@@ -102,5 +102,5 @@
         <child link="plato_f1_proxbracket" />
         <axis xyz="0 0 1"/>
-        <limit effort="1" velocity="20" lower="-0.52359877559829881566" upper="1.0471975511965976313"/>
+        <limit effort="0.04" velocity="20" lower="-0.52359877559829881566" upper="1.0471975511965976313"/>
         <joint_properties friction="0.0"/>
     </joint>
@@ -110,5 +110,5 @@
         <child link="plato_f1_prox" />
         <axis xyz="0 0 1"/>
-        <limit effort="1" velocity="20" lower="-1.570796326794896558" upper="0.52359877559829881566"/>
+        <limit effort="0.04" velocity="20" lower="-1.570796326794896558" upper="0.52359877559829881566"/>
         <joint_properties friction="0.0"/>
     </joint>
@@ -118,5 +118,5 @@
         <child link="plato_f1_mid" />
         <axis xyz="0 0 1"/>
-        <limit effort="1" velocity="20" lower="-2.0943951023931952626" upper="2.0943951023931952626"/>
+        <limit effort="0.04" velocity="20" lower="-2.0943951023931952626" upper="2.0943951023931952626"/>
         <joint_properties friction="0.0"/>
     </joint>
@@ -199,5 +199,5 @@
         <child link="plato_f2_proxbracket" />
         <axis xyz="0 0 1"/>
-        <limit effort="1" velocity="20" lower="-0.26179938779914940783" upper="0.26179938779914940783"/>
+        <limit effort="0.04" velocity="20" lower="-0.26179938779914940783" upper="0.26179938779914940783"/>
         <joint_properties friction="0.0"/>
     </joint>
@@ -207,5 +207,5 @@
         <child link="plato_f2_prox" />
         <axis xyz="0 0 1"/>
-        <limit effort="1" velocity="20" lower="-1.570796326794896558" upper="1.570796326794896558"/>
+        <limit effort="0.04" velocity="20" lower="-1.570796326794896558" upper="1.570796326794896558"/>
         <joint_properties friction="0.0"/>
     </joint>
@@ -215,5 +215,5 @@
         <child link="plato_f2_mid" />
         <axis xyz="0 0 1"/>
-        <limit effort="1" velocity="20" lower="-2.0943951023931952626" upper="2.0943951023931952626"/>
+        <limit effort="0.04" velocity="20" lower="-2.0943951023931952626" upper="2.0943951023931952626"/>
         <joint_properties friction="0.0"/>
     </joint>
@@ -296,5 +296,5 @@
         <child link="plato_f3_proxbracket" />
         <axis xyz="0 0 1"/>
-        <limit effort="1" velocity="20" lower="-0.26179938779914940783" upper="0.26179938779914940783"/>
+        <limit effort="0.04" velocity="20" lower="-0.26179938779914940783" upper="0.26179938779914940783"/>
         <joint_properties friction="0.0"/>
     </joint>
@@ -304,5 +304,5 @@
         <child link="plato_f3_prox" />
         <axis xyz="0 0 1"/>
-        <limit effort="1" velocity="20" lower="-1.570796326794896558" upper="1.570796326794896558"/>
+        <limit effort="0.04" velocity="20" lower="-1.570796326794896558" upper="1.570796326794896558"/>
         <joint_properties friction="0.0"/>
     </joint>
@@ -312,5 +312,5 @@
         <child link="plato_f3_mid" />
         <axis xyz="0 0 1"/>
-        <limit effort="1" velocity="20" lower="-2.0943951023931952626" upper="2.0943951023931952626"/>
+        <limit effort="0.04" velocity="20" lower="-2.0943951023931952626" upper="2.0943951023931952626"/>
         <joint_properties friction="0.0"/>
     </joint>
