Commit message: fixed wrist offset

File: plato_description/urdf/plato_xacro/plato_hand.xacro (robot description, xacro)
@@ -97,13 +97,13 @@
     </link>
     <joint name="plato_f1_pip_pitch" type="revolute">
-        <origin xyz="0.047999999999999293232 -9.7144514654701197287e-17 -0.0027000000000018120616" rpy="-2.1461177382147364842e-14 2.258685845680399537e-14 1.1702444568937959782e-14" />
+        <origin xyz="0.047999999999999279354 -9.7144514654701197287e-17 -0.0027000000000018120616" rpy="1.4288004010678779623e-14 5.8002972942348347565e-14 1.1102230245143881434e-16" />
         <parent link="plato_f1_prox" />
         <child link="plato_f1_mid" />
         <axis xyz="0 0 1"/>
-        <limit effort="1" velocity="20" lower="-1.570796326794896558" upper="0.34906585039886589561"/>
+        <limit effort="1" velocity="20" lower="-0.34906585039886589561" upper="1.570796326794896558"/>
         <joint_properties friction="0.0"/>
     </joint>
     <joint name="plato_f1_mcp_pitch" type="revolute">
-        <origin xyz="-0.0050000000000000009714 -0.028150000000000004879 -0.0098999999999999921396" rpy="-4.3545121968198811335e-28 -1.5707963267948379382 0" />
+        <origin xyz="-0.0050000000000000009714 -0.028149999999999997941 -0.0099000000000000198952" rpy="-4.3545121968198811335e-28 -1.5707963267948379382 0" />
         <parent link="plato_f1_proxbracket" />
         <child link="plato_f1_prox" />
@@ -113,5 +113,5 @@
     </joint>
     <joint name="plato_f1_mcp_roll" type="revolute">
-        <origin xyz="0.15070000000000047247 0.029000000000000043104 -0.031000000000000055289" rpy="1.5707963267948970021 -4.0301095793892904738e-14 1.57079632679489678" />
+        <origin xyz="0.084000000000000227263 0.029000000000000015349 -0.031000000000000034472" rpy="1.5707963267948970021 -4.0301095793892904738e-14 1.57079632679489678" />
         <parent link="palm_base" />
         <child link="plato_f1_proxbracket" />
@@ -194,5 +194,5 @@
     </link>
     <joint name="plato_f2_pip_pitch" type="revolute">
-        <origin xyz="0.047999999999998960165 -1.4627242559545061695e-16 -0.0029000000000008394063" rpy="8.6736173798921644372e-17 2.6809573080062448739e-14 -5.1904703123014745533e-17" />
+        <origin xyz="0.047999999999998960165 -1.2632310562171733537e-16 -0.0029000000000008498147" rpy="8.6736173798921644372e-17 2.6809573080062448739e-14 -5.1904703123014745533e-17" />
         <parent link="plato_f2_prox" />
         <child link="plato_f2_mid" />
@@ -202,5 +202,5 @@
     </joint>
     <joint name="plato_f2_mcp_pitch" type="revolute">
-        <origin xyz="-0.0049999999999999801548 0.028150000000000091616 -0.0098999999999997475436" rpy="-1.5707963267949098807 1.0921682003593975385e-14 1.5707963267949234254" />
+        <origin xyz="-0.0049999999999999801548 0.028150000000000105493 -0.0098999999999997492783" rpy="-1.5707963267949098807 1.0921682003593975385e-14 1.5707963267949234254" />
         <parent link="plato_f2_proxbracket" />
         <child link="plato_f2_prox" />
@@ -210,5 +210,5 @@
     </joint>
     <joint name="plato_f2_mcp_yaw" type="revolute">
-        <origin xyz="0.14970000000000047158 0.029000000000000046574 -0.01000000000000005225" rpy="-3.141592653589793116 1.0230539864584981437e-29 1.570796326794896558" />
+        <origin xyz="0.083000000000000212497 0.029000000000000018818 -0.010000000000000034903" rpy="-3.141592653589793116 1.0230539864584981437e-29 1.570796326794896558" />
         <parent link="palm_base" />
         <child link="plato_f2_proxbracket" />
@@ -291,5 +291,5 @@
     </link>
     <joint name="plato_f3_pip_pitch" type="revolute">
-        <origin xyz="0.048000000000000542233 -4.0156137963431870475e-17 -0.0029000000000002287837" rpy="1.0555934094656064912e-14 1.1602401833798466844e-14 1.6653345369355321631e-16" />
+        <origin xyz="0.0480000000000005006 -4.5699121570264011893e-17 -0.0029000000000002357226" rpy="1.0555934094656064912e-14 1.1602401833798466844e-14 1.6653345369355321631e-16" />
         <parent link="plato_f3_prox" />
         <child link="plato_f3_mid" />
@@ -299,5 +299,5 @@
     </joint>
     <joint name="plato_f3_mcp_pitch" type="revolute">
-        <origin xyz="-0.0049999999999998274991 0.028150000000000174882 -0.0099000000000001205092" rpy="-1.5707963267949085484 6.1550351739900040327e-15 1.5707963267948936714" />
+        <origin xyz="-0.0049999999999998170908 0.028150000000000105493 -0.0099000000000001205092" rpy="-1.5707963267949085484 6.1550351739900040327e-15 1.5707963267948936714" />
         <parent link="plato_f3_proxbracket" />
         <child link="plato_f3_prox" />
@@ -307,5 +307,5 @@
     </joint>
     <joint name="plato_f3_mcp_yaw" type="revolute">
-        <origin xyz="0.14970000000000047158 -0.029000000000000088207 -0.01000000000000005225" rpy="3.1415926535897891192 -1.7461186382788093093e-14 1.5707963267949038855" />
+        <origin xyz="0.083000000000000212497 -0.029000000000000115963 -0.010000000000000034903" rpy="3.1415926535897891192 -1.7461186382788093093e-14 1.5707963267949038855" />
         <parent link="palm_base" />
         <child link="plato_f3_proxbracket" />
