Commit message: grav comp & moveit

File: plato_description/urdf/plato_xacro/plato.ros2_control.xacro (robot description, xacro)
@@ -3,6 +3,6 @@
     <xacro:macro name="plato_ros2_control" params="
                                                 name
-                                                gazebo_classic:=^|false"
-                                                >
+                                                gazebo_classic:=^|false
+                                                mock_hardware:=^|false">
         <!-- Gazebo ROS2 Control Plugin -->
         <xacro:if value="${gazebo_classic}">
@@ -19,5 +19,8 @@
                     <plugin>gazebo_ros2_control/GazeboSystem</plugin>
                 </xacro:if>
-                <xacro:unless value="${gazebo_classic}">
+                <xacro:if value="${mock_hardware}">
+                    <plugin>mock_components/GenericSystem</plugin>
+                </xacro:if>
+                <xacro:unless value="${gazebo_classic or mock_hardware }">
                     <plugin>plato_hardware_interface/PLATOHardware</plugin>
                 </xacro:unless>

File: plato_description/urdf/plato_xacro/plato_hand_description.xacro (robot description, xacro)
@@ -4,9 +4,9 @@
     <!-- if connector_link is defined -->
     <!-- Connector Joint -->
-    <!-- <joint name="plato_connector_joint" type="fixed">
+    <joint name="plato_connector_joint" type="fixed">
         <parent link="${connector_link}"/>
         <child link="plato_base_link"/>
         <origin xyz="${xyz}" rpy="${rpy}"/>
-    </joint> -->
+    </joint>
     <!-- Base Link -->
     <link name="plato_base_link">

File: plato_moveit_config/config/plato_hand.urdf.xacro (robot description, xacro)
@@ -2,5 +2,5 @@
 <robot name="plato_hand" xmlns:xacro="http://www.ros.org/wiki/xacro">
     <!-- Arguments -->
-    <xacro:arg name="mock_hardware" default="false" />
+    <xacro:arg name="mock_hardware" default="true" />
     <xacro:arg name="gazebo_classic" default="false" />
     <!-- Set World Frame -->
@@ -18,6 +18,7 @@
     <!-- Plato Hand Ros2 Control -->
     <xacro:plato_ros2_control
-        name="plato_hand_gazebo_controller"
-        gazebo_classic="$(arg gazebo_classic)"/>
+        name="plato_ros2_controller"
+        gazebo_classic="$(arg gazebo_classic)"
+        mock_hardware="$(arg mock_hardware)"/>
     <xacro:plato_gazebo
         name="plato_gazebo"
