Commit message: tf node name change

File: plato_description/urdf/plato_xacro/plato_hand_description.xacro (robot description, xacro)
@@ -4,9 +4,9 @@
     <!-- if connector_link is defined -->
     <!-- Connector Joint -->
-    <joint name="plato_connector_joint" type="fixed">
+    <!-- <joint name="plato_connector_joint" type="fixed">
         <parent link="${connector_link}"/>
         <child link="plato_base_link"/>
         <origin xyz="${xyz}" rpy="${rpy}"/>
-    </joint>
+    </joint> -->
     <!-- Base Link -->
     <link name="plato_base_link">

Commit message: RTOS testing

File: plato_description/urdf/plato_xacro/plato_hand_description.xacro (robot description, xacro)
@@ -139,5 +139,5 @@
         <child link="plato_distal_1" />
         <axis xyz="0 0 1"/>
-        <limit effort="0.06" velocity="0.0872665" lower="-0.34906585039886589561" upper="1.570796326794896558"/>
+        <limit effort="0.06" velocity="0.0872665" lower="0.0" upper="1.570796326794896558"/>
         <joint_properties friction="0.03"/>
     </joint>
@@ -230,5 +230,5 @@
         <child link="plato_distal_2" />
         <axis xyz="0 0 1"/>
-        <limit effort="0.06" velocity="0.0872665" lower="-1.570796326794896558" upper="0.34906585039886589561"/>
+        <limit effort="0.06" velocity="0.0872665" lower="-1.570796326794896558" upper="0.0"/>
         <joint_properties friction="0.03"/>
     </joint>
@@ -321,5 +321,5 @@
         <child link="plato_distal_3" />
         <axis xyz="0 0 1"/>
-        <limit effort="0.06" velocity="0.0872665" lower="-1.570796326794896558" upper="0.34906585039886589561"/>
+        <limit effort="0.06" velocity="0.0872665" lower="-1.570796326794896558" upper="0.0"/>
         <joint_properties friction="0.01"/>
     </joint>
