Commit message: integration with gz debugging

File: optimo_description/urdf/archive/optimo.xacro (robot description, xacro)
@@ -310,15 +310,4 @@
                 <param name="max">150</param>
             </command_interface>
-            <state_interface name="position"/>
-            <state_interface name="velocity" />
-            <state_interface name="effort" />
-        </joint>
-        <joint name="joint6">
-            <command_interface name="effort">
-                <param name="min">-150</param>
-                <param name="max">150</param>
-            </command_interface>
-            <state_interface name="position"/>
-            <state_interface name="velocity" />
             <state_interface name="effort" />
         </joint>

File: optimo_description/urdf/optimo.urdf.xacro (robot description, xacro)
@@ -3,3 +3,5 @@
     <!-- Include the URDF of the robot arm -->
     <xacro:include filename="optimo_xacro/optimo_arm.xacro" />
+    <!-- Include gz configuration -->
+    <!-- <xacro:include filename="optimo_xacro/optimo.gz.xacro" /> -->
 </robot>

File: optimo_description/urdf/optimo_xacro/optimo_arm.xacro (robot description, xacro)
@@ -43,5 +43,5 @@
                 <mesh filename="file://$(find optimo_description)/meshes/link1.stl"/>
             </geometry>
-            <material name="white">
+            <material name="white"/>
         </visual>
         <collision>
