Commit message: commit before testing

File: plato_description/urdf/plato_manipulator.urdf.xacro (robot description, xacro)
@@ -7,4 +7,6 @@
     <xacro:include filename="$(find optimo_description)/urdf/optimo_xacro/optimo_description.xacro"/>
     <xacro:include filename="$(find plato_description)/urdf/plato_xacro/plato_hand_description.xacro"/>
+    <xacro:include filename="$(find plato_description)/urdf/plato_xacro/plato.transmission.xacro"/>
+    <xacro:include filename="$(find plato_description)/urdf/plato_xacro/plato.ros2_control.xacro"/>
     <!-- Pedestal -->
     <xacro:pedestal_description connector_link="world" />
@@ -13,3 +15,4 @@
     <!-- Plato Hand -->
     <xacro:plato_description connector_link="optimo_ee_link"/>
+    <xacro:plato_ros2_control name="plato_hand_controller" />
 </robot>

File: plato_description/urdf/plato_xacro/plato.ros2_control.xacro (robot description, xacro)
@@ -1,8 +1,25 @@
 <?xml version="1.0.0"?>
 <robot xmlns:xacro="http://www.ros.org/wiki/xacro">
-  <xacro:macro name="plato_ros2_control" params="name">
+  <xacro:macro name="plato_ros2_control" params="
+                                                name
+                                                use_mock_hardware:=^|false
+                                                gazebo_classic:=^|true
+                                                gazebo:=^|false
+                                                plato_hardware:=^|false"
+                                                >
     <ros2_control name="${name}" type="system">
         <hardware>
-            <plugin>plato_hardware_interface/PLATOHardware</plugin>
+            <xacro:if value="${use_mock_hardware}">
+                <plugin>mock_componets/GenericSystem</plugin>
+            </xacro:if>
+            <xacro:if value="${gazebo_classic}">
+                <plugin>gazebo_ros2_control/GazeboSystem</plugin>
+            </xacro:if>
+            <xacro:if value="${gazebo}">
+                <plugin>ign_ros2_control/IgnitionSystem</plugin>
+            </xacro:if>
+            <xacro:if value="${plato_hardware}">
+                <plugin>plato_hardware_interface/PLATOHardware</plugin>
+            </xacro:if>
         </hardware>
         <joint name="plato_joint0">
