Commit message: commit before intergating can

File: plato_description/urdf/plato_hand.urdf.xacro (robot description, xacro)
@@ -5,5 +5,9 @@
     <!-- Include Xacro -->
     <xacro:include filename="$(find plato_description)/urdf/plato_xacro/plato_hand_description.xacro"/>
+    <xacro:include filename="$(find plato_description)/urdf/plato_xacro/plato.transmission.xacro"/>
+    <xacro:include filename="$(find plato_description)/urdf/plato_xacro/plato.ros2_control.xacro"/>
     <!-- Plato Hand -->
     <xacro:plato_description connector_link="world"/>
+    <!-- Plato Hand Ros2 Control -->
+    <xacro:plato_ros2_control name="plato_hand_controller" />
 </robot>

File: plato_description/urdf/plato_xacro/plato_hand_description.xacro (robot description, xacro)
@@ -122,5 +122,5 @@
         <child link="plato_bracket_1" />
         <axis xyz="0 0 1"/>
-        <limit effort="1.5" velocity="1.5706999999999999851" lower="-0.1745329251994329478" upper="0.785398163397448279"/>
+        <limit effort="0.09" velocity="1.5706999999999999851" lower="-0.1745329251994329478" upper="0.785398163397448279"/>
         <joint_properties friction="0.0"/>
     </joint>
@@ -130,5 +130,5 @@
         <child link="plato_proximal_1" />
         <axis xyz="0 0 1"/>
-        <limit effort="1.5" velocity="1.5706999999999999851" lower="-1.570796326794896558" upper="0.34906585039886589561"/>
+        <limit effort="0.09" velocity="1.5706999999999999851" lower="-1.570796326794896558" upper="0.34906585039886589561"/>
         <joint_properties friction="0.0"/>
     </joint>
@@ -138,5 +138,5 @@
         <child link="plato_distal_1" />
         <axis xyz="0 0 1"/>
-        <limit effort="1.5" velocity="1.5706999999999999851" lower="-0.34906585039886589561" upper="1.570796326794896558"/>
+        <limit effort="0.09" velocity="1.5706999999999999851" lower="-0.34906585039886589561" upper="1.570796326794896558"/>
         <joint_properties friction="0.0"/>
     </joint>
@@ -213,5 +213,5 @@
         <child link="plato_bracket_2" />
         <axis xyz="0 0 1"/>
-        <limit effort="1.5" velocity="1.5706999999999999851" lower="-0.087266462599716473902" upper="0.087266462599716473902"/>
+        <limit effort="0.09" velocity="1.5706999999999999851" lower="-0.087266462599716473902" upper="0.087266462599716473902"/>
         <joint_properties friction="0.0"/>
     </joint>
@@ -221,5 +221,5 @@
         <child link="plato_proximal_2" />
         <axis xyz="0 0 1"/>
-        <limit effort="1.5" velocity="1.5706999999999999851" lower="-0.87266462599716476678" upper="0.87266462599716476678"/>
+        <limit effort="0.09" velocity="1.5706999999999999851" lower="-0.87266462599716476678" upper="0.87266462599716476678"/>
         <joint_properties friction="0.0"/>
     </joint>
@@ -229,5 +229,5 @@
         <child link="plato_distal_2" />
         <axis xyz="0 0 1"/>
-        <limit effort="1.5" velocity="1.5706999999999999851" lower="-1.570796326794896558" upper="0.34906585039886589561"/>
+        <limit effort="0.09" velocity="1.5706999999999999851" lower="-1.570796326794896558" upper="0.34906585039886589561"/>
         <joint_properties friction="0.0"/>
     </joint>
@@ -304,5 +304,5 @@
         <child link="plato_bracket_3" />
         <axis xyz="0 0 1"/>
-        <limit effort="1.5" velocity="1.5706999999999999851" lower="-0.087266462599716473902" upper="0.087266462599716473902"/>
+        <limit effort="0.09" velocity="1.5706999999999999851" lower="-0.087266462599716473902" upper="0.087266462599716473902"/>
         <joint_properties friction="0.0"/>
     </joint>
@@ -312,5 +312,5 @@
         <child link="plato_proximal_3" />
         <axis xyz="0 0 1"/>
-        <limit effort="1.5" velocity="1.5706999999999999851" lower="-0.87266462599716476678" upper="0.87266462599716476678"/>
+        <limit effort="0.09" velocity="1.5706999999999999851" lower="-0.87266462599716476678" upper="0.87266462599716476678"/>
         <joint_properties friction="0.0"/>
     </joint>
@@ -320,5 +320,5 @@
         <child link="plato_distal_3" />
         <axis xyz="0 0 1"/>
-        <limit effort="1.5" velocity="1.5706999999999999851" lower="-1.570796326794896558" upper="0.34906585039886589561"/>
+        <limit effort="0.09" velocity="1.5706999999999999851" lower="-1.570796326794896558" upper="0.34906585039886589561"/>
         <joint_properties friction="0.0"/>
     </joint>

Commit message: cleanup

File: plato_description/urdf/plato_hand.urdf.xacro (robot description, xacro)
@@ -1,4 +1,9 @@
 <?xml version="1.0"?>
 <robot name="plato_hand" xmlns:xacro="http://www.ros.org/wiki/xacro">
+    <!-- Arguments -->
+    <xacro:arg name="mock_hardware" default="false" />
+    <xacro:arg name="gazebo_classic" default="false" />
+    <xacro:arg name="gazebo" default="true" />
+    <xacro:arg name="simulation_controllers" default="" />
     <!-- Set World Frame -->
     <link name="world"/>
@@ -10,4 +15,7 @@
     <xacro:plato_description connector_link="world"/>
     <!-- Plato Hand Ros2 Control -->
-    <xacro:plato_ros2_control name="plato_hand_controller" />
+    <xacro:plato_ros2_control name="plato_hand_controller"
+                              mock_hardware="$(arg mock_hardware)"
+                              gazebo_classic="$(arg gazebo_classic)"
+                              gazebo ="$(arg gazebo)"/>
 </robot>

File: plato_description/urdf/plato_xacro/plato.ros2_control.xacro (robot description, xacro)
@@ -1,31 +1,36 @@
-<?xml version="1.0.0"?>
+<?xml version="0.06.0"?>
 <robot xmlns:xacro="http://www.ros.org/wiki/xacro">
   <xacro:macro name="plato_ros2_control" params="
                                                 name
-                                                use_mock_hardware:=^|false
+                                                mock_hardware:=^|false
                                                 gazebo_classic:=^|false
-                                                gazebo:=^|false
-                                                plato_hardware:=^|true"
+                                                gazebo:=^|false"
                                                 >
     <ros2_control name="${name}" type="system">
         <hardware>
-            <xacro:if value="${use_mock_hardware}">
+            <xacro:if value="${mock_hardware}">
                 <plugin>mock_componets/GenericSystem</plugin>
             </xacro:if>
             <xacro:if value="${gazebo_classic}">
                 <plugin>gazebo_ros2_control/GazeboSystem</plugin>
+                <gazebo>
+                    <plugin filename="libgazebo_ros2_control.so" name="gazebo_ros2_control">
+                        <parameters>$(find plato_bringup)/config/plato_hand_controllers.yaml</parameters>
+                    </plugin>
+                </gazebo>
             </xacro:if>
             <xacro:if value="${gazebo}">
                 <plugin>ign_ros2_control/IgnitionSystem</plugin>
             </xacro:if>
-            <xacro:if value="${plato_hardware}">
+            <xacro:unless value="${mock_hardware or gazebo_classic or gazebo}">
                 <plugin>plato_hardware_interface/PLATOHardware</plugin>
-            </xacro:if>
+            </xacro:unless>
         </hardware>
         <joint name="plato_joint0">
             <command_interface name="effort">
-                <param name="min">-1.0</param>
-                <param name="max">1.0</param>
+                <param name="min">-0.06</param>
+                <param name="max">0.06</param>
             </command_interface>
+            <command_interface name="position"/>
             <state_interface name="position"/>
             <state_interface name="velocity" />
@@ -34,6 +39,6 @@
         <joint name="plato_joint1">
             <command_interface name="effort">
-                <param name="min">-1.0</param>
-                <param name="max">1.0</param>
+                <param name="min">-0.06</param>
+                <param name="max">0.06</param>
             </command_interface>
             <state_interface name="position"/>
@@ -43,6 +48,6 @@
         <joint name="plato_joint2">
             <command_interface name="effort">
-                <param name="min">-1.0</param>
-                <param name="max">1.0</param>
+                <param name="min">-0.06</param>
+                <param name="max">0.06</param>
             </command_interface>
             <state_interface name="position">
@@ -53,6 +58,6 @@
         <joint name="plato_joint3">
             <command_interface name="effort">
-                <param name="min">-1.0</param>
-                <param name="max">1.0</param>
+                <param name="min">-0.06</param>
+                <param name="max">0.06</param>
             </command_interface>
             <state_interface name="position"/>
@@ -62,6 +67,6 @@
         <joint name="plato_joint4">
             <command_interface name="effort">
-                <param name="min">-1.0</param>
-                <param name="max">1.0</param>
+                <param name="min">-0.06</param>
+                <param name="max">0.06</param>
             </command_interface>
             <state_interface name="position"/>
@@ -71,6 +76,6 @@
         <joint name="plato_joint5">
             <command_interface name="effort">
-                <param name="min">-1.0</param>
-                <param name="max">1.0</param>
+                <param name="min">-0.06</param>
+                <param name="max">0.06</param>
             </command_interface>
             <state_interface name="position"/>
@@ -80,6 +85,6 @@
         <joint name="plato_joint6">
             <command_interface name="effort">
-                <param name="min">-1.0</param>
-                <param name="max">1.0</param>
+                <param name="min">-0.06</param>
+                <param name="max">0.06</param>
             </command_interface>
             <state_interface name="position"/>
@@ -89,6 +94,6 @@
         <joint name="plato_joint7">
             <command_interface name="effort">
-                <param name="min">-1.0</param>
-                <param name="max">1.0</param>
+                <param name="min">-0.06</param>
+                <param name="max">0.06</param>
             </command_interface>
             <state_interface name="position"/>
@@ -98,6 +103,6 @@
         <joint name="plato_joint8">
             <command_interface name="effort">
-                <param name="min">-1.0</param>
-                <param name="max">1.0</param>
+                <param name="min">-0.06</param>
+                <param name="max">0.06</param>
             </command_interface>
             <state_interface name="position"/>

File: plato_description/urdf/plato_xacro/plato_hand_description.xacro (robot description, xacro)
@@ -122,5 +122,5 @@
         <child link="plato_bracket_1" />
         <axis xyz="0 0 1"/>
-        <limit effort="0.09" velocity="1.5706999999999999851" lower="-0.1745329251994329478" upper="0.785398163397448279"/>
+        <limit effort="0.06" velocity="1.5706999999999999851" lower="-0.1745329251994329478" upper="0.785398163397448279"/>
         <joint_properties friction="0.0"/>
     </joint>
@@ -130,5 +130,5 @@
         <child link="plato_proximal_1" />
         <axis xyz="0 0 1"/>
-        <limit effort="0.09" velocity="1.5706999999999999851" lower="-1.570796326794896558" upper="0.34906585039886589561"/>
+        <limit effort="0.06" velocity="1.5706999999999999851" lower="-1.570796326794896558" upper="0.34906585039886589561"/>
         <joint_properties friction="0.0"/>
     </joint>
@@ -138,5 +138,5 @@
         <child link="plato_distal_1" />
         <axis xyz="0 0 1"/>
-        <limit effort="0.09" velocity="1.5706999999999999851" lower="-0.34906585039886589561" upper="1.570796326794896558"/>
+        <limit effort="0.06" velocity="1.5706999999999999851" lower="-0.34906585039886589561" upper="1.570796326794896558"/>
         <joint_properties friction="0.0"/>
     </joint>
@@ -213,5 +213,5 @@
         <child link="plato_bracket_2" />
         <axis xyz="0 0 1"/>
-        <limit effort="0.09" velocity="1.5706999999999999851" lower="-0.087266462599716473902" upper="0.087266462599716473902"/>
+        <limit effort="0.06" velocity="1.5706999999999999851" lower="-0.087266462599716473902" upper="0.087266462599716473902"/>
         <joint_properties friction="0.0"/>
     </joint>
@@ -221,5 +221,5 @@
         <child link="plato_proximal_2" />
         <axis xyz="0 0 1"/>
-        <limit effort="0.09" velocity="1.5706999999999999851" lower="-0.87266462599716476678" upper="0.87266462599716476678"/>
+        <limit effort="0.06" velocity="1.5706999999999999851" lower="-0.87266462599716476678" upper="0.87266462599716476678"/>
         <joint_properties friction="0.0"/>
     </joint>
@@ -229,5 +229,5 @@
         <child link="plato_distal_2" />
         <axis xyz="0 0 1"/>
-        <limit effort="0.09" velocity="1.5706999999999999851" lower="-1.570796326794896558" upper="0.34906585039886589561"/>
+        <limit effort="0.06" velocity="1.5706999999999999851" lower="-1.570796326794896558" upper="0.34906585039886589561"/>
         <joint_properties friction="0.0"/>
     </joint>
@@ -304,5 +304,5 @@
         <child link="plato_bracket_3" />
         <axis xyz="0 0 1"/>
-        <limit effort="0.09" velocity="1.5706999999999999851" lower="-0.087266462599716473902" upper="0.087266462599716473902"/>
+        <limit effort="0.06" velocity="1.5706999999999999851" lower="-0.087266462599716473902" upper="0.087266462599716473902"/>
         <joint_properties friction="0.0"/>
     </joint>
@@ -312,5 +312,5 @@
         <child link="plato_proximal_3" />
         <axis xyz="0 0 1"/>
-        <limit effort="0.09" velocity="1.5706999999999999851" lower="-0.87266462599716476678" upper="0.87266462599716476678"/>
+        <limit effort="0.06" velocity="1.5706999999999999851" lower="-0.87266462599716476678" upper="0.87266462599716476678"/>
         <joint_properties friction="0.0"/>
     </joint>
@@ -320,5 +320,5 @@
         <child link="plato_distal_3" />
         <axis xyz="0 0 1"/>
-        <limit effort="0.09" velocity="1.5706999999999999851" lower="-1.570796326794896558" upper="0.34906585039886589561"/>
+        <limit effort="0.06" velocity="1.5706999999999999851" lower="-1.570796326794896558" upper="0.34906585039886589561"/>
         <joint_properties friction="0.0"/>
     </joint>

Commit message: plato hand gazebo joint traj controller with effort

File: plato_description/urdf/plato_hand.urdf.xacro (robot description, xacro)
@@ -11,6 +11,9 @@
     <xacro:include filename="$(find plato_description)/urdf/plato_xacro/plato.transmission.xacro"/>
     <xacro:include filename="$(find plato_description)/urdf/plato_xacro/plato.ros2_control.xacro"/>
+    <xacro:include filename="$(find optimo_description)/urdf/optimo_xacro/pedestal.xacro"/>
+    <!-- Pedestal -->
+    <xacro:pedestal_description connector_link="world"/>
     <!-- Plato Hand -->
-    <xacro:plato_description connector_link="world"/>
+    <xacro:plato_description connector_link="stand_link" xyz="0.15 0 0.0" />
     <!-- Plato Hand Ros2 Control -->
     <xacro:plato_ros2_control name="plato_hand_controller" />

File: plato_description/urdf/plato_xacro/plato_hand_description.xacro (robot description, xacro)
@@ -1,10 +1,10 @@
 <?xml version="1.0"?>
 <robot xmlns:xacro="http://www.ros.org/wiki/xacro">
-<xacro:macro name="plato_description" params="connector_link">
+<xacro:macro name="plato_description" params="connector_link  xyz:='0 0 0'  rpy:='0 0 0' ">
     <!-- Connector Joint -->
     <joint name="plato_connector_joint" type="fixed">
         <parent link="${connector_link}"/>
         <child link="plato_base_link"/>
-        <origin xyz="0 0 0" rpy="0 0 0"/>
+        <origin xyz="${xyz}" rpy="${rpy}"/>
     </joint>
     <!-- Base Link -->
