Commit message: wip

File: plato_description/urdf/plato_hand.urdf.xacro (robot description, xacro)
@@ -4,5 +4,4 @@
     <xacro:arg name="mock_hardware" default="false" />
     <xacro:arg name="gazebo_classic" default="false" />
-    <xacro:arg name="gazebo" default="true" />
     <!-- Set World Frame -->
     <link name="world"/>
@@ -11,4 +10,5 @@
     <xacro:include filename="$(find plato_description)/urdf/plato_xacro/plato.transmission.xacro"/>
     <xacro:include filename="$(find plato_description)/urdf/plato_xacro/plato.ros2_control.xacro"/>
+    <xacro:include filename="$(find plato_description)/urdf/plato_xacro/plato.gazebo.xacro"/>
     <xacro:include filename="$(find optimo_description)/urdf/optimo_xacro/pedestal.xacro"/>
     <!-- Pedestal -->
@@ -17,4 +17,9 @@
     <xacro:plato_description connector_link="stand_link" xyz="0.15 0 0.0" />
     <!-- Plato Hand Ros2 Control -->
-    <xacro:plato_ros2_control name="plato_hand_controller" />
+    <xacro:plato_ros2_control
+        name="plato_hand_gazebo_controller"
+        gazebo_classic="$(arg gazebo_classic)"/>
+    <!-- <xacro:plato_gazebo
+        name="plato_gazebo"
+        gazebo_classic="$(arg gazebo_classic)"/> -->
 </robot>

File: plato_description/urdf/plato_xacro/plato.ros2_control.xacro (robot description, xacro)
@@ -1,101 +1,118 @@
 <?xml version="0.06.0"?>
 <robot xmlns:xacro="http://www.ros.org/wiki/xacro">
-  <xacro:macro name="plato_ros2_control" params="
-                                                name"
+    <xacro:macro name="plato_ros2_control" params="
+                                                name
+                                                gazebo_classic:=^|false"
                                                 >
-    <gazebo>
-        <plugin filename="libgazebo_ros2_control.so" name="gazebo_ros2_control">
-            <parameters>$(find plato_bringup)/config/plato_gazebo_controllers.yaml</parameters>
-        </plugin>
-    </gazebo>
-    <ros2_control name="${name}" type="system">
-        <hardware>
-                <plugin>gazebo_ros2_control/GazeboSystem</plugin>
-                <!-- <plugin>plato_hardware_interface/PLATOHardware</plugin> -->
-        </hardware>
-        <joint name="plato_joint0">
-            <command_interface name="effort">
-                <param name="min">-0.06</param>
-                <param name="max">0.06</param>
-            </command_interface>
-            <command_interface name="position"/>
-            <state_interface name="position"/>
-            <state_interface name="velocity" />
-            <state_interface name="effort" />
-        </joint>
-        <joint name="plato_joint1">
-            <command_interface name="effort">
-                <param name="min">-0.06</param>
-                <param name="max">0.06</param>
-            </command_interface>
-            <state_interface name="position"/>
-            <state_interface name="velocity" />
-            <state_interface name="effort" />
-        </joint>
-        <joint name="plato_joint2">
-            <command_interface name="effort">
-                <param name="min">-0.06</param>
-                <param name="max">0.06</param>
-            </command_interface>
-            <state_interface name="position">
-            </state_interface>
-            <state_interface name="velocity" />
-            <state_interface name="effort" />
-        </joint>
-        <joint name="plato_joint3">
-            <command_interface name="effort">
-                <param name="min">-0.06</param>
-                <param name="max">0.06</param>
-            </command_interface>
-            <state_interface name="position"/>
-            <state_interface name="velocity" />
-            <state_interface name="effort" />
-        </joint>
-        <joint name="plato_joint4">
-            <command_interface name="effort">
-                <param name="min">-0.06</param>
-                <param name="max">0.06</param>
-            </command_interface>
-            <state_interface name="position"/>
-            <state_interface name="velocity" />
-            <state_interface name="effort" />
-        </joint>
-        <joint name="plato_joint5">
-            <command_interface name="effort">
-                <param name="min">-0.06</param>
-                <param name="max">0.06</param>
-            </command_interface>
-            <state_interface name="position"/>
-            <state_interface name="velocity" />
-            <state_interface name="effort" />
-        </joint>
-        <joint name="plato_joint6">
-            <command_interface name="effort">
-                <param name="min">-0.06</param>
-                <param name="max">0.06</param>
-            </command_interface>
-            <state_interface name="position"/>
-            <state_interface name="velocity" />
-            <state_interface name="effort" />
-        </joint>
-        <joint name="plato_joint7">
-            <command_interface name="effort">
-                <param name="min">-0.06</param>
-                <param name="max">0.06</param>
-            </command_interface>
-            <state_interface name="position"/>
-            <state_interface name="velocity" />
-            <state_interface name="effort" />
-        </joint>
-        <joint name="plato_joint8">
-            <command_interface name="effort">
-                <param name="min">-0.06</param>
-                <param name="max">0.06</param>
-            </command_interface>
-            <state_interface name="position"/>
-            <state_interface name="velocity" />
-            <state_interface name="effort" />
-        </joint>
-    </ros2_control>
+        <!-- Gazebo ROS2 Control Plugin -->
+        <xacro:if value="${gazebo_classic}">
+            <gazebo>
+                <plugin filename="libgazebo_ros2_control.so" name="gazebo_ros2_control">
+                    <parameters>$(find plato_bringup)/config/plato_gazebo_controllers.yaml</parameters>
+                </plugin>
+            </gazebo>
+        </xacro:if>
+        <ros2_control name="${name}" type="system">
+            <!-- Hardware -->
+            <hardware>
+                <xacro:if value="${gazebo_classic}">
+                    <plugin>gazebo_ros2_control/GazeboSystem</plugin>
+                </xacro:if>
+                <xacro:unless value="${gazebo_classic}">
+                    <plugin>plato_hardware_interface/PLATOHardware</plugin>
+                </xacro:unless>
+            </hardware>
+            <joint name="plato_joint0">
+                <command_interface name="effort">
+                    <param name="min">-0.06</param>
+                    <param name="max">0.06</param>
+                </command_interface>
+                <!-- <command_interface name="position"/> -->
+                <state_interface name="position"/>
+                <state_interface name="velocity" />
+                <state_interface name="effort" />
+            </joint>
+            <joint name="plato_joint1">
+                <command_interface name="effort">
+                    <param name="min">-0.06</param>
+                    <param name="max">0.06</param>
+                </command_interface>
+                <!-- <command_interface name="position"/> -->
+                <state_interface name="position"/>
+                <state_interface name="velocity" />
+                <state_interface name="effort" />
+            </joint>
+            <joint name="plato_joint2">
+                <command_interface name="effort">
+                    <param name="min">-0.06</param>
+                    <param name="max">0.06</param>
+                </command_interface>
+                <!-- <command_interface name="position"/> -->
+                <state_interface name="position">
+                </state_interface>
+                <state_interface name="velocity" />
+                <state_interface name="effort" />
+            </joint>
+            <joint name="plato_joint3">
+                <command_interface name="effort">
+                    <param name="min">-0.06</param>
+                    <param name="max">0.06</param>
+                </command_interface>
+                <!-- <command_interface name="position"/> -->
+                <state_interface name="position"/>
+                <state_interface name="velocity" />
+                <state_interface name="effort" />
+            </joint>
+            <joint name="plato_joint4">
+                <command_interface name="effort">
+                    <param name="min">-0.06</param>
+                    <param name="max">0.06</param>
+                </command_interface>
+                <!-- <command_interface name="position"/> -->
+                <state_interface name="position"/>
+                <state_interface name="velocity" />
+                <state_interface name="effort" />
+            </joint>
+            <joint name="plato_joint5">
+                <command_interface name="effort">
+                    <param name="min">-0.06</param>
+                    <param name="max">0.06</param>
+                </command_interface>
+                <!-- <command_interface name="position"/> -->
+                <state_interface name="position"/>
+                <state_interface name="velocity" />
+                <state_interface name="effort" />
+            </joint>
+            <joint name="plato_joint6">
+                <command_interface name="effort">
+                    <param name="min">-0.06</param>
+                    <param name="max">0.06</param>
+                </command_interface>
+                <!-- <command_interface name="position"/> -->
+                <state_interface name="position"/>
+                <state_interface name="velocity" />
+                <state_interface name="effort" />
+            </joint>
+            <joint name="plato_joint7">
+                <command_interface name="effort">
+                    <param name="min">-0.06</param>
+                    <param name="max">0.06</param>
+                </command_interface>
+                <!-- <command_interface name="position"/> -->
+                <state_interface name="position"/>
+                <state_interface name="velocity" />
+                <state_interface name="effort" />
+            </joint>
+            <joint name="plato_joint8">
+                <command_interface name="effort">
+                    <param name="min">-0.06</param>
+                    <param name="max">0.06</param>
+                </command_interface>
+                <!-- <command_interface name="position"/> -->
+                <state_interface name="position"/>
+                <state_interface name="velocity" />
+                <state_interface name="effort" />
+            </joint>
+        </ros2_control>
   </xacro:macro>
 </robot>

File: plato_description/urdf/plato_xacro/plato_hand_description.xacro (robot description, xacro)
@@ -123,5 +123,5 @@
         <axis xyz="0 0 1"/>
         <limit effort="0.06" velocity="1.5706999999999999851" lower="-0.1745329251994329478" upper="0.785398163397448279"/>
-        <joint_properties friction="0.0"/>
+        <joint_properties friction="0.03"/>
     </joint>
     <joint name="plato_joint1" type="revolute">
@@ -131,5 +131,5 @@
         <axis xyz="0 0 1"/>
         <limit effort="0.06" velocity="1.5706999999999999851" lower="-1.570796326794896558" upper="0.34906585039886589561"/>
-        <joint_properties friction="0.0"/>
+        <joint_properties friction="0.03"/>
     </joint>
     <joint name="plato_joint2" type="revolute">
@@ -139,5 +139,5 @@
         <axis xyz="0 0 1"/>
         <limit effort="0.06" velocity="1.5706999999999999851" lower="-0.34906585039886589561" upper="1.570796326794896558"/>
-        <joint_properties friction="0.0"/>
+        <joint_properties friction="0.03"/>
     </joint>
     <!-- Finger 2: Index -->
@@ -214,5 +214,5 @@
         <axis xyz="0 0 1"/>
         <limit effort="0.06" velocity="1.5706999999999999851" lower="-0.087266462599716473902" upper="0.087266462599716473902"/>
-        <joint_properties friction="0.0"/>
+        <joint_properties friction="0.03"/>
     </joint>
     <joint name="plato_joint4" type="revolute">
@@ -222,5 +222,5 @@
         <axis xyz="0 0 1"/>
         <limit effort="0.06" velocity="1.5706999999999999851" lower="-0.87266462599716476678" upper="0.87266462599716476678"/>
-        <joint_properties friction="0.0"/>
+        <joint_properties friction="0.03"/>
     </joint>
     <joint name="plato_joint5" type="revolute">
@@ -230,5 +230,5 @@
         <axis xyz="0 0 1"/>
         <limit effort="0.06" velocity="1.5706999999999999851" lower="-1.570796326794896558" upper="0.34906585039886589561"/>
-        <joint_properties friction="0.0"/>
+        <joint_properties friction="0.03"/>
     </joint>
     <!-- Finger 3: Pinky (or Middle) -->
@@ -305,5 +305,5 @@
         <axis xyz="0 0 1"/>
         <limit effort="0.06" velocity="1.5706999999999999851" lower="-0.087266462599716473902" upper="0.087266462599716473902"/>
-        <joint_properties friction="0.0"/>
+        <joint_properties friction="0.03"/>
     </joint>
     <joint name="plato_joint7" type="revolute">
@@ -313,5 +313,5 @@
         <axis xyz="0 0 1"/>
         <limit effort="0.06" velocity="1.5706999999999999851" lower="-0.87266462599716476678" upper="0.87266462599716476678"/>
-        <joint_properties friction="0.0"/>
+        <joint_properties friction="0.03"/>
     </joint>
     <joint name="plato_joint8" type="revolute">
@@ -321,5 +321,5 @@
         <axis xyz="0 0 1"/>
         <limit effort="0.06" velocity="1.5706999999999999851" lower="-1.570796326794896558" upper="0.34906585039886589561"/>
-        <joint_properties friction="0.0"/>
+        <joint_properties friction="0.01"/>
     </joint>
 </xacro:macro>

Commit message: joint traj effort controller in gazebo

File: plato_description/urdf/plato_hand.urdf.xacro (robot description, xacro)
@@ -20,6 +20,6 @@
         name="plato_hand_gazebo_controller"
         gazebo_classic="$(arg gazebo_classic)"/>
-    <!-- <xacro:plato_gazebo
+    <xacro:plato_gazebo
         name="plato_gazebo"
-        gazebo_classic="$(arg gazebo_classic)"/> -->
+        gazebo_classic="$(arg gazebo_classic)"/>
 </robot>

File: plato_description/urdf/plato_xacro/plato.gazebo.xacro (robot description, xacro)
@@ -6,13 +6,36 @@
                                             >
         <xacro:if value="${gazebo_classic}">
+            <xacro:property name="damping" value="0.5"/>
+            <xacro:property name="friction" value="10.0"/>
+            <xacro:property name="spring_reference" value="0.0"/>
+            <xacro:property name="spring_stiffness" value="0.5"/>
             <!-- Joint Dynamics -->
-            <!-- <joint name="plato_joint0">
-                <dynamics>
-                    <damping>0.0</damping>
-                    <friction>0.0</friction>
-                    <spring_reference>0.0</spring_reference>
-                    <spring_stiffness>0.0</spring_stiffness>
-                </dynamics>
-            </joint>     -->
+            <gazebo reference="plato_joint0">
+                <dynamics damping="${damping}" friction="${friction}" spring_reference="${spring_reference}" spring_stiffness="${spring_stiffness}"/>
+            </gazebo>
+            <gazebo reference="plato_joint1">
+                <dynamics damping="${damping}" friction="${friction}" spring_reference="${spring_reference}" spring_stiffness="${spring_stiffness}"/>
+            </gazebo>
+            <gazebo reference="plato_joint2">
+                <dynamics damping="${damping}" friction="${friction}" spring_reference="${spring_reference}" spring_stiffness="${spring_stiffness}"/>
+            </gazebo>
+            <gazebo reference="plato_joint3">
+                <dynamics damping="${damping}" friction="${friction}" spring_reference="${spring_reference}" spring_stiffness="${spring_stiffness}"/>
+            </gazebo>
+            <gazebo reference="plato_joint4">
+                <dynamics damping="${damping}" friction="${friction}" spring_reference="${spring_reference}" spring_stiffness="${spring_stiffness}"/>
+            </gazebo>
+            <gazebo reference="plato_joint5">
+                <dynamics damping="${damping}" friction="${friction}" spring_reference="${spring_reference}" spring_stiffness="${spring_stiffness}"/>
+            </gazebo>
+            <gazebo reference="plato_joint6">
+                <dynamics damping="${damping}" friction="${friction}" spring_reference="${spring_reference}" spring_stiffness="${spring_stiffness}"/>
+            </gazebo>
+            <gazebo reference="plato_joint7">
+                <dynamics damping="${damping}" friction="${friction}" spring_reference="${spring_reference}" spring_stiffness="${spring_stiffness}"/>
+            </gazebo>
+            <gazebo reference="plato_joint8">
+                <dynamics damping="${damping}" friction="${friction}" spring_reference="${spring_reference}" spring_stiffness="${spring_stiffness}"/>
+            </gazebo>
         </xacro:if>
     </xacro:macro>

Commit message: optimo name conflict -> optiman

File: plato_description/urdf/plato_hand.urdf.xacro (robot description, xacro)
@@ -11,5 +11,5 @@
     <xacro:include filename="$(find plato_description)/urdf/plato_xacro/plato.ros2_control.xacro"/>
     <xacro:include filename="$(find plato_description)/urdf/plato_xacro/plato.gazebo.xacro"/>
-    <xacro:include filename="$(find optimo_description)/urdf/optimo_xacro/pedestal.xacro"/>
+    <xacro:include filename="$(find optiman_description)/urdf/optimo_xacro/pedestal.xacro"/>
     <!-- Pedestal -->
     <xacro:pedestal_description connector_link="world"/>

File: plato_description/urdf/plato_manipulator.urdf.xacro (robot description, xacro)
@@ -5,5 +5,5 @@
     <!-- Include Xacro -->
     <xacro:include filename="$(find optimo_description)/urdf/optimo_xacro/pedestal.xacro" />
-    <xacro:include filename="$(find optimo_description)/urdf/optimo_xacro/optimo_description.xacro"/>
+    <xacro:include filename="$(find optiman_description)/urdf/optimo_xacro/optimo_description.xacro"/>
     <xacro:include filename="$(find plato_description)/urdf/plato_xacro/plato_hand_description.xacro"/>
     <xacro:include filename="$(find plato_description)/urdf/plato_xacro/plato.transmission.xacro"/>

File: plato_description/urdf/plato_xacro/plato_hand_description.xacro (robot description, xacro)
@@ -122,5 +122,5 @@
         <child link="plato_bracket_1" />
         <axis xyz="0 0 1"/>
-        <limit effort="0.06" velocity="1.5706999999999999851" lower="-0.1745329251994329478" upper="0.785398163397448279"/>
+        <limit effort="0.06" velocity="0.0872665" lower="-0.1745329251994329478" upper="0.785398163397448279"/>
         <joint_properties friction="0.03"/>
     </joint>
@@ -130,5 +130,5 @@
         <child link="plato_proximal_1" />
         <axis xyz="0 0 1"/>
-        <limit effort="0.06" velocity="1.5706999999999999851" lower="-1.570796326794896558" upper="0.34906585039886589561"/>
+        <limit effort="0.06" velocity="0.0872665" lower="-1.570796326794896558" upper="0.34906585039886589561"/>
         <joint_properties friction="0.03"/>
     </joint>
@@ -138,5 +138,5 @@
         <child link="plato_distal_1" />
         <axis xyz="0 0 1"/>
-        <limit effort="0.06" velocity="1.5706999999999999851" lower="-0.34906585039886589561" upper="1.570796326794896558"/>
+        <limit effort="0.06" velocity="0.0872665" lower="-0.34906585039886589561" upper="1.570796326794896558"/>
         <joint_properties friction="0.03"/>
     </joint>
@@ -213,5 +213,5 @@
         <child link="plato_bracket_2" />
         <axis xyz="0 0 1"/>
-        <limit effort="0.06" velocity="1.5706999999999999851" lower="-0.087266462599716473902" upper="0.087266462599716473902"/>
+        <limit effort="0.06" velocity="0.0872665" lower="-0.087266462599716473902" upper="0.087266462599716473902"/>
         <joint_properties friction="0.03"/>
     </joint>
@@ -221,5 +221,5 @@
         <child link="plato_proximal_2" />
         <axis xyz="0 0 1"/>
-        <limit effort="0.06" velocity="1.5706999999999999851" lower="-0.87266462599716476678" upper="0.87266462599716476678"/>
+        <limit effort="0.06" velocity="0.0872665" lower="-0.87266462599716476678" upper="0.87266462599716476678"/>
         <joint_properties friction="0.03"/>
     </joint>
@@ -229,5 +229,5 @@
         <child link="plato_distal_2" />
         <axis xyz="0 0 1"/>
-        <limit effort="0.06" velocity="1.5706999999999999851" lower="-1.570796326794896558" upper="0.34906585039886589561"/>
+        <limit effort="0.06" velocity="0.0872665" lower="-1.570796326794896558" upper="0.34906585039886589561"/>
         <joint_properties friction="0.03"/>
     </joint>
@@ -304,5 +304,5 @@
         <child link="plato_bracket_3" />
         <axis xyz="0 0 1"/>
-        <limit effort="0.06" velocity="1.5706999999999999851" lower="-0.087266462599716473902" upper="0.087266462599716473902"/>
+        <limit effort="0.06" velocity="0.0872665" lower="-0.087266462599716473902" upper="0.087266462599716473902"/>
         <joint_properties friction="0.03"/>
     </joint>
@@ -312,5 +312,5 @@
         <child link="plato_proximal_3" />
         <axis xyz="0 0 1"/>
-        <limit effort="0.06" velocity="1.5706999999999999851" lower="-0.87266462599716476678" upper="0.87266462599716476678"/>
+        <limit effort="0.06" velocity="0.0872665" lower="-0.87266462599716476678" upper="0.87266462599716476678"/>
         <joint_properties friction="0.03"/>
     </joint>
@@ -320,5 +320,5 @@
         <child link="plato_distal_3" />
         <axis xyz="0 0 1"/>
-        <limit effort="0.06" velocity="1.5706999999999999851" lower="-1.570796326794896558" upper="0.34906585039886589561"/>
+        <limit effort="0.06" velocity="0.0872665" lower="-1.570796326794896558" upper="0.34906585039886589561"/>
         <joint_properties friction="0.01"/>
     </joint>
