Commit message: PID contorl

File: plato_description/urdf/plato_hand.urdf.xacro (robot description, xacro)
@@ -5,5 +5,5 @@
     <xacro:arg name="gazebo_classic" default="false" />
     <!-- Set World Frame -->
-    <link name="world"/>
+    <!-- <link name="world"/> -->
     <!-- Include Xacro -->
     <xacro:include filename="$(find plato_description)/urdf/plato_xacro/plato_hand_description.xacro"/>
@@ -11,9 +11,8 @@
     <xacro:include filename="$(find plato_description)/urdf/plato_xacro/plato.ros2_control.xacro"/>
     <xacro:include filename="$(find plato_description)/urdf/plato_xacro/plato.gazebo.xacro"/>
-    <xacro:include filename="$(find optiman_description)/urdf/optimo_xacro/pedestal.xacro"/>
     <!-- Pedestal -->
-    <xacro:pedestal_description connector_link="world"/>
+    <!-- <xacro:pedestal_description connector_link="world"/> -->
     <!-- Plato Hand -->
-    <xacro:plato_description connector_link="stand_link" xyz="0.15 0 0.0" />
+    <xacro:plato_description connector_link="optimo"/>
     <!-- Plato Hand Ros2 Control -->
     <xacro:plato_ros2_control

File: plato_description/urdf/plato_xacro/plato_hand_description.xacro (robot description, xacro)
@@ -2,10 +2,11 @@
 <robot xmlns:xacro="http://www.ros.org/wiki/xacro">
 <xacro:macro name="plato_description" params="connector_link  xyz:='0 0 0'  rpy:='0 0 0' ">
+    <!-- if connector_link is defined -->
     <!-- Connector Joint -->
-    <joint name="plato_connector_joint" type="fixed">
-        <parent link="${connector_link}"/>
+    <!-- <joint name="plato_connector_joint" type="fixed">
+        <parent link="base_link"/>
         <child link="plato_base_link"/>
         <origin xyz="${xyz}" rpy="${rpy}"/>
-    </joint>
+    </joint> -->
     <!-- Base Link -->
     <link name="plato_base_link">
@@ -37,15 +38,15 @@
     <joint name="plato_ee_joint1" type="fixed">
         <origin xyz="0.05060 0.0 0.0" rpy="-1.5707 0.0 0.0"/>
-        <parent link="plato_proximal_1"/>
+        <parent link="plato_distal_1"/>
         <child link="plato_end_effector_1"/>
     </joint>
     <joint name="plato_ee_joint2" type="fixed">
         <origin xyz="0.05060 0.0 0.0" rpy="-1.5707 0.0 0.0"/>
-        <parent link="plato_proximal_2"/>
+        <parent link="plato_distal_2"/>
         <child link="plato_end_effector_2"/>
     </joint>
     <joint name="plato_ee_joint3" type="fixed">
         <origin xyz="0.05060 0.0 0.0" rpy="-1.5707 0.0 0.0"/>
-        <parent link="plato_proximal_3"/>
+        <parent link="plato_distal_3"/>
         <child link="plato_end_effector_3"/>
     </joint>

Commit message: new moveit

File: plato_description/urdf/plato_hand.urdf.xacro (robot description, xacro)
@@ -5,5 +5,5 @@
     <xacro:arg name="gazebo_classic" default="false" />
     <!-- Set World Frame -->
-    <!-- <link name="world"/> -->
+    <link name="world"/>
     <!-- Include Xacro -->
     <xacro:include filename="$(find plato_description)/urdf/plato_xacro/plato_hand_description.xacro"/>
@@ -11,8 +11,9 @@
     <xacro:include filename="$(find plato_description)/urdf/plato_xacro/plato.ros2_control.xacro"/>
     <xacro:include filename="$(find plato_description)/urdf/plato_xacro/plato.gazebo.xacro"/>
+    <xacro:include filename="$(find optiman_description)/urdf/optimo_xacro/pedestal.xacro"/>
     <!-- Pedestal -->
-    <!-- <xacro:pedestal_description connector_link="world"/> -->
+    <xacro:pedestal_description connector_link="world"/>
     <!-- Plato Hand -->
-    <xacro:plato_description connector_link="optimo"/>
+    <xacro:plato_description connector_link="stand_link"/>
     <!-- Plato Hand Ros2 Control -->
     <xacro:plato_ros2_control

File: plato_description/urdf/plato_xacro/plato_hand_description.xacro (robot description, xacro)
@@ -4,9 +4,9 @@
     <!-- if connector_link is defined -->
     <!-- Connector Joint -->
-    <!-- <joint name="plato_connector_joint" type="fixed">
-        <parent link="base_link"/>
+    <joint name="plato_connector_joint" type="fixed">
+        <parent link="${connector_link}"/>
         <child link="plato_base_link"/>
         <origin xyz="${xyz}" rpy="${rpy}"/>
-    </joint> -->
+    </joint>
     <!-- Base Link -->
     <link name="plato_base_link">

Commit message: commit before changingto pos interface

File: plato_description/urdf/plato_hand.urdf.xacro (robot description, xacro)
@@ -5,5 +5,4 @@
     <xacro:arg name="gazebo_classic" default="false" />
     <!-- Set World Frame -->
-    <link name="world"/>
     <!-- Include Xacro -->
     <xacro:include filename="$(find plato_description)/urdf/plato_xacro/plato_hand_description.xacro"/>

File: plato_description/urdf/plato_xacro/plato.ros2_control.xacro (robot description, xacro)
@@ -32,5 +32,7 @@
                 </command_interface>
                 <!-- <command_interface name="position"/> -->
-                <state_interface name="position"/>
+                <state_interface name="position">
+                    <initial_value>0.0</initial_value>
+                </state_interface>
                 <state_interface name="velocity" />
                 <state_interface name="effort" />
@@ -43,4 +45,5 @@
                 <!-- <command_interface name="position"/> -->
                 <state_interface name="position"/>
+                    <initial_value>-0.9</initial_value>
                 <state_interface name="velocity" />
                 <state_interface name="effort" />
@@ -53,4 +56,5 @@
                 <!-- <command_interface name="position"/> -->
                 <state_interface name="position">
+                    <initial_value>0.9</initial_value>
                 </state_interface>
                 <state_interface name="velocity" />
@@ -63,5 +67,7 @@
                 </command_interface>
                 <!-- <command_interface name="position"/> -->
-                <state_interface name="position"/>
+                <state_interface name="position">
+                    <initial_value>0.0</initial_value>
+                </state_interface>
                 <state_interface name="velocity" />
                 <state_interface name="effort" />
@@ -73,15 +79,19 @@
                 </command_interface>
                 <!-- <command_interface name="position"/> -->
-                <state_interface name="position"/>
+                <state_interface name="position">
+                    <initial_value>-0.44</initial_value>
+                </state_interface>
                 <state_interface name="velocity" />
                 <state_interface name="effort" />
             </joint>
             <joint name="plato_joint5">
-                <command_interface name="effort">
+              <command_interface name="effort">
                     <param name="min">-0.06</param>
                     <param name="max">0.06</param>
                 </command_interface>
                 <!-- <command_interface name="position"/> -->
-                <state_interface name="position"/>
+                <state_interface name="position">
+                    <initial_value>-0.44</initial_value>
+                </state_interface>
                 <state_interface name="velocity" />
                 <state_interface name="effort" />
@@ -98,10 +108,12 @@
             </joint>
             <joint name="plato_joint7">
-                <command_interface name="effort">
+               <command_interface name="effort">
                     <param name="min">-0.06</param>
                     <param name="max">0.06</param>
                 </command_interface>
                 <!-- <command_interface name="position"/> -->
-                <state_interface name="position"/>
+                <state_interface name="position">
+                    <initial_value>0.0</initial_value>
+                </state_interface>
                 <state_interface name="velocity" />
                 <state_interface name="effort" />
@@ -113,5 +125,7 @@
                 </command_interface>
                 <!-- <command_interface name="position"/> -->
-                <state_interface name="position"/>
+                <state_interface name="position">
+                    <initial_value>-0.44</initial_value>
+                </state_interface>
                 <state_interface name="velocity" />
                 <state_interface name="effort" />

Commit message: tuing wip

File: plato_description/urdf/plato_hand.urdf.xacro (robot description, xacro)
@@ -5,4 +5,5 @@
     <xacro:arg name="gazebo_classic" default="false" />
     <!-- Set World Frame -->
+    <link name="world"/>
     <!-- Include Xacro -->
     <xacro:include filename="$(find plato_description)/urdf/plato_xacro/plato_hand_description.xacro"/>

File: plato_description/urdf/plato_xacro/plato_hand_description.xacro (robot description, xacro)
@@ -4,9 +4,9 @@
     <!-- if connector_link is defined -->
     <!-- Connector Joint -->
-    <!-- <joint name="plato_connector_joint" type="fixed">
+    <joint name="plato_connector_joint" type="fixed">
         <parent link="${connector_link}"/>
         <child link="plato_base_link"/>
         <origin xyz="${xyz}" rpy="${rpy}"/>
-    </joint> -->
+    </joint>
     <!-- Base Link -->
     <link name="plato_base_link">
