Commit message: plato urdf namespace added

File: plato_description/urdf/plato.urdf.xacro (robot description, xacro)
@@ -2,3 +2,5 @@
 <robot name="plato" xmlns:xacro="http://www.ros.org/wiki/xacro">
     <xacro:include filename="plato_property/plato_hand.xacro"/>
+    <!-- define namespace for plato urdf -->
+    <xacro:plato_hand ns="plato"/>
 </robot>

File: plato_description/urdf/plato_property/plato_hand.xacro (robot description, xacro)
@@ -1,280 +1,18 @@
 <?xml version="1.0"?>
-<robot name="plato" xmlns:xacro="http://www.ros.org/wiki/xacro">
-<link name="base_link"></link>
-<joint name="base_link_to_base" type="fixed">
-<parent link="base_link"/>
-<child link="base" />
-<origin rpy="0.0 0 0" xyz="0 0 0"/>
-</joint>
-<link name="base">
-<visual>
-<origin xyz="0 0 0" rpy="0 -0 0" />
-<geometry>
-<mesh filename="file://$(find plato_description)/meshes/plato/base_visual.stl"/>
-</geometry>
-<material name="base_material">
-<color rgba="0.89999999999999991118 0.89999999999999991118 0.89999999999999991118 1.0"/>
-</material>
-</visual>
-<collision>
-<origin xyz="0 0 0" rpy="0 -0 0" />
-<geometry>
-<mesh filename="file://$(find plato_description)/meshes/plato/base_collision.stl"/>
-</geometry>
-</collision>
-<inertial>
-<origin xyz="0.045493179467456464071 0.00075885043291842098779 -0.00682767319963901477" rpy="0 0 0"/>
-<mass value="0.17280321549697399974" />
-<inertia ixx="0.000124447216717875575" ixy="-2.1184002504334913161e-06"  ixz="-5.2375390643355526047e-06" iyy="0.00022114103876778816297" iyz="2.4145885068302643992e-06" izz="0.00030593848378724351235" />
-</inertial>
-</link>
-<!-- Finger 1 (Thumb) -->
-    <link name="f1_proxbracket">
-    <visual>
-    <origin xyz="0 0 0" rpy="0 -0 0" />
-    <geometry>
-    <mesh filename="file://$(find plato_description)/meshes/plato/proxbracket_visual.stl"/>
-    </geometry>
-    <material name="proxbracket_material">
-    <color rgba="0.9000000000000000222 0.9000000000000000222 0.9000000000000000222 1.0"/>
-    </material>
-    </visual>
-    <collision>
-    <origin xyz="0 0 0" rpy="0 -0 0" />
-    <geometry>
-    <mesh filename="file://$(find plato_description)/meshes/plato/proxbracket_collision.stl"/>
-    </geometry>
-    </collision>
-    <inertial>
-    <origin xyz="-0.0079504685553139688853 -0.013983661603934150613 -0.0095130973110596206421" rpy="0 0 0"/>
-    <mass value="0.12656081824380860379" />
-    <inertia ixx="3.5117165939882084044e-05" ixy="-1.3052140141476243181e-05"  ixz="1.9957519826334250588e-07" iyy="1.7537495218030365739e-05" iyz="-4.9180486622828042765e-07" izz="4.2451494821237482414e-05" />
-    </inertial>
-    </link>
-    <link name="f1_prox">
-    <visual>
-    <origin xyz="0 0 0" rpy="0 -0 0" />
-    <geometry>
-    <mesh filename="file://$(find plato_description)/meshes/plato/prox_visual.stl"/>
-    </geometry>
-    <material name="prox_material">
-    <color rgba="0.9000000000000000222 0.9000000000000000222 0.9000000000000000222 1.0"/>
-    </material>
-    </visual>
-    <collision>
-    <origin xyz="0 0 0" rpy="0 -0 0" />
-    <geometry>
-    <mesh filename="file://$(find plato_description)/meshes/plato/prox_collision.stl"/>
-    </geometry>
-    </collision>
-    <inertial>
-    <origin xyz="0.0020817714488827496026 3.9659156972864230043e-10 -0.015795112278833203096" rpy="0 0 0"/>
-    <mass value="0.069114549940711839104" />
-    <inertia ixx="5.8883565545031638029e-06" ixy="-9.2074790702963013961e-09"  ixz="-1.1640174651110935915e-06" iyy="9.6829622072775541655e-06" iyz="-9.4322537406537712947e-14" izz="9.2871592762525393485e-06" />
-    </inertial>
-    </link>
-    <link name="f1_mid">
-    <visual>
-    <origin xyz="0 0 0" rpy="0 -0 0" />
-    <geometry>
-    <mesh filename="file://$(find plato_description)/meshes/plato/mid_visual.stl"/>
-    </geometry>
-    <material name="mid_material">
-    <color rgba="0.89999999999999991118 0.89999999999999991118 0.89999999999999991118 1.0"/>
-    </material>
-    </visual>
-    <collision>
-    <origin xyz="0 0 0" rpy="0 -0 0" />
-    <geometry>
-    <mesh filename="file://$(find plato_description)/meshes/plato/mid_collision.stl"/>
-    </geometry>
-    </collision>
-    <inertial>
-    <origin xyz="0.02083906332658447616 -0.00066661768468519438241 -0.0023008505382949022595" rpy="0 0 0"/>
-    <mass value="0.0080671501064400220893" />
-    <inertia ixx="2.1185571765449022898e-07" ixy="3.6426243959716221213e-08"  ixz="-1.3233834119316724662e-10" iyy="1.2852102149793263521e-06" iyz="-3.1084190127067859768e-11" izz="1.3237276294092989039e-06" />
-    </inertial>
-    </link>
-    <link name="f1_ee_frame">
-    </link>
-    <joint name="f1_pip_pitch" type="revolute">
-    <origin xyz="0.048000000000000028755 6.9388939039072283776e-18 -0.0026999999999999871325" rpy="6.6672023420374162248e-16 1.5291665303066472343e-16 3.3306690741059185714e-16" />
-    <parent link="f1_prox" />
-    <child link="f1_mid" />
-    <axis xyz="0 0 1"/>
-    <limit effort="1" velocity="20" lower="-1.570796326794896558" upper="1.570796326794896558"/>
-    <joint_properties friction="0.0"/>
+<robot xmlns:xacro="http://www.ros.org/wiki/xacro">
+<xacro:macro name="plato_hand" params="connected_to:='' ns:='plato' rpy:='0 0 0' xyz:='0 0 0' ">
+    <link name="${ns}_base_link"></link>
+        <joint name="${ns}_base_link_to_palm" type="fixed">
+        <parent link="${ns}_base_link"/>
+        <child link="${ns}_palm" />
+        <origin rpy="0.0 0 0" xyz="0 0 0"/>
     </joint>
-    <joint name="f1_mcp_pitch" type="revolute">
-    <origin xyz="-0.0049999999999999697464 -0.028150000000000133249 -0.0098999999999999366285" rpy="-2.8657554781383847745e-16 -1.5707963267948961139 0" />
-    <parent link="f1_proxbracket" />
-    <child link="f1_prox" />
-    <axis xyz="0 0 1"/>
-    <limit effort="1" velocity="20" lower="-2.0943951023931952626" upper="0.52359877559829881566"/>
-    <joint_properties friction="0.0"/>
-    </joint>
-    <joint name="f1_mcp_roll" type="revolute">
-    <origin xyz="0.084500000000000047296 0.029999999999999988481 -0.033000000000000008493" rpy="1.5707963267948958919 -2.5535129566378612263e-15 1.5707963267948938935" />
-    <parent link="base" />
-    <child link="f1_proxbracket" />
-    <axis xyz="0 0 1"/>
-    <limit effort="1" velocity="20" lower="-0.52359877559829881566" upper="1.0471975511965976313"/>
-    <joint_properties friction="0.0"/>
-    </joint>
-    <joint name="f1_ee_joint" type="fixed">
-        <origin xyz="0.05060 0.0 0.0" rpy="-1.5707 0.0 0.0"/>
-        <parent link="f1_mid"/>
-        <child link="f1_ee_frame"/>
-    </joint>
-<!-- Finger 2 (Index) -->
-    <link name="f2_proxbracket">
-    <visual>
-    <origin xyz="0 0 0" rpy="0 -0 0" />
-    <geometry>
-    <mesh filename="file://$(find plato_description)/meshes/plato/proxbracket_2_visual.stl"/>
-    </geometry>
-    <material name="proxbracket_2_material">
-    <color rgba="0.9000000000000000222 0.9000000000000000222 0.9000000000000000222 1.0"/>
-    </material>
-    </visual>
-    <collision>
-    <origin xyz="0 0 0" rpy="0 -0 0" />
-    <geometry>
-    <mesh filename="file://$(find plato_description)/meshes/plato/proxbracket_2_collision.stl"/>
-    </geometry>
-    </collision>
-    <inertial>
-    <origin xyz="-0.0079504685553134692849 -0.01398366160393426337 -0.0095130973110598305437" rpy="0 0 0"/>
-    <mass value="0.12656081824380860379" />
-    <inertia ixx="3.5117165939882477067e-05" ixy="-1.305214014147555539e-05"  ixz="1.9957519826318953702e-07" iyy="1.7537495218029413674e-05" iyz="-4.9180486622862919346e-07" izz="4.2451494821237075838e-05" />
-    </inertial>
-    </link>
-    <link name="f2_prox">
-    <visual>
-    <origin xyz="0 0 0" rpy="0 -0 0" />
-    <geometry>
-    <mesh filename="file://$(find plato_description)/meshes/plato/prox_2_visual.stl"/>
-    </geometry>
-    <material name="prox_2_material">
-    <color rgba="0.9000000000000000222 0.9000000000000000222 0.9000000000000000222 1.0"/>
-    </material>
-    </visual>
-    <collision>
-    <origin xyz="0 0 0" rpy="0 -0 0" />
-    <geometry>
-    <mesh filename="file://$(find plato_description)/meshes/plato/prox_2_collision.stl"/>
-    </geometry>
-    </collision>
-    <inertial>
-    <origin xyz="0.0020817714488827318217 -3.9659157728695655077e-10 0.013295112278833310163" rpy="0 0 0"/>
-    <mass value="0.069114549940711839104" />
-    <inertia ixx="5.8883565545030553827e-06" ixy="9.2074790702970640566e-09"  ixz="1.164017465111112438e-06" iyy="9.6829622072775270604e-06" iyz="-9.4322531718453391682e-14" izz="9.2871592762523818003e-06" />
-    </inertial>
-    </link>
-    <link name="f2_mid">
-    <visual>
-    <origin xyz="0 0 0" rpy="0 -0 0" />
-    <geometry>
-    <mesh filename="file://$(find plato_description)/meshes/plato/mid_2_visual.stl"/>
-    </geometry>
-    <material name="mid_2_material">
-    <color rgba="0.89999999999999991118 0.89999999999999991118 0.89999999999999991118 1.0"/>
-    </material>
-    </visual>
-    <collision>
-    <origin xyz="0 0 0" rpy="0 -0 0" />
-    <geometry>
-    <mesh filename="file://$(find plato_description)/meshes/plato/mid_2_collision.stl"/>
-    </geometry>
-    </collision>
-    <inertial>
-    <origin xyz="0.020839063326584340852 0.00066661768468522192115 -0.0022991494617051059027" rpy="0 0 0"/>
-    <mass value="0.0080671501064400220893" />
-    <inertia ixx="2.1185571765448480268e-07" ixy="-3.6426243959717557937e-08"  ixz="1.3233834119313656339e-10" iyy="1.2852102149793043292e-06" iyz="-3.1084190128060967641e-11" izz="1.3237276294092734929e-06" />
-    </inertial>
-    </link>
-    <link name="f2_ee_frame">
-    </link>
-    <joint name="f2_pip_pitch" type="revolute">
-    <origin xyz="0.047999999999999792832 0 0.0047999999999999813649" rpy="8.673617379890070258e-17 5.7824115865889863811e-17 -1.5021026917775434348e-15" />
-    <parent link="f2_prox" />
-    <child link="f2_mid" />
-    <axis xyz="0 0 1"/>
-    <limit effort="1" velocity="20" lower="-1.570796326794896558" upper="1.570796326794896558"/>
-    <joint_properties friction="0.0"/>
-    </joint>
-    <joint name="f2_mcp_pitch" type="revolute">
-    <origin xyz="-0.0024999999999990307753 -0.028150000000000355294 -0.0099000000000003564316" rpy="-1.570796326794896558 6.9017807609091964755e-16 -1.5707963267948907848" />
-    <parent link="f2_proxbracket" />
-    <child link="f2_prox" />
-    <axis xyz="0 0 1"/>
-    <limit effort="1" velocity="20" lower="-1.570796326794896558" upper="0.785398163397448279"/>
-    <joint_properties friction="0.0"/>
-    </joint>
-    <joint name="f2_mcp_yaw" type="revolute">
-    <origin xyz="0.1000000000000001027 0.029999999999999974604 -0.015000000000000013323" rpy="3.141592653589793116 -1.1714553645825245089e-15 -1.5707963267948998887" />
-    <parent link="base" />
-    <child link="f2_proxbracket" />
-    <axis xyz="0 0 1"/>
-    <limit effort="1" velocity="20" lower="-1.570796326794896558" upper="0.26179938779914940783"/>
-    <joint_properties friction="0.0"/>
-    </joint>
-    <joint name="f2_ee_joint" type="fixed">
-        <origin xyz="0.05060 0.0 0.0" rpy="-1.5707 0.0 0.0"/>
-        <parent link="f2_mid"/>
-        <child link="f2_ee_frame"/>
-    </joint>
-<!-- Finger 3: Middle -->
-    <link name="f3_proxbracket">
-    <visual>
-    <origin xyz="0 0 0" rpy="0 -0 0" />
-    <geometry>
-    <mesh filename="file://$(find plato_description)/meshes/plato/proxbracket_3_visual.stl"/>
-    </geometry>
-    <material name="proxbracket_3_material">
-    <color rgba="0.9000000000000000222 0.9000000000000000222 0.9000000000000000222 1.0"/>
-    </material>
-    </visual>
-    <collision>
-    <origin xyz="0 0 0" rpy="0 -0 0" />
-    <geometry>
-    <mesh filename="file://$(find plato_description)/meshes/plato/proxbracket_3_collision.stl"/>
-    </geometry>
-    </collision>
-    <inertial>
-    <origin xyz="-0.0079504685553140486826 -0.013983661603934124593 -0.0095130973110597195214" rpy="0 0 0"/>
-    <mass value="0.12656081824380860379" />
-    <inertia ixx="3.5117165939882016281e-05" ixy="-1.3052140141476346519e-05"  ixz="1.9957519826327045514e-07" iyy="1.7537495218030480935e-05" iyz="-4.9180486622843035248e-07" izz="4.2451494821237509519e-05" />
-    </inertial>
-    </link>
-    <link name="f3_prox">
+    <link name="${ns}_palm">
         <visual>
         <origin xyz="0 0 0" rpy="0 -0 0" />
         <geometry>
-        <mesh filename="file://$(find plato_description)/meshes/plato/prox_3_visual.stl"/>
+        <mesh filename="file://$(find plato_description)/meshes/plato/base_visual.stl"/>
         </geometry>
-        <material name="prox_3_material">
-        <color rgba="0.9000000000000000222 0.9000000000000000222 0.9000000000000000222 1.0"/>
-        </material>
-        </visual>
-        <collision>
-        <origin xyz="0 0 0" rpy="0 -0 0" />
-        <geometry>
-        <mesh filename="file://$(find plato_description)/meshes/plato/prox_3_collision.stl"/>
-        </geometry>
-        </collision>
-        <inertial>
-        <origin xyz="0.0020817714488827331228 -3.9659157098710811182e-10 0.013295112278833216488" rpy="0 0 0"/>
-        <mass value="0.069114549940711839104" />
-        <inertia ixx="5.8883565545029046108e-06" ixy="9.2074790703146002856e-09"  ixz="1.1640174651110802507e-06" iyy="9.6829622072771458956e-06" iyz="-9.4322525854387518435e-14" izz="9.2871592762523953529e-06" />
-        </inertial>
-    </link>
-    <link name="f3_mid">
-        <visual>
-        <origin xyz="0 0 0" rpy="0 -0 0" />
-        <geometry>
-        <mesh filename="file://$(find plato_description)/meshes/plato/mid_3_visual.stl"/>
-        </geometry>
-        <material name="mid_3_material">
+        <material name="base_material">
         <color rgba="0.89999999999999991118 0.89999999999999991118 0.89999999999999991118 1.0"/>
         </material>
@@ -283,43 +21,307 @@
         <origin xyz="0 0 0" rpy="0 -0 0" />
         <geometry>
-        <mesh filename="file://$(find plato_description)/meshes/plato/mid_3_collision.stl"/>
+        <mesh filename="file://$(find plato_description)/meshes/plato/base_collision.stl"/>
         </geometry>
         </collision>
         <inertial>
-        <origin xyz="0.020839063326584514324 0.00066661768468518982876 -0.0022991494617050798818" rpy="0 0 0"/>
-        <mass value="0.0080671501064400220893" />
-        <inertia ixx="2.1185571765449242598e-07" ixy="-3.6426243959717088098e-08"  ixz="1.3233834119147816966e-10" iyy="1.2852102149793367282e-06" iyz="-3.1084190127996925767e-11" izz="1.3237276294093048331e-06" />
+        <origin xyz="0.045493179467456464071 0.00075885043291842098779 -0.00682767319963901477" rpy="0 0 0"/>
+        <mass value="0.17280321549697399974" />
+        <inertia ixx="0.000124447216717875575" ixy="-2.1184002504334913161e-06"  ixz="-5.2375390643355526047e-06" iyy="0.00022114103876778816297" iyz="2.4145885068302643992e-06" izz="0.00030593848378724351235" />
         </inertial>
     </link>
-    <link name="f3_ee_frame">
-    </link>
-    <joint name="f3_pip_pitch" type="revolute">
-        <origin xyz="0.047999999999998654854 2.0122792321330962295e-16 0.0047999999999999917732" rpy="-1.9081958235950694314e-16 5.7824115816011125546e-17 1.7763568393717672612e-15" />
-        <parent link="f3_prox" />
-        <child link="f3_mid" />
-        <axis xyz="0 0 1"/>
-        <limit effort="1" velocity="20" lower="-1.570796326794896558" upper="1.570796326794896558"/>
-        <joint_properties friction="0.0"/>
-    </joint>
-    <joint name="f3_mcp_pitch" type="revolute">
-        <origin xyz="-0.002500000000000099365 -0.028150000000000077738 -0.0099000000000001291828" rpy="-1.570796326794896558 -3.7816971775725042188e-15 -1.5707963267948943376" />
-        <parent link="f3_proxbracket" />
-        <child link="f3_prox" />
-        <axis xyz="0 0 1"/>
-        <limit effort="1" velocity="20" lower="-1.570796326794896558" upper="0.785398163397448279"/>
-        <joint_properties friction="0.0"/>
-    </joint>
-    <joint name="f3_mcp_yaw" type="revolute">
-        <origin xyz="0.10000000000000000555 -0.029999999999999964195 -0.015000000000000048017" rpy="-3.1415926535897926719 1.1057720720235713428e-16 -1.5707963267948983344" />
-        <parent link="base" />
-        <child link="f3_proxbracket" />
-        <axis xyz="0 0 1"/>
-        <limit effort="1" velocity="20" lower="-0.26179938779914940783" upper="0.785398163397448279"/>
-        <joint_properties friction="0.0"/>
-    </joint>
-    <joint name="f3_ee_joint" type="fixed">
-        <origin xyz="0.05060 0.0 0.0" rpy="-1.5707 0.0 0.0"/>
-        <parent link="f3_mid"/>
-        <child link="f3_ee_frame"/>
-    </joint>
+    <!-- Finger 1 (Thumb) -->
+        <link name="${ns}_f1_proxbracket">
+            <visual>
+            <origin xyz="0 0 0" rpy="0 -0 0" />
+            <geometry>
+            <mesh filename="file://$(find plato_description)/meshes/plato/proxbracket_visual.stl"/>
+            </geometry>
+            <material name="proxbracket_material">
+            <color rgba="0.9000000000000000222 0.9000000000000000222 0.9000000000000000222 1.0"/>
+            </material>
+            </visual>
+            <collision>
+            <origin xyz="0 0 0" rpy="0 -0 0" />
+            <geometry>
+            <mesh filename="file://$(find plato_description)/meshes/plato/proxbracket_collision.stl"/>
+            </geometry>
+            </collision>
+            <inertial>
+            <origin xyz="-0.0079504685553139688853 -0.013983661603934150613 -0.0095130973110596206421" rpy="0 0 0"/>
+            <mass value="0.12656081824380860379" />
+            <inertia ixx="3.5117165939882084044e-05" ixy="-1.3052140141476243181e-05"  ixz="1.9957519826334250588e-07" iyy="1.7537495218030365739e-05" iyz="-4.9180486622828042765e-07" izz="4.2451494821237482414e-05" />
+            </inertial>
+        </link>
+        <link name="${ns}_f1_prox">
+            <visual>
+            <origin xyz="0 0 0" rpy="0 -0 0" />
+            <geometry>
+            <mesh filename="file://$(find plato_description)/meshes/plato/prox_visual.stl"/>
+            </geometry>
+            <material name="prox_material">
+            <color rgba="0.9000000000000000222 0.9000000000000000222 0.9000000000000000222 1.0"/>
+            </material>
+            </visual>
+            <collision>
+            <origin xyz="0 0 0" rpy="0 -0 0" />
+            <geometry>
+            <mesh filename="file://$(find plato_description)/meshes/plato/prox_collision.stl"/>
+            </geometry>
+            </collision>
+            <inertial>
+            <origin xyz="0.0020817714488827496026 3.9659156972864230043e-10 -0.015795112278833203096" rpy="0 0 0"/>
+            <mass value="0.069114549940711839104" />
+            <inertia ixx="5.8883565545031638029e-06" ixy="-9.2074790702963013961e-09"  ixz="-1.1640174651110935915e-06" iyy="9.6829622072775541655e-06" iyz="-9.4322537406537712947e-14" izz="9.2871592762525393485e-06" />
+            </inertial>
+        </link>
+        <link name="${ns}_f1_mid">
+            <visual>
+            <origin xyz="0 0 0" rpy="0 -0 0" />
+            <geometry>
+            <mesh filename="file://$(find plato_description)/meshes/plato/mid_visual.stl"/>
+            </geometry>
+            <material name="mid_material">
+            <color rgba="0.89999999999999991118 0.89999999999999991118 0.89999999999999991118 1.0"/>
+            </material>
+            </visual>
+            <collision>
+            <origin xyz="0 0 0" rpy="0 -0 0" />
+            <geometry>
+            <mesh filename="file://$(find plato_description)/meshes/plato/mid_collision.stl"/>
+            </geometry>
+            </collision>
+            <inertial>
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
Commit message: arm and hand connected

File: plato_description/urdf/plato.urdf.xacro (robot description, xacro)
@@ -1,6 +1,26 @@
 <?xml version="1.0"?>
 <robot name="plato" xmlns:xacro="http://www.ros.org/wiki/xacro">
-    <xacro:include filename="plato_property/plato_hand.xacro"/>
-    <!-- define namespace for plato urdf -->
-    <xacro:plato_hand ns="plato"/>
+    <!-- Include Optimo Arm and PLATO Hand Xacro -->
+    <xacro:include filename="$(find optimo_description)/urdf/optimo_xacro/optimo_arm.xacro"/>
+    <xacro:include filename="$(find plato_description)/urdf/plato_xacro/plato_hand.xacro"/>
+    <!-- Set Namespace for the Optimo Arm -->
+    <xacro:property name="arm_ns" value="optimo" />
+    <xacro:optimo_arm ns = "${arm_ns}"/>
+    <!-- Set Namespace for the PLATO Hand -->
+    <xacro:property name="hand_ns" value="plato" />
+    <xacro:plato_hand ns = "${hand_ns}"/>
+    <!-- Set World Frame for Gazebo -->
+    <link name="world"/>
+    <!-- Connect the Optimo to the World-->
+    <joint name="world_joint" type="fixed">
+        <parent link="world"/>
+        <child link="${arm_ns}_base_link"/>
+        <origin xyz="0 0 0" rpy="0 0 0"/>
+    </joint>
+    <!-- Connect PLATO Hand to Optimo Arm -->
+    <joint name="hand_arm_joint" type="fixed">
+        <parent link="${arm_ns}_link7_passive"/>
+        <child link="${hand_ns}_base_link"/>
+        <origin xyz="0 0.15 0" rpy="0 0 1.57"/>
+    </joint>
 </robot>

Commit message: 500 Hz comm at AHG

File: plato_description/urdf/plato.urdf.xacro (robot description, xacro)
@@ -3,5 +3,4 @@
   <xacro:arg name="fake_hardware" default="false"/>
   <xacro:arg name="zeroing" default="false"/>
-  <xacro:arg name="direct_tx_inter_frame_gap_us" default="100"/>
   <xacro:include filename="$(find plato_description)/urdf/xacro/plato_description.xacro"/>
   <xacro:include filename="$(find plato_description)/urdf/ros2_control/plato.ros2_control.xacro"/>
@@ -10,5 +9,4 @@
     name="plato_ros2_control"
     fake_hardware="$(arg fake_hardware)"
-    zeroing="$(arg zeroing)"
-    direct_tx_inter_frame_gap_us="$(arg direct_tx_inter_frame_gap_us)"/>
+    zeroing="$(arg zeroing)"/>
 </robot>

File: plato_description/urdf/ros2_control/plato.ros2_control.xacro (robot description, xacro)
@@ -1,6 +1,9 @@
 <?xml version="0.06.0"?>
 <robot xmlns:xacro="http://www.ros.org/wiki/xacro">
-  <xacro:macro name="plato_ros2_control" params="name fake_hardware='false' zeroing='false' direct_tx_inter_frame_gap_us='100'">
+  <xacro:macro name="plato_ros2_control" params="name fake_hardware='false' zeroing='false'">
     <xacro:property name="use_mock" value="${fake_hardware == 'true' or fake_hardware == 'True' or fake_hardware == '1' or fake_hardware == 1 or fake_hardware == True}"/>
+    <xacro:property
+      name="hardware_config"
+      value="${xacro.load_yaml('$(find plato_hardware_interface)/config/plato_hardware.yaml')}"/>
     <ros2_control name="${name}" type="system">
       <hardware>
@@ -11,5 +14,5 @@
           <plugin>plato_hardware_interface/PlatoHardware</plugin>
           <param name="zeroing">${zeroing}</param>
-          <param name="direct_tx_inter_frame_gap_us">${direct_tx_inter_frame_gap_us}</param>
+          <param name="direct_tx_inter_frame_gap_us">${hardware_config['direct_tx_inter_frame_gap_us']}</param>
         </xacro:unless>
       </hardware>
