Commit message: code simplification

File: plato_description/urdf/aristo.urdf.xacro (robot description, xacro)
@@ -1,4 +1,7 @@
 <?xml version="1.0"?>
 <robot name="aristo_hand" xmlns:xacro="http://www.ros.org/wiki/xacro">
+  <xacro:arg name="fake_hardware" default="false"/>
+  <xacro:arg name="zeroing" default="false"/>
+  <xacro:arg name="actuator_config_yaml_path" default=""/>
   <!-- Root link for TF tree -->
   <link name="base_link"/>
@@ -8,4 +11,8 @@
   <!-- Instantiate geometry/tree and ros2_control -->
   <xacro:aristo_description connector_link="base_link" xyz="0 0 0" rpy="0 0 0"/>
-  <xacro:aristo_ros2_control name="aristo_ros2_control"/>
+  <xacro:aristo_ros2_control
+    name="aristo_ros2_control"
+    fake_hardware="$(arg fake_hardware)"
+    zeroing="$(arg zeroing)"
+    actuator_config_yaml_path="$(arg actuator_config_yaml_path)"/>
 </robot>

File: plato_description/urdf/ros2_control/aristo.ros2_control.xacro (robot description, xacro)
@@ -1,5 +1,5 @@
 <?xml version="0.06.0"?>
 <robot xmlns:xacro="http://www.ros.org/wiki/xacro">
-    <xacro:macro name="aristo_ros2_control" params="name fake_hardware='false'">
+    <xacro:macro name="aristo_ros2_control" params="name fake_hardware='false' zeroing='false' actuator_config_yaml_path=''">
         <!-- Normalize fake_hardware values so callers can pass true/False, 1/0, or strings -->
         <xacro:property name="use_mock" value="${fake_hardware == 'true' or fake_hardware == 'True' or fake_hardware == '1' or fake_hardware == 1 or fake_hardware == True}"/>
@@ -13,4 +13,8 @@
                 <xacro:unless value="${use_mock}">
                     <plugin>aristo_hardware_interface/AristoHardware</plugin>
+                    <param name="zeroing">${zeroing}</param>
+                    <xacro:if value="${actuator_config_yaml_path != ''}">
+                        <param name="actuator_config_yaml_path">${actuator_config_yaml_path}</param>
+                    </xacro:if>
                 </xacro:unless>
             </hardware>

Commit message: activation table

File: plato_description/urdf/aristo.urdf.xacro (robot description, xacro)
@@ -4,4 +4,5 @@
   <xacro:arg name="zeroing" default="false"/>
   <xacro:arg name="actuator_config_yaml_path" default=""/>
+  <xacro:arg name="activation_summary_path" default="/tmp/aristo_activation_summary.txt"/>
   <!-- Root link for TF tree -->
   <link name="base_link"/>
@@ -13,6 +14,7 @@
   <xacro:aristo_ros2_control
     name="aristo_ros2_control"
-    fake_hardware="$(arg fake_hardware)"
-    zeroing="$(arg zeroing)"
-    actuator_config_yaml_path="$(arg actuator_config_yaml_path)"/>
+	    fake_hardware="$(arg fake_hardware)"
+	    zeroing="$(arg zeroing)"
+	    actuator_config_yaml_path="$(arg actuator_config_yaml_path)"
+	    activation_summary_path="$(arg activation_summary_path)"/>
 </robot>

File: plato_description/urdf/ros2_control/aristo.ros2_control.xacro (robot description, xacro)
@@ -1,5 +1,5 @@
 <?xml version="0.06.0"?>
 <robot xmlns:xacro="http://www.ros.org/wiki/xacro">
-    <xacro:macro name="aristo_ros2_control" params="name fake_hardware='false' zeroing='false' actuator_config_yaml_path=''">
+    <xacro:macro name="aristo_ros2_control" params="name fake_hardware='false' zeroing='false' actuator_config_yaml_path='' activation_summary_path='/tmp/aristo_activation_summary.txt'">
         <!-- Normalize fake_hardware values so callers can pass true/False, 1/0, or strings -->
         <xacro:property name="use_mock" value="${fake_hardware == 'true' or fake_hardware == 'True' or fake_hardware == '1' or fake_hardware == 1 or fake_hardware == True}"/>
@@ -12,9 +12,10 @@
                 </xacro:if>
                 <xacro:unless value="${use_mock}">
-                    <plugin>aristo_hardware_interface/AristoHardware</plugin>
-                    <param name="zeroing">${zeroing}</param>
-                    <xacro:if value="${actuator_config_yaml_path != ''}">
-                        <param name="actuator_config_yaml_path">${actuator_config_yaml_path}</param>
-                    </xacro:if>
+	                    <plugin>aristo_hardware_interface/AristoHardware</plugin>
+	                    <param name="zeroing">${zeroing}</param>
+	                    <param name="activation_summary_path">${activation_summary_path}</param>
+	                    <xacro:if value="${actuator_config_yaml_path != ''}">
+	                        <param name="actuator_config_yaml_path">${actuator_config_yaml_path}</param>
+	                    </xacro:if>
                 </xacro:unless>
             </hardware>

Commit message: wip

File: plato_description/urdf/aristo.urdf.xacro (robot description, xacro)
@@ -4,5 +4,4 @@
   <xacro:arg name="zeroing" default="false"/>
   <xacro:arg name="actuator_config_yaml_path" default=""/>
-  <xacro:arg name="activation_summary_path" default="/tmp/aristo_activation_summary.txt"/>
   <!-- Root link for TF tree -->
   <link name="base_link"/>
@@ -16,5 +15,4 @@
 	    fake_hardware="$(arg fake_hardware)"
 	    zeroing="$(arg zeroing)"
-	    actuator_config_yaml_path="$(arg actuator_config_yaml_path)"
-	    activation_summary_path="$(arg activation_summary_path)"/>
+	    actuator_config_yaml_path="$(arg actuator_config_yaml_path)"/>
 </robot>

File: plato_description/urdf/ros2_control/aristo.ros2_control.xacro (robot description, xacro)
@@ -1,5 +1,5 @@
 <?xml version="0.06.0"?>
 <robot xmlns:xacro="http://www.ros.org/wiki/xacro">
-    <xacro:macro name="aristo_ros2_control" params="name fake_hardware='false' zeroing='false' actuator_config_yaml_path='' activation_summary_path='/tmp/aristo_activation_summary.txt'">
+    <xacro:macro name="aristo_ros2_control" params="name fake_hardware='false' zeroing='false' actuator_config_yaml_path=''">
         <!-- Normalize fake_hardware values so callers can pass true/False, 1/0, or strings -->
         <xacro:property name="use_mock" value="${fake_hardware == 'true' or fake_hardware == 'True' or fake_hardware == '1' or fake_hardware == 1 or fake_hardware == True}"/>
@@ -14,5 +14,4 @@
 	                    <plugin>aristo_hardware_interface/AristoHardware</plugin>
 	                    <param name="zeroing">${zeroing}</param>
-	                    <param name="activation_summary_path">${activation_summary_path}</param>
 	                    <xacro:if value="${actuator_config_yaml_path != ''}">
 	                        <param name="actuator_config_yaml_path">${actuator_config_yaml_path}</param>
