Commit message: wip

File: plato_description/urdf/aristo.urdf.xacro (robot description, xacro)
@@ -4,9 +4,11 @@
   <xacro:arg name="zeroing" default="false"/>
   <xacro:arg name="actuator_config_yaml_path" default=""/>
+  <xacro:arg name="can_backend" default="pcan"/>
+  <xacro:arg name="socketcan_interface" default="can0"/>
   <!-- Root link for TF tree -->
   <link name="base_link"/>
   <!-- Includes -->
-    <xacro:include filename="$(find plato_description)/urdf/xacro/aristo_description.xacro"/>
-    <xacro:include filename="$(find plato_description)/urdf/ros2_control/aristo.ros2_control.xacro"/>
+    <xacro:include filename="xacro/aristo_description.xacro"/>
+    <xacro:include filename="ros2_control/aristo.ros2_control.xacro"/>
   <!-- Instantiate geometry/tree and ros2_control -->
   <xacro:aristo_description connector_link="base_link" xyz="0 0 0" rpy="0 0 0"/>
@@ -15,4 +17,6 @@
 	    fake_hardware="$(arg fake_hardware)"
 	    zeroing="$(arg zeroing)"
-	    actuator_config_yaml_path="$(arg actuator_config_yaml_path)"/>
+	    actuator_config_yaml_path="$(arg actuator_config_yaml_path)"
+	    can_backend="$(arg can_backend)"
+	    socketcan_interface="$(arg socketcan_interface)"/>
 </robot>

File: plato_description/urdf/plato.urdf.xacro (robot description, xacro)
@@ -3,4 +3,6 @@
   <xacro:arg name="fake_hardware" default="false"/>
   <xacro:arg name="zeroing" default="false"/>
+  <xacro:arg name="can_backend" default="pcan"/>
+  <xacro:arg name="socketcan_interface" default="can0"/>
   <xacro:include filename="$(find plato_description)/urdf/xacro/plato_description.xacro"/>
   <xacro:include filename="$(find plato_description)/urdf/ros2_control/plato.ros2_control.xacro"/>
@@ -9,4 +11,6 @@
     name="plato_ros2_control"
     fake_hardware="$(arg fake_hardware)"
-    zeroing="$(arg zeroing)"/>
+    zeroing="$(arg zeroing)"
+    can_backend="$(arg can_backend)"
+    socketcan_interface="$(arg socketcan_interface)"/>
 </robot>

File: plato_description/urdf/plato_naritouch.urdf.xacro (robot description, xacro)
@@ -3,4 +3,6 @@
   <xacro:arg name="fake_hardware" default="false"/>
   <xacro:arg name="zeroing" default="false"/>
+  <xacro:arg name="can_backend" default="pcan"/>
+  <xacro:arg name="socketcan_interface" default="can0"/>
   <xacro:include filename="xacro/plato_naritouch_description.xacro"/>
   <xacro:include filename="ros2_control/plato.ros2_control.xacro"/>
@@ -9,4 +11,6 @@
     name="plato_ros2_control"
     fake_hardware="$(arg fake_hardware)"
-    zeroing="$(arg zeroing)"/>
+    zeroing="$(arg zeroing)"
+    can_backend="$(arg can_backend)"
+    socketcan_interface="$(arg socketcan_interface)"/>
 </robot>

File: plato_description/urdf/ros2_control/aristo.ros2_control.xacro (robot description, xacro)
@@ -1,5 +1,7 @@
 <?xml version="0.06.0"?>
 <robot xmlns:xacro="http://www.ros.org/wiki/xacro">
-    <xacro:macro name="aristo_ros2_control" params="name fake_hardware='false' zeroing='false' actuator_config_yaml_path=''">
+    <xacro:macro
+        name="aristo_ros2_control"
+        params="name fake_hardware='false' zeroing='false' actuator_config_yaml_path='' can_backend='pcan' socketcan_interface='can0'">
         <!-- Normalize fake_hardware values so callers can pass true/False, 1/0, or strings -->
         <xacro:property name="use_mock" value="${fake_hardware == 'true' or fake_hardware == 'True' or fake_hardware == '1' or fake_hardware == 1 or fake_hardware == True}"/>
@@ -14,4 +16,6 @@
 	                    <plugin>aristo_hardware_interface/AristoHardware</plugin>
 	                    <param name="zeroing">${zeroing}</param>
+	                    <param name="can_backend">${can_backend}</param>
+	                    <param name="socketcan_interface">${socketcan_interface}</param>
 	                    <xacro:if value="${actuator_config_yaml_path != ''}">
 	                        <param name="actuator_config_yaml_path">${actuator_config_yaml_path}</param>

File: plato_description/urdf/ros2_control/plato.ros2_control.xacro (robot description, xacro)
@@ -1,5 +1,7 @@
 <?xml version="0.06.0"?>
 <robot xmlns:xacro="http://www.ros.org/wiki/xacro">
-  <xacro:macro name="plato_ros2_control" params="name fake_hardware='false' zeroing='false'">
+  <xacro:macro
+    name="plato_ros2_control"
+    params="name fake_hardware='false' zeroing='false' can_backend='pcan' socketcan_interface='can0'">
     <xacro:property name="use_mock" value="${fake_hardware == 'true' or fake_hardware == 'True' or fake_hardware == '1' or fake_hardware == 1 or fake_hardware == True}"/>
     <xacro:property
@@ -14,4 +16,6 @@
           <plugin>plato_hardware_interface/PlatoHardware</plugin>
           <param name="zeroing">${zeroing}</param>
+          <param name="can_backend">${can_backend}</param>
+          <param name="socketcan_interface">${socketcan_interface}</param>
           <param name="direct_tx_inter_frame_gap_us">${hardware_config['direct_tx_inter_frame_gap_us']}</param>
           <param name="servo_stiffness_scale">${hardware_config['servo_stiffness_scale']}</param>
