Commit message: wip

File: optiman_description/urdf/optimo.urdf.xacro (robot description, xacro)
@@ -9,5 +9,5 @@
     <link name="world"/>
     <!-- Pedestal -->
-    <xacro:pedestal connector_link="world" />
+    <xacro:pedestal_description connector_link="world" />
     <!-- Optimo Arm -->
     <xacro:optimo_description connector_link="stand_link"/>

File: optiman_description/urdf/optimo_xacro/optimo_description.xacro (robot description, xacro)
@@ -16,5 +16,5 @@
         <parent link="${connector_link}"/>
         <child link="optimo_base_link"/>
-        <origin xyz="0 0 0" rpy="0 0 0"/>
+        <origin xyz="0 0 0.5" rpy="0 0 0"/>
     </joint>
     <!-- Optimo Robot Arm Links -->
@@ -29,11 +29,11 @@
         <visual>
             <geometry>
-                <mesh filename="file://$(find optimo_description)/meshes/link0.stl"/>
-            </geometry>
-            <material name="blue"/>
-        </visual>
-        <collision>
-            <geometry>
-                <mesh filename="file://$(find optimo_description)/meshes/col0.stl"/>
+                <mesh filename="file://$(find optiman_description)/meshes/link0.stl"/>
+            </geometry>
+            <material name="blue"/>
+        </visual>
+        <collision>
+            <geometry>
+                <mesh filename="file://$(find optiman_description)/meshes/col0.stl"/>
             </geometry>
         </collision>
@@ -48,11 +48,11 @@
         <visual>
             <geometry>
-                <mesh filename="file://$(find optimo_description)/meshes/link1.stl"/>
-            </geometry>
-            <material name="white"/>
-        </visual>
-        <collision>
-            <geometry>
-                <mesh filename="file://$(find optimo_description)/meshes/col1.stl"/>
+                <mesh filename="file://$(find optiman_description)/meshes/link1.stl"/>
+            </geometry>
+            <material name="white"/>
+        </visual>
+        <collision>
+            <geometry>
+                <mesh filename="file://$(find optiman_description)/meshes/col1.stl"/>
             </geometry>
         </collision>
@@ -67,11 +67,11 @@
         <visual>
             <geometry>
-                <mesh filename="file://$(find optimo_description)/meshes/link2.stl"/>
-            </geometry>
-            <material name="blue"/>
-        </visual>
-        <collision>
-            <geometry>
-                <mesh filename="file://$(find optimo_description)/meshes/col2.stl"/>
+                <mesh filename="file://$(find optiman_description)/meshes/link2.stl"/>
+            </geometry>
+            <material name="blue"/>
+        </visual>
+        <collision>
+            <geometry>
+                <mesh filename="file://$(find optiman_description)/meshes/col2.stl"/>
             </geometry>
         </collision>
@@ -86,11 +86,11 @@
         <visual>
             <geometry>
-                <mesh filename="file://$(find optimo_description)/meshes/link3.stl"/>
-            </geometry>
-            <material name="white"/>
-        </visual>
-        <collision>
-            <geometry>
-                <mesh filename="file://$(find optimo_description)/meshes/col3.stl"/>
+                <mesh filename="file://$(find optiman_description)/meshes/link3.stl"/>
+            </geometry>
+            <material name="white"/>
+        </visual>
+        <collision>
+            <geometry>
+                <mesh filename="file://$(find optiman_description)/meshes/col3.stl"/>
             </geometry>
         </collision>
@@ -106,11 +106,11 @@
         <visual>
             <geometry>
-                <mesh filename="file://$(find optimo_description)/meshes/link4.stl"/>
-            </geometry>
-            <material name="blue"/>
-        </visual>
-        <collision>
-            <geometry>
-                <mesh filename="file://$(find optimo_description)/meshes/col4.stl"/>
+                <mesh filename="file://$(find optiman_description)/meshes/link4.stl"/>
+            </geometry>
+            <material name="blue"/>
+        </visual>
+        <collision>
+            <geometry>
+                <mesh filename="file://$(find optiman_description)/meshes/col4.stl"/>
             </geometry>
         </collision>
@@ -125,11 +125,11 @@
         <visual>
             <geometry>
-                <mesh filename="file://$(find optimo_description)/meshes/link5.stl"/>
-            </geometry>
-            <material name="white"/>
-        </visual>
-        <collision>
-            <geometry>
-                <mesh filename="file://$(find optimo_description)/meshes/col5.stl"/>
+                <mesh filename="file://$(find optiman_description)/meshes/link5.stl"/>
+            </geometry>
+            <material name="white"/>
+        </visual>
+        <collision>
+            <geometry>
+                <mesh filename="file://$(find optiman_description)/meshes/col5.stl"/>
             </geometry>
         </collision>
@@ -144,11 +144,11 @@
         <visual>
             <geometry>
-                <mesh filename="file://$(find optimo_description)/meshes/link6.stl"/>
-            </geometry>
-            <material name="blue"/>
-        </visual>
-        <collision>
-            <geometry>
-                <mesh filename="file://$(find optimo_description)/meshes/col6.stl"/>
+                <mesh filename="file://$(find optiman_description)/meshes/link6.stl"/>
+            </geometry>
+            <material name="blue"/>
+        </visual>
+        <collision>
+            <geometry>
+                <mesh filename="file://$(find optiman_description)/meshes/col6.stl"/>
             </geometry>
         </collision>
@@ -163,11 +163,11 @@
         <visual>
             <geometry>
-                <mesh filename="file://$(find optimo_description)/meshes/link7.stl"/>
-            </geometry>
-            <material name="white"/>
-        </visual>
-        <collision>
-            <geometry>
-                <mesh filename="file://$(find optimo_description)/meshes/col7.stl"/>
+                <mesh filename="file://$(find optiman_description)/meshes/link7.stl"/>
+            </geometry>
+            <material name="white"/>
+        </visual>
+        <collision>
+            <geometry>
+                <mesh filename="file://$(find optiman_description)/meshes/col7.stl"/>
             </geometry>
         </collision>

File: optiman_description/urdf/optimo_xacro/pedestal.xacro (robot description, xacro)
@@ -4,5 +4,5 @@
     <link name="stand_link">
         <visual>
-            <origin xyz="0 0 -0.5" rpy="0 0 0"/>
+            <origin xyz="0 0 0" rpy="0 0 0"/>
             <geometry>
                 <box size="0.3 0.3 1"/>
@@ -11,5 +11,5 @@
         </visual>
         <collision>
-            <origin xyz="0 0 -0.5" rpy="0 0 0"/>
+            <origin xyz="0 0 0" rpy="0 0 0"/>
             <geometry>
                 <box size="0.3 0.3 1"/>

File: plato_description/urdf/plato.urdf (robot description, URDF)
Before this commit: robot plato_hand, 13 links, 12 joints
Links:
- link plato_base_link: geometry collision mesh filename=file:///home/dk/workspaces/plato_ws/install/plato_descripti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; visual mesh filename=file:///home/dk/workspaces/plato_ws/install/plato_descripti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
- link plato_bracket_1: geometry collision mesh filename=file:///home/dk/workspaces/plato_ws/install/plato_descripti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; visual mesh filename=file:///home/dk/workspaces/plato_ws/install/plato_descripti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
- link plato_bracket_2: geometry collision mesh filename=file:///home/dk/workspaces/plato_ws/install/plato_descripti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; visual mesh filename=file:///home/dk/workspaces/plato_ws/install/plato_descripti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
- link plato_bracket_3: geometry collision mesh filename=file:///home/dk/workspaces/plato_ws/install/plato_descripti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; visual mesh filename=file:///home/dk/workspaces/plato_ws/install/plato_descripti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
- link plato_distal_1: geometry collision mesh filename=file:///home/dk/workspaces/plato_ws/install/plato_descripti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; visual mesh filename=file:///home/dk/workspaces/plato_ws/install/plato_descripti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
- link plato_distal_2: geometry collision mesh filename=file:///home/dk/workspaces/plato_ws/install/plato_descripti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; visual mesh filename=file:///home/dk/workspaces/plato_ws/install/plato_descripti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
- link plato_distal_3: geometry collision mesh filename=file:///home/dk/workspaces/plato_ws/install/plato_descripti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; visual mesh filename=file:///home/dk/workspaces/plato_ws/install/plato_descripti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
- link plato_proximal_1: geometry collision mesh filename=file:///home/dk/workspaces/plato_ws/install/plato_descripti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; visual mesh filename=file:///home/dk/workspaces/plato_ws/install/plato_descripti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
- link plato_proximal_2: geometry collision mesh filename=file:///home/dk/workspaces/plato_ws/install/plato_descripti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; visual mesh filename=file:///home/dk/workspaces/plato_ws/install/plato_descripti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
- link plato_proximal_3: geometry collision mesh filename=file:///home/dk/workspaces/plato_ws/install/plato_descripti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; visual mesh filename=file:///home/dk/workspaces/plato_ws/install/plato_descripti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
Joints:
- added joint plato_connector_joint: type fixed, parent world, child plato_base_link, origin xyz=0 0 0 rpy=0 0 0
- joint plato_joint2: limit lower=-0.34906585039886589561 upper=1.570796326794896558 effort=0.06 velocity=0.0872665 -> lower=0.0 upper=1.570796326794896558 effort=0.06 velocity=0.0872665
- joint plato_joint5: limit lower=-1.570796326794896558 upper=0.34906585039886589561 effort=0.06 velocity=0.0872665 -> lower=-1.570796326794896558 upper=0.0 effort=0.06 velocity=0.0872665
- joint plato_joint8: limit lower=-1.570796326794896558 upper=0.34906585039886589561 effort=0.06 velocity=0.0872665 -> lower=-1.570796326794896558 upper=0.0 effort=0.06 velocity=0.0872665
