Commit message: wip

File: optiman_description/urdf/optimo_xacro/optimo_description.xacro (robot description, xacro)
@@ -16,5 +16,5 @@
         <parent link="${connector_link}"/>
         <child link="optimo_base_link"/>
-        <origin xyz="0 0 0.5" rpy="0 0 0"/>
+        <origin xyz="0 0 0.5" rpy="0.785 0 0"/>
     </joint>
     <!-- Optimo Robot Arm Links -->
