Commit message: joint state working

File: plato2_description/urdf/ros2_control/plato2.ros2_control.xacro (robot description, xacro)
@@ -19,4 +19,10 @@
                 <state_interface name="effort"/>
             </joint>
+            <joint name="joint4">
+                <command_interface name="position"/>
+                <state_interface name="position"/>
+                <state_interface name="velocity"/>
+                <state_interface name="effort"/>
+            </joint>
             <joint name="joint3">
                 <command_interface name="position"/>
@@ -25,5 +31,5 @@
                 <state_interface name="effort"/>
             </joint>
-            <joint name="joint4">
+            <joint name="joint6">
                 <command_interface name="position"/>
                 <state_interface name="position"/>
@@ -37,5 +43,5 @@
                 <state_interface name="effort"/>
             </joint>
-            <joint name="joint6">
+            <joint name="joint8">
                 <command_interface name="position"/>
                 <state_interface name="position"/>
@@ -49,10 +55,4 @@
                 <state_interface name="effort"/>
             </joint>
-            <joint name="joint8">
-                <command_interface name="position"/>
-                <state_interface name="position"/>
-                <state_interface name="velocity"/>
-                <state_interface name="effort"/>
-            </joint>
         </ros2_control>
   </xacro:macro>

File: plato2_description/urdf/xacro/plato2_description.xacro (robot description, xacro)
@@ -126,36 +126,4 @@
 <axis xyz="0 0 0"/>
 </joint>
-<joint name="joint4" type="revolute">
-<origin xyz="0.060000000000000011657 -1.3877787807814456755e-17 -6.9388939039072283776e-18" rpy="1.9153167705881153685e-14 6.1331864267087110065e-15 -3.141592653589788231" />
-<parent link="thumb_proximal" />
-<child link="thumb_distal" />
-<axis xyz="0 0 1"/>
-<limit effort="0.8499999999999999778" velocity="1.5700000000000000622" lower="-2.0943951023931952626" upper="0"/>
-<joint_properties friction="0.0"/>
-</joint>
-<joint name="joint3" type="revolute">
-<origin xyz="-0.024997917591194747378 -0.011999999478458957258 -0.023999999999999993561" rpy="-1.5707963267948970021 -7.7297547565167041677e-16 -3.1415926535897908956" />
-<parent link="thumb_actuators" />
-<child link="thumb_proximal" />
-<axis xyz="0 0 1"/>
-<limit effort="0.8499999999999999778" velocity="1.5700000000000000622" lower="-1.0471975511965976313" upper="1.0471975511965976313"/>
-<joint_properties friction="0.0"/>
-</joint>
-<joint name="joint2" type="revolute">
-<origin xyz="0.058249999999999593769 5.5511151231257827021e-16 0.03224999999999998701" rpy="-3.1415926535897891192 1.5707963267948927832 0" />
-<parent link="thumb_metacarpal" />
-<child link="thumb_actuators" />
-<axis xyz="0 0 1"/>
-<limit effort="0.8499999999999999778" velocity="1.5700000000000000622" lower="-0.785398163397448279" upper="0.785398163397448279"/>
-<joint_properties friction="0.0"/>
-</joint>
-<joint name="joint1" type="revolute">
-<origin xyz="0.01149999999999984715 0.039000000000000659139 -0.015849999999999926648" rpy="-1.3045120539345319165e-15 1.5707963267948643615 0" />
-<parent link="base_link" />
-<child link="thumb_metacarpal" />
-<axis xyz="0 0 1"/>
-<limit effort="0.8499999999999999778" velocity="1.5700000000000000622" lower="-0.34906585039886589561" upper="1.2217304763960306069"/>
-<joint_properties friction="0.0"/>
-</joint>
 <link name="index_proximal">
 <visual>
@@ -215,20 +183,4 @@
 <axis xyz="0 0 0"/>
 </joint>
-<joint name="joint6" type="revolute">
-<origin xyz="0.060000000000000011657 -3.4694469519536141888e-18 0" rpy="-2.1461027329066007583e-16 3.0473921289930194632e-15 3.141592653589793116" />
-<parent link="index_proximal" />
-<child link="index_distal" />
-<axis xyz="0 0 1"/>
-<limit effort="0.8499999999999999778" velocity="1.5700000000000000622" lower="0" upper="2.0943951023931952626"/>
-<joint_properties friction="0.0"/>
-</joint>
-<joint name="joint5" type="revolute">
-<origin xyz="0.11342115258546792145 0.041187262013853524756 0.025999851934806916809" rpy="-1.57079632679489678 2.2482016248662969818e-15 -1.850249261987616476e-15" />
-<parent link="base_link" />
-<child link="index_proximal" />
-<axis xyz="0 0 1"/>
-<limit effort="0.8499999999999999778" velocity="1.5700000000000000622" lower="-1.0471975511965976313" upper="1.0471975511965976313"/>
-<joint_properties friction="0.0"/>
-</joint>
 <link name="middle_proximal">
 <visual>
@@ -288,4 +240,60 @@
 <axis xyz="0 0 0"/>
 </joint>
+<joint name="joint1" type="revolute">
+<origin xyz="0.01149999999999984715 0.039000000000000659139 -0.015849999999999926648" rpy="-1.3045120539345319165e-15 1.5707963267948643615 0" />
+<parent link="base_link" />
+<child link="thumb_metacarpal" />
+<axis xyz="0 0 1"/>
+<limit effort="0.8499999999999999778" velocity="1.5700000000000000622" lower="-0.34906585039886589561" upper="1.2217304763960306069"/>
+<joint_properties friction="0.0"/>
+</joint>
+<joint name="joint2" type="revolute">
+<origin xyz="0.058249999999999593769 5.5511151231257827021e-16 0.03224999999999998701" rpy="-3.1415926535897891192 1.5707963267948927832 0" />
+<parent link="thumb_metacarpal" />
+<child link="thumb_actuators" />
+<axis xyz="0 0 1"/>
+<limit effort="0.8499999999999999778" velocity="1.5700000000000000622" lower="-0.785398163397448279" upper="0.785398163397448279"/>
+<joint_properties friction="0.0"/>
+</joint>
+<joint name="joint3" type="revolute">
+<origin xyz="-0.024997917591194747378 -0.011999999478458957258 -0.023999999999999993561" rpy="-1.5707963267948970021 -7.7297547565167041677e-16 -3.1415926535897908956" />
+<parent link="thumb_actuators" />
+<child link="thumb_proximal" />
+<axis xyz="0 0 1"/>
+<limit effort="0.8499999999999999778" velocity="1.5700000000000000622" lower="-1.0471975511965976313" upper="1.0471975511965976313"/>
+<joint_properties friction="0.0"/>
+</joint>
+<joint name="joint4" type="revolute">
+<origin xyz="0.060000000000000011657 -1.3877787807814456755e-17 -6.9388939039072283776e-18" rpy="1.9153167705881153685e-14 6.1331864267087110065e-15 -3.141592653589788231" />
+<parent link="thumb_proximal" />
+<child link="thumb_distal" />
+<axis xyz="0 0 1"/>
+<limit effort="0.8499999999999999778" velocity="1.5700000000000000622" lower="-2.0943951023931952626" upper="0"/>
+<joint_properties friction="0.0"/>
+</joint>
+<joint name="joint5" type="revolute">
+<origin xyz="0.11342115258546792145 0.041187262013853524756 0.025999851934806916809" rpy="-1.57079632679489678 2.2482016248662969818e-15 -1.850249261987616476e-15" />
+<parent link="base_link" />
+<child link="index_proximal" />
+<axis xyz="0 0 1"/>
+<limit effort="0.8499999999999999778" velocity="1.5700000000000000622" lower="-1.0471975511965976313" upper="1.0471975511965976313"/>
+<joint_properties friction="0.0"/>
+</joint>
+<joint name="joint6" type="revolute">
+<origin xyz="0.060000000000000011657 -3.4694469519536141888e-18 0" rpy="-2.1461027329066007583e-16 3.0473921289930194632e-15 3.141592653589793116" />
+<parent link="index_proximal" />
+<child link="index_distal" />
+<axis xyz="0 0 1"/>
+<limit effort="0.8499999999999999778" velocity="1.5700000000000000622" lower="0" upper="2.0943951023931952626"/>
+<joint_properties friction="0.0"/>
+</joint>
+<joint name="joint7" type="revolute">
+<origin xyz="0.11349791759135398339 -0.036249999478459471458 0.026000000000000023093" rpy="-1.570796326794896336 2.4702462297869142187e-15 1.5081753875048004426e-15" />
+<parent link="base_link" />
+<child link="middle_proximal" />
+<axis xyz="0 0 1"/>
+<limit effort="0.8499999999999999778" velocity="1.5700000000000000622" lower="-1.0471975511965976313" upper="1.0471975511965976313"/>
+<joint_properties friction="0.0"/>
+</joint>
 <joint name="joint8" type="revolute">
 <origin xyz="0.05999999999999999778 3.4694469519536141888e-18 6.9388939039072283776e-18" rpy="-2.7755575615281513959e-16 3.4694469519536398268e-16 3.141592653589793116" />
@@ -296,12 +304,4 @@
 <joint_properties friction="0.0"/>
 </joint>
-<joint name="joint7" type="revolute">
-<origin xyz="0.11349791759135398339 -0.036249999478459471458 0.026000000000000023093" rpy="-1.570796326794896336 2.4702462297869142187e-15 1.5081753875048004426e-15" />
-<parent link="base_link" />
-<child link="middle_proximal" />
-<axis xyz="0 0 1"/>
-<limit effort="0.8499999999999999778" velocity="1.5700000000000000622" lower="-1.0471975511965976313" upper="1.0471975511965976313"/>
-<joint_properties friction="0.0"/>
-</joint>
 </xacro:macro>
 </robot>

Commit message: joint_states working wo offset

File: plato2_description/urdf/ros2_control/plato2.ros2_control.xacro (robot description, xacro)
@@ -19,4 +19,10 @@
                 <state_interface name="effort"/>
             </joint>
+            <joint name="joint3">
+                <command_interface name="position"/>
+                <state_interface name="position"/>
+                <state_interface name="velocity"/>
+                <state_interface name="effort"/>
+            </joint>
             <joint name="joint4">
                 <command_interface name="position"/>
@@ -25,5 +31,5 @@
                 <state_interface name="effort"/>
             </joint>
-            <joint name="joint3">
+            <joint name="joint5">
                 <command_interface name="position"/>
                 <state_interface name="position"/>
@@ -37,5 +43,5 @@
                 <state_interface name="effort"/>
             </joint>
-            <joint name="joint5">
+            <joint name="joint7">
                 <command_interface name="position"/>
                 <state_interface name="position"/>
@@ -49,10 +55,4 @@
                 <state_interface name="effort"/>
             </joint>
-            <joint name="joint7">
-                <command_interface name="position"/>
-                <state_interface name="position"/>
-                <state_interface name="velocity"/>
-                <state_interface name="effort"/>
-            </joint>
         </ros2_control>
   </xacro:macro>

Commit message: ft sensor integration

File: plato2_description/urdf/ros2_control/plato2.ros2_control.xacro (robot description, xacro)
@@ -55,4 +55,12 @@
                 <state_interface name="effort"/>
             </joint>
+        <sensor name="ft_sensor">
+            <state_interface name="force.x"/>
+            <state_interface name="force.y"/>
+            <state_interface name="force.z"/>
+            <state_interface name="torque.x"/>
+            <state_interface name="torque.y"/>
+            <state_interface name="torque.z"/>
+        </sensor>
         </ros2_control>
   </xacro:macro>

File: plato2_description/urdf/xacro/plato2_description.xacro (robot description, xacro)
@@ -118,5 +118,5 @@
 </inertial>
 </link>
-<link name="index_fingertip">
+<!-- <link name="index_fingertip">
 </link>
 <joint name="index_fingertip_frame" type="fixed">
@@ -125,5 +125,5 @@
 <child link="index_fingertip" />
 <axis xyz="0 0 0"/>
-</joint>
+</joint> -->
 <link name="index_proximal">
 <visual>
@@ -170,5 +170,12 @@
 </inertial>
 </link>
-<link name="thumb_fingertip">
+<link name="index_ft_sensor">
+</link>
+<joint name="index_ft_sensor_frame" type="fixed">
+<origin xyz = "-0.0494 0.0 0.0" rpy = "-1.57 0 1.57"/>
+<parent link="index_distal"/>
+<child link="index_ft_sensor"/>
+</joint>
+<!-- <link name="thumb_fingertip">
 <inertial>
 <origin xyz="0 0 0" rpy="0 0 0" />
@@ -182,5 +189,5 @@
 <child link="thumb_fingertip" />
 <axis xyz="0 0 0"/>
-</joint>
+</joint> -->
 <link name="middle_proximal">
 <visual>
@@ -193,15 +200,4 @@
 </material>
 </visual>
-<collision>
-<origin xyz="0 0 0" rpy="0 -0 0" />
-<geometry>
-<mesh filename="file://$(find plato2_description)/meshes/middle_proximal_collision.stl"/>
-</geometry>
-</collision>
-<inertial>
-<origin xyz="0.041723592555954480687 0.00015325900345948331445 -0.0024652665929218429454" rpy="0 0 0"/>
-<mass value="0.046493308366953339794" />
-<inertia ixx="5.9693787373143511043e-06" ixy="-3.1828148640349575716e-08"  ixz="1.0284240810849584112e-08" iyy="2.0043167951845242434e-05" iyz="2.6933150995912662265e-10" izz="1.9050463454403372931e-05" />
-</inertial>
 </link>
 <link name="middle_distal">
@@ -227,5 +223,5 @@
 </inertial>
 </link>
-<link name="middle_fingertip">
+<!-- <link name="middle_fingertip">
 <inertial>
 <origin xyz="0 0 0" rpy="0 0 0" />
@@ -239,5 +235,5 @@
 <child link="middle_fingertip" />
 <axis xyz="0 0 0"/>
-</joint>
+</joint> -->
 <joint name="joint1" type="revolute">
 <origin xyz="0.01149999999999984715 0.039000000000000659139 -0.015849999999999926648" rpy="-1.3045120539345319165e-15 1.5707963267948643615 0" />

Commit message: ros2_control sensor implementation

File: plato2_description/urdf/ros2_control/plato2.ros2_control.xacro (robot description, xacro)
@@ -55,6 +55,6 @@
                 <state_interface name="effort"/>
             </joint>
-        <!-- FT Sensor -->
-        <!-- <sensor name="ft_sensor" type="force_torque">
+      <!-- FT Sensors -->
+        <sensor name="ft_sensor1" type="force_torque">
             <state_interface name="force.x"/>
             <state_interface name="force.y"/>
@@ -63,5 +63,21 @@
             <state_interface name="torque.y"/>
             <state_interface name="torque.z"/>
-        </sensor> -->
+        </sensor>
+        <sensor name="ft_sensor2" type="force_torque">
+            <state_interface name="force.x"/>
+            <state_interface name="force.y"/>
+            <state_interface name="force.z"/>
+            <state_interface name="torque.x"/>
+            <state_interface name="torque.y"/>
+            <state_interface name="torque.z"/>
+        </sensor>
+        <sensor name="ft_sensor3" type="force_torque">
+            <state_interface name="force.x"/>
+            <state_interface name="force.y"/>
+            <state_interface name="force.z"/>
+            <state_interface name="torque.x"/>
+            <state_interface name="torque.y"/>
+            <state_interface name="torque.z"/>
+        </sensor>
         </ros2_control>
   </xacro:macro>

File: plato2_description/urdf/xacro/plato2_description.xacro (robot description, xacro)
@@ -118,12 +118,11 @@
 </inertial>
 </link>
-<!-- <link name="index_fingertip">
-</link>
-<joint name="index_fingertip_frame" type="fixed">
-<origin xyz="-0.076100000000000417311 -0.0050000000000001570966 -0.0024999999998208122243" rpy="1.57079632679491632 1.0729310576333032043e-14 -3.141592653589793116" />
-<parent link="thumb_distal" />
-<child link="index_fingertip" />
-<axis xyz="0 0 0"/>
-</joint> -->
+<link name="thumb_ft_sensor">
+</link>
+<joint name="middle_ft_sensor_frame" type="fixed">
+<origin xyz = "-0.0494 0.0 0.0" rpy = "-1.57 0 1.57"/>
+<parent link="thumb_distal"/>
+<child link="thumb_ft_sensor"/>
+</joint>
 <link name="index_proximal">
 <visual>
@@ -236,4 +235,11 @@
 <axis xyz="0 0 0"/>
 </joint> -->
+<link name="middle_ft_sensor">
+</link>
+<joint name="middle_ft_sensor_frame" type="fixed">
+<origin xyz = "-0.0494 0.0 0.0" rpy = "-1.57 0 1.57"/>
+<parent link="middle_distal"/>
+<child link="index_ft_sensor"/>
+</joint>
 <joint name="joint1" type="revolute">
 <origin xyz="0.01149999999999984715 0.039000000000000659139 -0.015849999999999926648" rpy="-1.3045120539345319165e-15 1.5707963267948643615 0" />
