Commit message: mock hardware

File: plato2_description/urdf/ros2_control/aristo.ros2_control.xacro (robot description, xacro)
@@ -1,12 +1,24 @@
 <?xml version="0.06.0"?>
 <robot xmlns:xacro="http://www.ros.org/wiki/xacro">
-    <xacro:macro name="aristo_ros2_control" params="name">
+    <xacro:macro name="aristo_ros2_control" params="name fake_hardware='false'">
+        <!-- Normalize fake_hardware values so callers can pass true/False, 1/0, or strings -->
+        <xacro:property name="use_mock" value="${fake_hardware == 'true' or fake_hardware == 'True' or fake_hardware == '1' or fake_hardware == 1 or fake_hardware == True}"/>
         <ros2_control name="${name}" type="system">
             <!-- Hardware -->
             <hardware>
-                <plugin>plato2_hardware_interface/PLATO2Hardware</plugin>
+                <!-- Choose real hardware or ros2_control mock component based on the fake_hardware flag -->
+                <xacro:if value="${use_mock}">
+                    <plugin>mock_components/GenericSystem</plugin>
+                </xacro:if>
+                <xacro:unless value="${use_mock}">
+                    <plugin>plato2_hardware_interface/PLATO2Hardware</plugin>
+                </xacro:unless>
             </hardware>
             <joint name="joint1">
+                <command_interface name="position"/>
+                <command_interface name="velocity"/>
                 <command_interface name="effort"/>
+                <command_interface name="stiffness"/>
+                <command_interface name="damping"/>
                 <state_interface name="position"/>
                 <state_interface name="velocity"/>
@@ -14,5 +26,9 @@
             </joint>
             <joint name="joint2">
+                <command_interface name="position"/>
+                <command_interface name="velocity"/>
                 <command_interface name="effort"/>
+                <command_interface name="stiffness"/>
+                <command_interface name="damping"/>
                 <state_interface name="position"/>
                 <state_interface name="velocity"/>
@@ -20,5 +36,9 @@
             </joint>
             <joint name="joint3">
+                <command_interface name="position"/>
+                <command_interface name="velocity"/>
                 <command_interface name="effort"/>
+                <command_interface name="stiffness"/>
+                <command_interface name="damping"/>
                 <state_interface name="position"/>
                 <state_interface name="velocity"/>
@@ -26,5 +46,9 @@
             </joint>
             <joint name="joint4">
+                <command_interface name="position"/>
+                <command_interface name="velocity"/>
                 <command_interface name="effort"/>
+                <command_interface name="stiffness"/>
+                <command_interface name="damping"/>
                 <state_interface name="position"/>
                 <state_interface name="velocity"/>
@@ -32,5 +56,9 @@
             </joint>
             <joint name="joint5">
+                <command_interface name="position"/>
+                <command_interface name="velocity"/>
                 <command_interface name="effort"/>
+                <command_interface name="stiffness"/>
+                <command_interface name="damping"/>
                 <state_interface name="position"/>
                 <state_interface name="velocity"/>
@@ -38,5 +66,9 @@
             </joint>
             <joint name="joint6">
+                <command_interface name="position"/>
+                <command_interface name="velocity"/>
                 <command_interface name="effort"/>
+                <command_interface name="stiffness"/>
+                <command_interface name="damping"/>
                 <state_interface name="position"/>
                 <state_interface name="velocity"/>
@@ -44,5 +76,9 @@
             </joint>
             <joint name="joint7">
+                <command_interface name="position"/>
+                <command_interface name="velocity"/>
                 <command_interface name="effort"/>
+                <command_interface name="stiffness"/>
+                <command_interface name="damping"/>
                 <state_interface name="position"/>
                 <state_interface name="velocity"/>
@@ -50,5 +86,9 @@
             </joint>
             <joint name="joint8">
+                <command_interface name="position"/>
+                <command_interface name="velocity"/>
                 <command_interface name="effort"/>
+                <command_interface name="stiffness"/>
+                <command_interface name="damping"/>
                 <state_interface name="position"/>
                 <state_interface name="velocity"/>
