Commit message: naritouch demo

File: plato2_description/urdf/plato2.urdf.xacro (robot description, xacro)
@@ -2,5 +2,5 @@
 <robot name="plato2_hand" xmlns:xacro="http://www.ros.org/wiki/xacro">
     <!-- Set World Frame -->
-    <link name="world"/>
+    <!-- <link name="world"/> -->
     <!-- Include Robot Description Xacro -->
     <xacro:include filename="$(find plato2_description)/urdf/xacro/plato2_description.xacro"/>

File: plato2_description/urdf/xacro/plato2_description.xacro (robot description, xacro)
@@ -3,9 +3,9 @@
 <xacro:macro name="plato2_description" params="connector_link  xyz:='0 0 0'  rpy:='0 0 0' ">
 <!-- Connector Joint -->
-<joint name="connector_joint" type="fixed">
+<!-- <joint name="connector_joint" type="fixed">
     <parent link="${connector_link}"/>
     <child link="base_link"/>
     <origin xyz="${xyz}" rpy="${rpy}"/>
-</joint>
+</joint> -->
 <link name="base_link">
 <visual>
