Commit message: wip

File: plato2_description/urdf/plato.urdf.xacro (robot description, xacro)
@@ -3,4 +3,5 @@
   <xacro:arg name="fake_hardware" default="false"/>
   <xacro:arg name="zeroing" default="false"/>
+  <xacro:arg name="direct_tx_inter_frame_gap_us" default="100"/>
   <xacro:include filename="$(find plato2_description)/urdf/xacro/plato_description.xacro"/>
   <xacro:include filename="$(find plato2_description)/urdf/ros2_control/plato.ros2_control.xacro"/>
@@ -9,4 +10,5 @@
     name="plato_ros2_control"
     fake_hardware="$(arg fake_hardware)"
-    zeroing="$(arg zeroing)"/>
+    zeroing="$(arg zeroing)"
+    direct_tx_inter_frame_gap_us="$(arg direct_tx_inter_frame_gap_us)"/>
 </robot>

File: plato2_description/urdf/ros2_control/plato.ros2_control.xacro (robot description, xacro)
@@ -1,5 +1,5 @@
 <?xml version="0.06.0"?>
 <robot xmlns:xacro="http://www.ros.org/wiki/xacro">
-  <xacro:macro name="plato_ros2_control" params="name fake_hardware='false' zeroing='false'">
+  <xacro:macro name="plato_ros2_control" params="name fake_hardware='false' zeroing='false' direct_tx_inter_frame_gap_us='100'">
     <xacro:property name="use_mock" value="${fake_hardware == 'true' or fake_hardware == 'True' or fake_hardware == '1' or fake_hardware == 1 or fake_hardware == True}"/>
     <ros2_control name="${name}" type="system">
@@ -11,4 +11,5 @@
           <plugin>plato_hardware_interface/PlatoHardware</plugin>
           <param name="zeroing">${zeroing}</param>
+          <param name="direct_tx_inter_frame_gap_us">${direct_tx_inter_frame_gap_us}</param>
         </xacro:unless>
       </hardware>
