Commit message: wip

File: plato2_description/urdf/aristo.urdf.xacro (robot description, xacro)
@@ -1,13 +1,10 @@
 <?xml version="1.0"?>
 <robot name="aristo_hand" xmlns:xacro="http://www.ros.org/wiki/xacro">
-    <!-- Set World Frame -->
-    <!-- <link name="world"/> -->
-    <!-- Include Robot Description Xacro -->
+  <link name="base_link"/>
+  <!-- Includes -->
     <xacro:include filename="$(find plato2_description)/urdf/xacro/aristo_description.xacro"/>
-    <!-- Include ros2 control Xacro -->
     <xacro:include filename="$(find plato2_description)/urdf/ros2_control/aristo.ros2_control.xacro"/>
-    <!-- Create URDF -->
-    <xacro:aristo_description connector_link="world" xyz="0 0 0" rpy="0 0 0"/>
-    <!-- Create ros2 control -->
-    <xacro:aristo_ros2_control name="aristo_ros2_control"/>
+  <!-- Instantiate geometry/tree and ros2_control -->
+  <xacro:aristo_description connector_link="base_link" xyz="0 0 0" rpy="0 0 0"/>
+  <xacro:aristo_ros2_control name="aristo_ros2_control"/>
 </robot>

File: plato2_description/urdf/ros2_control/aristo.ros2_control.xacro (robot description, xacro)
@@ -1,5 +1,5 @@
 <?xml version="0.06.0"?>
 <robot xmlns:xacro="http://www.ros.org/wiki/xacro">
-    <xacro:macro name="plato_ros2_control" params="name">
+    <xacro:macro name="aristo_ros2_control" params="name">
         <ros2_control name="${name}" type="system">
             <!-- Hardware -->

File: plato2_description/urdf/xacro/aristo_description.xacro (robot description, xacro)
@@ -1,285 +1,282 @@
 <?xml version="1.0"?>
 <robot xmlns:xacro="http://www.ros.org/wiki/xacro">
-<xacro:macro name="aristo_description" params="connector_link  xyz:='0 0 0'  rpy:='0 0 0' ">
-<!-- Link hand_base -->
-  <link name="hand_base">
-    <inertial>
-      <origin xyz="1.14624e-05 -0.0735402 0.00270001" rpy="0 0 0"/>
-      <mass value="0.739028"/>
-      <inertia ixx="0.00120378" ixy="-5.74097e-07" ixz="9.38706e-08" iyy="0.000581026" iyz="0.000226035" izz="0.00122618"/>
-    </inertial>
-    <!-- Part hand_base_parts -->
-    <visual>
-      <origin xyz="1.14624e-05 -0.0735402 0.00270001" rpy="0 -0 0"/>
-      <geometry>
-        <mesh filename="file://$(find plato2_description)/meshes/hand_base.stl"/>
-      </geometry>
-      <material name="hand_base_parts_material">
-        <color rgba="0.582976 0.583383 0.583584 1"/>
-      </material>
-    </visual>
-    <collision>
-      <origin xyz="1.14624e-05 -0.0735402 0.00270001" rpy="0 -0 0"/>
-      <geometry>
-        <mesh filename="file://$(find plato2_description)/meshes/hand_base.stl"/>
-      </geometry>
-    </collision>
-  </link>
-  <!-- Link thumb_metacarpal -->
-  <link name="thumb_metacarpal">
-    <inertial>
-      <origin xyz="5.08388e-05 -0.0186588 0.0228524" rpy="0 0 0"/>
-      <mass value="0.120521"/>
-      <inertia ixx="2.56992e-05" ixy="5.49331e-08" ixz="-4.85452e-08" iyy="3.3197e-05" iyz="2.03706e-06" izz="2.19064e-05"/>
-    </inertial>
-    <!-- Part thumb_metacarpal_parts -->
-    <visual>
-      <origin xyz="5.08388e-05 -0.0186588 0.0228524" rpy="-1.5708 1.92949e-16 -2.97318e-15"/>
-      <geometry>
-        <mesh filename="file://$(find plato2_description)/meshes/thumb_metacarpal.stl"/>
-      </geometry>
-      <material name="thumb_metacarpal_parts_material">
-        <color rgba="0.55008 0.55008 0.55008 1"/>
-      </material>
-    </visual>
-    <collision>
-      <origin xyz="5.08388e-05 -0.0186588 0.0228524" rpy="-1.5708 1.92949e-16 -2.97318e-15"/>
-      <geometry>
-        <mesh filename="file://$(find plato2_description)/meshes/thumb_metacarpal.stl"/>
-      </geometry>
-    </collision>
-  </link>
-  <!-- Link thumb_actuators -->
-  <link name="thumb_actuators">
-    <inertial>
-      <origin xyz="0.00119788 -0.0189545 -0.0225138" rpy="0 0 0"/>
-      <mass value="0.240831"/>
-      <inertia ixx="4.65934e-05" ixy="4.93309e-06" ixz="-5.99186e-07" iyy="0.00017164" iyz="-1.38804e-06" izz="0.000155026"/>
-    </inertial>
-    <!-- Part thumb_actuators_parts -->
-    <visual>
-      <origin xyz="0.00119788 -0.0189545 -0.0225138" rpy="-1.05301e-16 3.1033e-15 -1.5708"/>
-      <geometry>
-        <mesh filename="file://$(find plato2_description)/meshes/thumb_actuators.stl"/>
-      </geometry>
-      <material name="thumb_actuators_parts_material">
-        <color rgba="0.545814 0.546439 0.546747 1"/>
-      </material>
-    </visual>
-    <collision>
-      <origin xyz="0.00119788 -0.0189545 -0.0225138" rpy="-1.05301e-16 3.1033e-15 -1.5708"/>
-      <geometry>
-        <mesh filename="file://$(find plato2_description)/meshes/thumb_actuators.stl"/>
-      </geometry>
-    </collision>
-  </link>
-  <!-- Link thumb_proximal -->
-  <link name="thumb_proximal">
-    <inertial>
-      <origin xyz="0.0275353 8.61887e-05 0.00673205" rpy="0 0 0"/>
-      <mass value="0.0306406"/>
-      <inertia ixx="1.81672e-06" ixy="-4.24383e-08" ixz="-6.4245e-07" iyy="1.85497e-05" iyz="-2.07897e-09" izz="1.81545e-05"/>
-    </inertial>
-    <!-- Part thumb_proximal_parts -->
-    <visual>
-      <origin xyz="0.0275353 8.61887e-05 0.00673205" rpy="1.5708 -1.5708 0"/>
-      <geometry>
-        <mesh filename="file://$(find plato2_description)/meshes/thumb_proximal.stl"/>
-      </geometry>
-      <material name="thumb_proximal_parts_material">
-        <color rgba="0.63463 0.635887 0.633109 1"/>
-      </material>
-    </visual>
-    <collision>
-      <origin xyz="0.0275353 8.61887e-05 0.00673205" rpy="1.5708 -1.5708 0"/>
-      <geometry>
-        <mesh filename="file://$(find plato2_description)/meshes/thumb_proximal.stl"/>
-      </geometry>
-    </collision>
-  </link>
-  <!-- Link thumb_distal -->
-  <link name="thumb_distal">
-    <inertial>
-      <origin xyz="-0.0330685 -0.00101822 -0.00300906" rpy="0 0 0"/>
-      <mass value="0.0219871"/>
-      <inertia ixx="1.21431e-06" ixy="-1.08631e-07" ixz="-2.69395e-09" iyy="9.73575e-06" iyz="2.19882e-10" izz="9.42439e-06"/>
-    </inertial>
-    <!-- Part thumb_distal_parts -->
-    <visual>
-      <origin xyz="-0.0330685 -0.00101822 -0.00300906" rpy="-1.5708 -1.5708 0"/>
-      <geometry>
-        <mesh filename="file://$(find plato2_description)/meshes/thumb_distal.stl"/>
-      </geometry>
-      <material name="thumb_distal_parts_material">
-        <color rgba="0.670015 0.670243 0.668779 1"/>
-      </material>
-    </visual>
-    <collision>
-      <origin xyz="-0.0330685 -0.00101822 -0.00300906" rpy="-1.5708 -1.5708 0"/>
-      <geometry>
-        <mesh filename="file://$(find plato2_description)/meshes/thumb_distal.stl"/>
-      </geometry>
-    </collision>
-  </link>
-  <!-- Joint from thumb_proximal to thumb_distal -->
-  <joint name="joint4" type="revolute">
-    <origin xyz="0.06 -1.38778e-17 0.0105" rpy="-3.27793e-15 -3.41823e-15 3.14159"/>
-    <parent link="thumb_proximal"/>
-    <child link="thumb_distal"/>
-    <axis xyz="0 0 1"/>
-    <limit effort="10" velocity="10" lower="-2.0944" upper="1.0472"/>
-  </joint>
-  <!-- Joint from thumb_actuators to thumb_proximal -->
-  <joint name="joint3" type="revolute">
-    <origin xyz="-0.022 -0.0305 -0.0235" rpy="-1.5708 -7.76068e-17 3.14159"/>
-    <parent link="thumb_actuators"/>
-    <child link="thumb_proximal"/>
-    <axis xyz="0 0 1"/>
-    <limit effort="10" velocity="10" lower="-1.0472" upper="1.0472"/>
-  </joint>
-  <!-- Joint from thumb_metacarpal to thumb_actuators -->
-  <joint name="joint2" type="revolute">
-    <origin xyz="-1.42383e-10 -0.0315 0.025" rpy="-1.5708 1.5708 0"/>
-    <parent link="thumb_metacarpal"/>
-    <child link="thumb_actuators"/>
-    <axis xyz="0 0 1"/>
-    <limit effort="10" velocity="10" lower="-1.5708" upper="1.5708"/>
-  </joint>
-  <!-- Joint from hand_base to thumb_metacarpal -->
-  <joint name="joint1" type="revolute">
-    <origin xyz="4.56293e-16 -0.044 -0.0285" rpy="1.5708 -2.97318e-15 -1.92949e-16"/>
-    <parent link="hand_base"/>
-    <child link="thumb_metacarpal"/>
-    <axis xyz="0 0 1"/>
-    <limit effort="10" velocity="10" lower="-0.785398" upper="0.785398"/>
-  </joint>
-  <!-- Link index_proximal -->
-  <link name="index_proximal">
-    <inertial>
-      <origin xyz="0.0275353 -8.61566e-05 0.00673211" rpy="0 0 0"/>
-      <mass value="0.0306406"/>
-      <inertia ixx="1.81666e-06" ixy="4.24695e-08" ixz="-6.42349e-07" iyy="1.85498e-05" iyz="1.97055e-09" izz="1.81546e-05"/>
-    </inertial>
-    <!-- Part index_proximal_parts -->
-    <visual>
-      <origin xyz="0.0275353 -8.61566e-05 0.00673211" rpy="1.5708 -1.5708 0"/>
-      <geometry>
-        <mesh filename="file://$(find plato2_description)/meshes/index_proximal.stl"/>
-      </geometry>
-      <material name="index_proximal_parts_material">
-        <color rgba="0.63463 0.635887 0.633109 1"/>
-      </material>
-    </visual>
-    <collision>
-      <origin xyz="0.0275353 -8.61566e-05 0.00673211" rpy="1.5708 -1.5708 0"/>
-      <geometry>
-        <mesh filename="file://$(find plato2_description)/meshes/index_proximal.stl"/>
-      </geometry>
-    </collision>
-  </link>
-  <!-- Link index_distal -->
-  <link name="index_distal">
-    <inertial>
-      <origin xyz="-0.0330685 0.00101822 -0.00299094" rpy="0 0 0"/>
-      <mass value="0.0219871"/>
-      <inertia ixx="1.21431e-06" ixy="1.08631e-07" ixz="2.69395e-09" iyy="9.73575e-06" iyz="2.19882e-10" izz="9.42439e-06"/>
-    </inertial>
-    <!-- Part index_distal_parts -->
-    <visual>
-      <origin xyz="-0.0330685 0.00101822 -0.00299094" rpy="-1.5708 -1.5708 0"/>
-      <geometry>
-        <mesh filename="file://$(find plato2_description)/meshes/index_distal.stl"/>
-      </geometry>
-      <material name="index_distal_parts_material">
-        <color rgba="0.670015 0.670243 0.668779 1"/>
-      </material>
-    </visual>
-    <collision>
-      <origin xyz="-0.0330685 0.00101822 -0.00299094" rpy="-1.5708 -1.5708 0"/>
-      <geometry>
-        <mesh filename="file://$(find plato2_description)/meshes/index_distal.stl"/>
-      </geometry>
-    </collision>
-  </link>
-  <!-- Joint from index_proximal to index_distal -->
-  <joint name="joint6" type="revolute">
-    <origin xyz="0.06 0 0.0105" rpy="-1.11022e-16 -4.70442e-24 3.14159"/>
-    <parent link="index_proximal"/>
-    <child link="index_distal"/>
-    <axis xyz="0 0 1"/>
-    <limit effort="10" velocity="10" lower="-1.0472" upper="2.0944"/>
-  </joint>
-  <!-- Joint from hand_base to index_proximal -->
-  <joint name="joint5" type="revolute">
-    <origin xyz="0.0305 -0.113 0.0145" rpy="-1.5708 5.38458e-14 -1.5708"/>
-    <parent link="hand_base"/>
-    <child link="index_proximal"/>
-    <axis xyz="0 0 1"/>
-    <limit effort="10" velocity="10" lower="-1.0472" upper="1.0472"/>
-  </joint>
-  <!-- Link middle_proximal -->
-  <link name="middle_proximal">
-    <inertial>
-      <origin xyz="0.0275353 -8.61887e-05 -0.00673205" rpy="0 0 0"/>
-      <mass value="0.0306406"/>
-      <inertia ixx="1.81672e-06" ixy="4.24383e-08" ixz="6.4245e-07" iyy="1.85497e-05" iyz="-2.07897e-09" izz="1.81545e-05"/>
-    </inertial>
-    <!-- Part middle_proximal_parts -->
-    <visual>
-      <origin xyz="0.0275353 -8.61887e-05 -0.00673205" rpy="1.5708 -1.5708 0"/>
-      <geometry>
-        <mesh filename="file://$(find plato2_description)/meshes/middle_proximal.stl"/>
-      </geometry>
-      <material name="middle_proximal_parts_material">
-        <color rgba="0.63463 0.635887 0.633109 1"/>
-      </material>
-    </visual>
-    <collision>
-      <origin xyz="0.0275353 -8.61887e-05 -0.00673205" rpy="1.5708 -1.5708 0"/>
-      <geometry>
-        <mesh filename="file://$(find plato2_description)/meshes/middle_proximal.stl"/>
-      </geometry>
-    </collision>
-  </link>
-  <!-- Link middle_distal -->
-  <link name="middle_distal">
-    <inertial>
-      <origin xyz="-0.0330685 0.00101822 0.00300906" rpy="0 0 0"/>
-      <mass value="0.0219871"/>
-      <inertia ixx="1.21431e-06" ixy="1.08631e-07" ixz="2.69395e-09" iyy="9.73575e-06" iyz="2.19882e-10" izz="9.42439e-06"/>
-    </inertial>
-    <!-- Part middle_distal_parts -->
-    <visual>
-      <origin xyz="-0.0330685 0.00101822 0.00300906" rpy="-1.5708 -1.5708 0"/>
-      <geometry>
-        <mesh filename="file://$(find plato2_description)/meshes/middle_distal.stl"/>
-      </geometry>
-      <material name="middle_distal_parts_material">
-        <color rgba="0.670015 0.670243 0.668779 1"/>
-      </material>
-    </visual>
-    <collision>
-      <origin xyz="-0.0330685 0.00101822 0.00300906" rpy="-1.5708 -1.5708 0"/>
-      <geometry>
-        <mesh filename="file://$(find plato2_description)/meshes/middle_distal.stl"/>
-      </geometry>
-    </collision>
-  </link>
-  <!-- Joint from middle_proximal to middle_distal -->
-  <joint name="joint8" type="revolute">
-    <origin xyz="0.06 5.20417e-18 -0.0105" rpy="5.1871e-17 2.33151e-17 -3.14159"/>
-    <parent link="middle_proximal"/>
-    <child link="middle_distal"/>
-    <axis xyz="0 0 1"/>
-    <limit effort="10" velocity="10" lower="-2.0944" upper="1.0472"/>
-  </joint>
-  <!-- Joint from hand_base to middle_proximal -->
-  <joint name="joint7" type="revolute">
-    <origin xyz="-0.0305 -0.113 0.0145" rpy="-1.5708 -5.41789e-14 -1.5708"/>
-    <parent link="hand_base"/>
-    <child link="middle_proximal"/>
-    <axis xyz="0 0 1"/>
-    <limit effort="10" velocity="10" lower="-1.0472" upper="1.0472"/>
-  </joint>
-</xacro:macro>
+  <!--
+    Macro: builds the hand and attaches it to `connector_link` with a fixed joint.
+    Usage:
+      <xacro:aristo_description connector_link="world" xyz="0 0 0" rpy="0 0 0"/>
+  -->
+  <xacro:macro name="aristo_description" params="connector_link xyz:='0 0 0' rpy:='0 0 0'">
+    <!-- Base link of the hand -->
+    <link name="hand_base">
+      <inertial>
+        <origin xyz="1.14624e-05 -0.0735402 0.00270001" rpy="0 0 0"/>
+        <mass value="0.739028"/>
+        <inertia ixx="0.00120378" ixy="-5.74097e-07" ixz="9.38706e-08" iyy="0.000581026" iyz="0.000226035" izz="0.00122618"/>
+      </inertial>
+      <visual>
+        <origin xyz="1.14624e-05 -0.0735402 0.00270001" rpy="0 0 0"/>
+        <geometry>
+          <mesh filename="package://plato2_description/meshes/hand_base.stl"/>
+        </geometry>
+        <material name="hand_base_parts_material">
+          <color rgba="0.582976 0.583383 0.583584 1"/>
+        </material>
+      </visual>
+      <collision>
+        <origin xyz="1.14624e-05 -0.0735402 0.00270001" rpy="0 0 0"/>
+        <geometry>
+          <mesh filename="package://plato2_description/meshes/hand_base.stl"/>
+        </geometry>
+      </collision>
+    </link>
+    <!-- thumb_metacarpal -->
+    <link name="thumb_metacarpal">
+      <inertial>
+        <origin xyz="5.08388e-05 -0.0186588 0.0228524" rpy="0 0 0"/>
+        <mass value="0.120521"/>
+        <inertia ixx="2.56992e-05" ixy="5.49331e-08" ixz="-4.85452e-08" iyy="3.3197e-05" iyz="2.03706e-06" izz="2.19064e-05"/>
+      </inertial>
+      <visual>
+        <origin xyz="5.08388e-05 -0.0186588 0.0228524" rpy="-1.5708 0 -2.97318e-15"/>
+        <geometry>
+          <mesh filename="package://plato2_description/meshes/thumb_metacarpal.stl"/>
+        </geometry>
+        <material name="thumb_metacarpal_parts_material">
+          <color rgba="0.55008 0.55008 0.55008 1"/>
+        </material>
+      </visual>
+      <collision>
+        <origin xyz="5.08388e-05 -0.0186588 0.0228524" rpy="-1.5708 0 -2.97318e-15"/>
+        <geometry>
+          <mesh filename="package://plato2_description/meshes/thumb_metacarpal.stl"/>
+        </geometry>
+      </collision>
+    </link>
+    <!-- thumb_actuators -->
+    <link name="thumb_actuators">
+      <inertial>
+        <origin xyz="0.00119788 -0.0189545 -0.0225138" rpy="0 0 0"/>
+        <mass value="0.240831"/>
+        <inertia ixx="4.65934e-05" ixy="4.93309e-06" ixz="-5.99186e-07" iyy="0.00017164" iyz="-1.38804e-06" izz="0.000155026"/>
+      </inertial>
+      <visual>
+        <origin xyz="0.00119788 -0.0189545 -0.0225138" rpy="0 0 -1.5708"/>
+        <geometry>
+          <mesh filename="package://plato2_description/meshes/thumb_actuators.stl"/>
+        </geometry>
+        <material name="thumb_actuators_parts_material">
+          <color rgba="0.545814 0.546439 0.546747 1"/>
+        </material>
+      </visual>
+      <collision>
+        <origin xyz="0.00119788 -0.0189545 -0.0225138" rpy="0 0 -1.5708"/>
+        <geometry>
+          <mesh filename="package://plato2_description/meshes/thumb_actuators.stl"/>
+        </geometry>
+      </collision>
+    </link>
+    <!-- thumb_proximal -->
+    <link name="thumb_proximal">
+      <inertial>
+        <origin xyz="0.0275353 8.61887e-05 0.00673205" rpy="0 0 0"/>
+        <mass value="0.0306406"/>
+        <inertia ixx="1.81672e-06" ixy="-4.24383e-08" ixz="-6.4245e-07" iyy="1.85497e-05" iyz="-2.07897e-09" izz="1.81545e-05"/>
+      </inertial>
+      <visual>
+        <origin xyz="0.0275353 8.61887e-05 0.00673205" rpy="1.5708 -1.5708 0"/>
+        <geometry>
+          <mesh filename="package://plato2_description/meshes/thumb_proximal.stl"/>
+        </geometry>
+        <material name="thumb_proximal_parts_material">
+          <color rgba="0.63463 0.635887 0.633109 1"/>
+        </material>
+      </visual>
+      <collision>
+        <origin xyz="0.0275353 8.61887e-05 0.00673205" rpy="1.5708 -1.5708 0"/>
+        <geometry>
+          <mesh filename="package://plato2_description/meshes/thumb_proximal.stl"/>
+        </geometry>
+      </collision>
+    </link>
+    <!-- thumb_distal -->
+    <link name="thumb_distal">
+      <inertial>
+        <origin xyz="-0.0330685 -0.00101822 -0.00300906" rpy="0 0 0"/>
+        <mass value="0.0219871"/>
+        <inertia ixx="1.21431e-06" ixy="-1.08631e-07" ixz="-2.69395e-09" iyy="9.73575e-06" iyz="2.19882e-10" izz="9.42439e-06"/>
+      </inertial>
+      <visual>
+        <origin xyz="-0.0330685 -0.00101822 -0.00300906" rpy="-1.5708 -1.5708 0"/>
+        <geometry>
+          <mesh filename="package://plato2_description/meshes/thumb_distal.stl"/>
+        </geometry>
+        <material name="thumb_distal_parts_material">
+          <color rgba="0.670015 0.670243 0.668779 1"/>
+        </material>
+      </visual>
+      <collision>
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
Commit message: rap demo

File: plato2_description/urdf/aristo.urdf.xacro (robot description, xacro)
@@ -2,10 +2,10 @@
 <robot name="aristo_hand" xmlns:xacro="http://www.ros.org/wiki/xacro">
   <!-- Root link for TF tree -->
-  <link name="base_link"/>
+  <link name="world"/>
   <!-- Includes -->
     <xacro:include filename="$(find plato2_description)/urdf/xacro/aristo_description.xacro"/>
     <xacro:include filename="$(find plato2_description)/urdf/ros2_control/aristo.ros2_control.xacro"/>
   <!-- Instantiate geometry/tree and ros2_control -->
-  <xacro:aristo_description connector_link="base_link" xyz="0 0 0" rpy="0 0 0"/>
+  <xacro:aristo_description connector_link="world" xyz="0 0 0" rpy="0 0 0"/>
   <xacro:aristo_ros2_control name="aristo_ros2_control"/>
 </robot>
