Commit message: fixed mesh pathing

File: plato2_description/urdf/xacro/plato2_description.xacro (robot description, xacro)
@@ -13,5 +13,5 @@
       <origin xyz="0.0255 -0.0820815 0.00141852" rpy="1.5708 -2.23147e-26 1.5708"/>
       <geometry>
-        <mesh filename="package://assets/m2_5x8.stl"/>
+        <mesh filename="file://$(find plato2_description)/meshes/m2_5x8.stl"/>
       </geometry>
       <material name="m2_5x8_material">
@@ -22,5 +22,5 @@
       <origin xyz="0.0255 -0.0820815 0.00141852" rpy="1.5708 -2.23147e-26 1.5708"/>
       <geometry>
-        <mesh filename="package://assets/m2_5x8.stl"/>
+        <mesh filename="file://$(find plato2_description)/meshes/m2_5x8.stl"/>
       </geometry>
     </collision>
@@ -29,5 +29,5 @@
       <origin xyz="0.023 -0.066375 -0.01" rpy="1.5708 1.5708 0"/>
       <geometry>
-        <mesh filename="package://assets/2mm_dowel_x_5mm.stl"/>
+        <mesh filename="file://$(find plato2_description)/meshes/2mm_dowel_x_5mm.stl"/>
       </geometry>
       <material name="2mm_dowel_x_5mm_material">
@@ -38,5 +38,5 @@
       <origin xyz="0.023 -0.066375 -0.01" rpy="1.5708 1.5708 0"/>
       <geometry>
-        <mesh filename="package://assets/2mm_dowel_x_5mm.stl"/>
+        <mesh filename="file://$(find plato2_description)/meshes/2mm_dowel_x_5mm.stl"/>
       </geometry>
     </collision>
@@ -45,5 +45,5 @@
       <origin xyz="0.016 -0.005 0.01" rpy="-1.5708 1.66607e-26 2.04457e-26"/>
       <geometry>
-        <mesh filename="package://assets/m4x10.stl"/>
+        <mesh filename="file://$(find plato2_description)/meshes/m4x10.stl"/>
       </geometry>
       <material name="m4x10_material">
@@ -54,5 +54,5 @@
       <origin xyz="0.016 -0.005 0.01" rpy="-1.5708 1.66607e-26 2.04457e-26"/>
       <geometry>
-        <mesh filename="package://assets/m4x10.stl"/>
+        <mesh filename="file://$(find plato2_description)/meshes/m4x10.stl"/>
       </geometry>
     </collision>
@@ -61,5 +61,5 @@
       <origin xyz="0.038 -0.069 0.0145" rpy="-2.87681e-17 -1.0472 -1.5708"/>
       <geometry>
-        <mesh filename="package://assets/index_driver_pulley_mount.stl"/>
+        <mesh filename="file://$(find plato2_description)/meshes/index_driver_pulley_mount.stl"/>
       </geometry>
       <material name="index_driver_pulley_mount_material">
@@ -70,5 +70,5 @@
       <origin xyz="0.038 -0.069 0.0145" rpy="-2.87681e-17 -1.0472 -1.5708"/>
       <geometry>
-        <mesh filename="package://assets/index_driver_pulley_mount.stl"/>
+        <mesh filename="file://$(find plato2_description)/meshes/index_driver_pulley_mount.stl"/>
       </geometry>
     </collision>
@@ -77,5 +77,5 @@
       <origin xyz="-0.0160215 -0.039 -0.01925" rpy="1.5708 -1.5708 0"/>
       <geometry>
-        <mesh filename="package://assets/m2_5x8.stl"/>
+        <mesh filename="file://$(find plato2_description)/meshes/m2_5x8.stl"/>
       </geometry>
       <material name="m2_5x8_2_material">
@@ -86,5 +86,5 @@
       <origin xyz="-0.0160215 -0.039 -0.01925" rpy="1.5708 -1.5708 0"/>
       <geometry>
-        <mesh filename="package://assets/m2_5x8.stl"/>
+        <mesh filename="file://$(find plato2_description)/meshes/m2_5x8.stl"/>
       </geometry>
     </collision>
@@ -93,5 +93,5 @@
       <origin xyz="0.0355 -0.0741962 0.0115" rpy="-3.01426e-17 -1.0472 -1.5708"/>
       <geometry>
-        <mesh filename="package://assets/tensioner_nut.stl"/>
+        <mesh filename="file://$(find plato2_description)/meshes/tensioner_nut.stl"/>
       </geometry>
       <material name="tensioner_nut_material">
@@ -102,5 +102,5 @@
       <origin xyz="0.0355 -0.0741962 0.0115" rpy="-3.01426e-17 -1.0472 -1.5708"/>
       <geometry>
-        <mesh filename="package://assets/tensioner_nut.stl"/>
+        <mesh filename="file://$(find plato2_description)/meshes/tensioner_nut.stl"/>
       </geometry>
     </collision>
@@ -109,5 +109,5 @@
       <origin xyz="4.45824e-16 -0.039 -0.047" rpy="1.5708 -1.5708 0"/>
       <geometry>
-        <mesh filename="package://assets/m2_5x8.stl"/>
+        <mesh filename="file://$(find plato2_description)/meshes/m2_5x8.stl"/>
       </geometry>
       <material name="m2_5x8_3_material">
@@ -118,5 +118,5 @@
       <origin xyz="4.45824e-16 -0.039 -0.047" rpy="1.5708 -1.5708 0"/>
       <geometry>
-        <mesh filename="package://assets/m2_5x8.stl"/>
+        <mesh filename="file://$(find plato2_description)/meshes/m2_5x8.stl"/>
       </geometry>
     </collision>
@@ -125,5 +125,5 @@
       <origin xyz="0.0205 -0.0205 -0.011" rpy="1.5708 6.68702e-26 1.5708"/>
       <geometry>
-        <mesh filename="package://assets/m3x6.stl"/>
+        <mesh filename="file://$(find plato2_description)/meshes/m3x6.stl"/>
       </geometry>
       <material name="m3x6_material">
@@ -134,5 +134,5 @@
       <origin xyz="0.0205 -0.0205 -0.011" rpy="1.5708 6.68702e-26 1.5708"/>
       <geometry>
-        <mesh filename="package://assets/m3x6.stl"/>
+        <mesh filename="file://$(find plato2_description)/meshes/m3x6.stl"/>
       </geometry>
     </collision>
@@ -141,5 +141,5 @@
       <origin xyz="0.0355 -0.0741962 0.0115" rpy="7.51543e-17 -1.0472 -1.5708"/>
       <geometry>
-        <mesh filename="package://assets/tensioner.stl"/>
+        <mesh filename="file://$(find plato2_description)/meshes/tensioner.stl"/>
       </geometry>
       <material name="tensioner_material">
@@ -150,5 +150,5 @@
       <origin xyz="0.0355 -0.0741962 0.0115" rpy="7.51543e-17 -1.0472 -1.5708"/>
       <geometry>
-        <mesh filename="package://assets/tensioner.stl"/>
+        <mesh filename="file://$(find plato2_description)/meshes/tensioner.stl"/>
       </geometry>
     </collision>
@@ -157,5 +157,5 @@
       <origin xyz="0.037 -0.0651 0.0145" rpy="-3.00419e-16 -0.523599 1.5708"/>
       <geometry>
-        <mesh filename="package://assets/m2_5x8__2.stl"/>
+        <mesh filename="file://$(find plato2_description)/meshes/m2_5x8__2.stl"/>
       </geometry>
       <material name="m2_5x8_4_material">
@@ -166,5 +166,5 @@
       <origin xyz="0.037 -0.0651 0.0145" rpy="-3.00419e-16 -0.523599 1.5708"/>
       <geometry>
-        <mesh filename="package://assets/m2_5x8__2.stl"/>
+        <mesh filename="file://$(find plato2_description)/meshes/m2_5x8__2.stl"/>
       </geometry>
     </collision>
@@ -173,5 +173,5 @@
       <origin xyz="-0.0305 -0.0905 -0.01625" rpy="-3.14159 1.66607e-26 -2.31296e-16"/>
       <geometry>
-        <mesh filename="package://assets/m2_5x6.stl"/>
+        <mesh filename="file://$(find plato2_description)/meshes/m2_5x6.stl"/>
       </geometry>
       <material name="m2_5x6_material">
@@ -182,5 +182,5 @@
       <origin xyz="-0.0305 -0.0905 -0.01625" rpy="-3.14159 1.66607e-26 -2.31296e-16"/>
       <geometry>
-        <mesh filename="package://assets/m2_5x6.stl"/>
+        <mesh filename="file://$(find plato2_description)/meshes/m2_5x6.stl"/>
       </geometry>
     </collision>
@@ -189,5 +189,5 @@
       <origin xyz="0.0305 -0.079 0.0145" rpy="-1.5708 0.523599 -1.5708"/>
       <geometry>
-        <mesh filename="package://assets/m2_5x8.stl"/>
+        <mesh filename="file://$(find plato2_description)/meshes/m2_5x8.stl"/>
       </geometry>
       <material name="m2_5x8_5_material">
@@ -198,5 +198,5 @@
       <origin xyz="0.0305 -0.079 0.0145" rpy="-1.5708 0.523599 -1.5708"/>
       <geometry>
-        <mesh filename="package://assets/m2_5x8.stl"/>
+        <mesh filename="file://$(find plato2_description)/meshes/m2_5x8.stl"/>
       </geometry>
     </collision>
@@ -205,5 +205,5 @@
       <origin xyz="0.0295 -0.113 -0.01" rpy="1.66607e-26 -6.68575e-26 1.5708"/>
       <geometry>
-        <mesh filename="package://assets/hand_palm.stl"/>
+        <mesh filename="file://$(find plato2_description)/meshes/hand_palm.stl"/>
       </geometry>
       <material name="hand_palm_material">
@@ -214,5 +214,5 @@
       <origin xyz="0.0295 -0.113 -0.01" rpy="1.66607e-26 -6.68575e-26 1.5708"/>
       <geometry>
-        <mesh filename="package://assets/hand_palm.stl"/>
+        <mesh filename="file://$(find plato2_description)/meshes/hand_palm.stl"/>
       </geometry>
     </collision>
@@ -221,5 +221,5 @@
       <origin xyz="0.0205 -0.0385 -0.011" rpy="1.5708 6.68702e-26 1.5708"/>
       <geometry>
-        <mesh filename="package://assets/m3x6.stl"/>
+        <mesh filename="file://$(find plato2_description)/meshes/m3x6.stl"/>
       </geometry>
       <material name="m3x6_2_material">
@@ -230,5 +230,5 @@
       <origin xyz="0.0205 -0.0385 -0.011" rpy="1.5708 6.68702e-26 1.5708"/>
       <geometry>
-        <mesh filename="package://assets/m3x6.stl"/>
+        <mesh filename="file://$(find plato2_description)/meshes/m3x6.stl"/>
       </geometry>
     </collision>
@@ -237,5 +237,5 @@
       <origin xyz="-1.21431e-17 -0.007 0.0214" rpy="1.5708 1.66481e-26 2.04457e-26"/>
       <geometry>
-        <mesh filename="package://assets/part_5_step.stl"/>
+        <mesh filename="file://$(find plato2_description)/meshes/part_5_step.stl"/>
       </geometry>
       <material name="part_5_step_material">
@@ -246,5 +246,5 @@
       <origin xyz="-1.21431e-17 -0.007 0.0214" rpy="1.5708 1.66481e-26 2.04457e-26"/>
       <geometry>
-        <mesh filename="package://assets/part_5_step.stl"/>
+        <mesh filename="file://$(find plato2_description)/meshes/part_5_step.stl"/>
       </geometry>
     </collision>
@@ -253,5 +253,5 @@
       <origin xyz="-0.0295 -0.0475 -0.0075" rpy="-3.31953e-27 -6.68575e-26 1.5708"/>
       <geometry>
-        <mesh filename="package://assets/middle_motor_mount.stl"/>
+        <mesh filename="file://$(find plato2_description)/meshes/middle_motor_mount.stl"/>
       </geometry>
       <material name="middle_motor_mount_material">
@@ -262,5 +262,5 @@
       <origin xyz="-0.0295 -0.0475 -0.0075" rpy="-3.31953e-27 -6.68575e-26 1.5708"/>
       <geometry>
-        <mesh filename="package://assets/middle_motor_mount.stl"/>
+        <mesh filename="file://$(find plato2_description)/meshes/middle_motor_mount.stl"/>
       </geometry>
     </collision>
@@ -269,5 +269,5 @@
       <origin xyz="-0.0405 -0.069 0.0145" rpy="1.98406e-16 -1.0472 -1.5708"/>
       <geometry>
-        <mesh filename="package://assets/tensioner_nut.stl"/>
+        <mesh filename="file://$(find plato2_description)/meshes/tensioner_nut.stl"/>
       </geometry>
       <material name="tensioner_nut_2_material">
@@ -278,5 +278,5 @@
       <origin xyz="-0.0405 -0.069 0.0145" rpy="1.98406e-16 -1.0472 -1.5708"/>
       <geometry>
-        <mesh filename="package://assets/tensioner_nut.stl"/>
+        <mesh filename="file://$(find plato2_description)/meshes/tensioner_nut.stl"/>
       </geometry>
     </collision>
@@ -285,5 +285,5 @@
       <origin xyz="0.0255 -0.0868696 0.0192882" rpy="1.5708 -2.2463e-26 1.5708"/>
       <geometry>
-        <mesh filename="package://assets/m2_5x8.stl"/>
+        <mesh filename="file://$(find plato2_description)/meshes/m2_5x8.stl"/>
       </geometry>
       <material name="m2_5x8_6_material">
@@ -294,5 +294,5 @@
       <origin xyz="0.0255 -0.0868696 0.0192882" rpy="1.5708 -2.2463e-26 1.5708"/>
       <geometry>
-        <mesh filename="package://assets/m2_5x8.stl"/>
+        <mesh filename="file://$(find plato2_description)/meshes/m2_5x8.stl"/>
       </geometry>
     </collision>
@@ -301,5 +301,5 @@
       <origin xyz="-0.0255 -0.0951304 0.00971185" rpy="-1.5708 -7.12247e-26 1.5708"/>
       <geometry>
-        <mesh filename="package://assets/m2_5x8.stl"/>
+        <mesh filename="file://$(find plato2_description)/meshes/m2_5x8.stl"/>
       </geometry>
       <material name="m2_5x8_7_material">
@@ -310,5 +310,5 @@
       <origin xyz="-0.0255 -0.0951304 0.00971185" rpy="-1.5708 -7.12247e-26 1.5708"/>
       <geometry>
-        <mesh filename="package://assets/m2_5x8.stl"/>
+        <mesh filename="file://$(find plato2_description)/meshes/m2_5x8.stl"/>
       </geometry>
     </collision>
@@ -317,5 +317,5 @@
       <origin xyz="-0.023 -0.018 -0.008" rpy="-8.47805e-26 -1.94969e-25 -1.5708"/>
       <geometry>
-        <mesh filename="package://assets/thumb_roll_mount.stl"/>
+        <mesh filename="file://$(find plato2_description)/meshes/thumb_roll_mount.stl"/>
       </geometry>
       <material name="thumb_roll_mount_material">
@@ -326,5 +326,5 @@
       <origin xyz="-0.023 -0.018 -0.008" rpy="-8.47805e-26 -1.94969e-25 -1.5708"/>
       <geometry>
-        <mesh filename="package://assets/thumb_roll_mount.stl"/>
+        <mesh filename="file://$(find plato2_description)/meshes/thumb_roll_mount.stl"/>
       </geometry>
     </collision>
@@ -333,5 +333,5 @@
       <origin xyz="-0.0205 -0.0255 -0.01" rpy="-1.5708 3.02039e-25 1.5708"/>
       <geometry>
-        <mesh filename="package://assets/2mm_dowel_x_4mm.stl"/>
+        <mesh filename="file://$(find plato2_description)/meshes/2mm_dowel_x_4mm.stl"/>
       </geometry>
       <material name="2mm_dowel_x_4mm_material">
@@ -342,5 +342,5 @@
       <origin xyz="-0.0205 -0.0255 -0.01" rpy="-1.5708 3.02039e-25 1.5708"/>
       <geometry>
-        <mesh filename="package://assets/2mm_dowel_x_4mm.stl"/>
+        <mesh filename="file://$(find plato2_description)/meshes/2mm_dowel_x_4mm.stl"/>
       </geometry>
     </collision>
@@ -349,5 +349,5 @@
       <origin xyz="-0.037 -0.07095 0.0178775" rpy="3.14159 -0.523599 1.5708"/>
       <geometry>
-        <mesh filename="package://assets/m2_5x8__2.stl"/>
+        <mesh filename="file://$(find plato2_description)/meshes/m2_5x8__2.stl"/>
       </geometry>
       <material name="m2_5x8_8_material">
@@ -358,5 +358,5 @@
       <origin xyz="-0.037 -0.07095 0.0178775" rpy="3.14159 -0.523599 1.5708"/>
       <geometry>
-        <mesh filename="package://assets/m2_5x8__2.stl"/>
+        <mesh filename="file://$(find plato2_description)/meshes/m2_5x8__2.stl"/>
       </geometry>
     </collision>
@@ -365,5 +365,5 @@
       <origin xyz="-0.0215 -0.0525 -0.011" rpy="3.14159 9.99645e-27 3.14159"/>
       <geometry>
-        <mesh filename="package://assets/m3x6__2.stl"/>
+        <mesh filename="file://$(find plato2_description)/meshes/m3x6__2.stl"/>
       </geometry>
       <material name="m3x6_3_material">
@@ -374,5 +374,5 @@
       <origin xyz="-0.0215 -0.0525 -0.011" rpy="3.14159 9.99645e-27 3.14159"/>
       <geometry>
-        <mesh filename="package://assets/m3x6__2.stl"/>
+        <mesh filename="file://$(find plato2_description)/meshes/m3x6__2.stl"/>
       </geometry>
     </collision>
@@ -381,5 +381,5 @@
       <origin xyz="0.0255 -0.0511304 0.00971185" rpy="1.5708 -2.23147e-26 1.5708"/>
       <geometry>
-        <mesh filename="package://assets/m2_5x8.stl"/>
+        <mesh filename="file://$(find plato2_description)/meshes/m2_5x8.stl"/>
       </geometry>
       <material name="m2_5x8_9_material">
@@ -390,5 +390,5 @@
       <origin xyz="0.0255 -0.0511304 0.00971185" rpy="1.5708 -2.23147e-26 1.5708"/>
       <geometry>
-        <mesh filename="package://assets/m2_5x8.stl"/>
+        <mesh filename="file://$(find plato2_description)/meshes/m2_5x8.stl"/>
       </geometry>
     </collision>
@@ -397,5 +397,5 @@
       <origin xyz="-0.038 -0.069 0.0145" rpy="3.32739e-16 -1.0472 -1.5708"/>
       <geometry>
-        <mesh filename="package://assets/middle_thumb_driver_pulley.stl"/>
+        <mesh filename="file://$(find plato2_description)/meshes/middle_thumb_driver_pulley.stl"/>
       </geometry>
       <material name="middle_thumb_driver_pulley_material">
@@ -406,5 +406,5 @@
       <origin xyz="-0.038 -0.069 0.0145" rpy="3.32739e-16 -1.0472 -1.5708"/>
       <geometry>
-        <mesh filename="package://assets/middle_thumb_driver_pulley.stl"/>
+        <mesh filename="file://$(find plato2_description)/meshes/middle_thumb_driver_pulley.stl"/>
       </geometry>
     </collision>
@@ -413,5 +413,5 @@
       <origin xyz="0.015 -0.0375 -0.0045" rpy="-1.59339e-16 -1.04773e-25 1.5708"/>
       <geometry>
-        <mesh filename="package://assets/m3x6.stl"/>
+        <mesh filename="file://$(find plato2_description)/meshes/m3x6.stl"/>
       </geometry>
       <material name="m3x6_4_material">
@@ -422,5 +422,5 @@
       <origin xyz="0.015 -0.0375 -0.0045" rpy="-1.59339e-16 -1.04773e-25 1.5708"/>
       <geometry>
-        <mesh filename="package://assets/m3x6.stl"/>
+        <mesh filename="file://$(find plato2_description)/meshes/m3x6.stl"/>
       </geometry>
     </collision>
@@ -429,5 +429,5 @@
       <origin xyz="-0.0305 -0.079 0.0145" rpy="-1.5708 -0.523599 1.5708"/>
       <geometry>
-        <mesh filename="package://assets/m2_5x8.stl"/>
+        <mesh filename="file://$(find plato2_description)/meshes/m2_5x8.stl"/>
       </geometry>
       <material name="m2_5x8_10_material">
@@ -438,5 +438,5 @@
       <origin xyz="-0.0305 -0.079 0.0145" rpy="-1.5708 -0.523599 1.5708"/>
       <geometry>
-        <mesh filename="package://assets/m2_5x8.stl"/>
+        <mesh filename="file://$(find plato2_description)/meshes/m2_5x8.stl"/>
       </geometry>
     </collision>
@@ -445,5 +445,5 @@
       <origin xyz="-0.0405 -0.069 0.0145" rpy="5.12486e-16 -1.0472 -1.5708"/>
       <geometry>
-        <mesh filename="package://assets/tensioner.stl"/>
+        <mesh filename="file://$(find plato2_description)/meshes/tensioner.stl"/>
       </geometry>
       <material name="tensioner_2_material">
@@ -454,5 +454,5 @@
       <origin xyz="-0.0405 -0.069 0.0145" rpy="5.12486e-16 -1.0472 -1.5708"/>
       <geometry>
-        <mesh filename="package://assets/tensioner.stl"/>
+        <mesh filename="file://$(find plato2_description)/meshes/tensioner.stl"/>
       </geometry>
     </collision>
@@ -461,5 +461,5 @@
       <origin xyz="-0.01016 -0.0086 -0.00646" rpy="2.04457e-26 -1.5708 0"/>
       <geometry>
-        <mesh filename="package://assets/bolt_bhs3x8_768340404_std.stl"/>
+        <mesh filename="file://$(find plato2_description)/meshes/bolt_bhs3x8_768340404_std.stl"/>
       </geometry>
       <material name="bolt_bhs3x8_768340404_std_material">
@@ -470,5 +470,5 @@
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