Commit message: update xacro and meshes

File: plato2_description/urdf/xacro/plato2_description.xacro (robot description, xacro)
@@ -5,2086 +5,22 @@
   <link name="hand_base">
     <inertial>
-      <origin xyz="1.15031e-05 -0.0735225 0.00270148" rpy="0 0 0"/>
-      <mass value="0.736326"/>
-      <inertia ixx="0.00119873" ixy="-5.7388e-07" ixz="9.38594e-08" iyy="0.000579924" iyz="0.000224407" izz="0.00122208"/>
-    </inertial>
-    <!-- Part m2_5x8 -->
-    <visual>
-      <origin xyz="0.0255 -0.0820815 0.00141852" rpy="1.5708 -2.23147e-26 1.5708"/>
-      <geometry>
-        <mesh filename="file://$(find plato2_description)/meshes/m2_5x8.stl"/>
-      </geometry>
-      <material name="m2_5x8_material">
-        <color rgba="0.752941 0.752941 0.752941 1"/>
-      </material>
-    </visual>
-    <collision>
-      <origin xyz="0.0255 -0.0820815 0.00141852" rpy="1.5708 -2.23147e-26 1.5708"/>
-      <geometry>
-        <mesh filename="file://$(find plato2_description)/meshes/m2_5x8.stl"/>
-      </geometry>
-    </collision>
-    <!-- Part 2mm_dowel_x_5mm -->
-    <visual>
-      <origin xyz="0.023 -0.066375 -0.01" rpy="1.5708 1.5708 0"/>
-      <geometry>
-        <mesh filename="file://$(find plato2_description)/meshes/2mm_dowel_x_5mm.stl"/>
-      </geometry>
-      <material name="2mm_dowel_x_5mm_material">
-        <color rgba="0.752941 0.752941 0.752941 1"/>
-      </material>
-    </visual>
-    <collision>
-      <origin xyz="0.023 -0.066375 -0.01" rpy="1.5708 1.5708 0"/>
-      <geometry>
-        <mesh filename="file://$(find plato2_description)/meshes/2mm_dowel_x_5mm.stl"/>
-      </geometry>
-    </collision>
-    <!-- Part m4x10 -->
-    <visual>
-      <origin xyz="0.016 -0.005 0.01" rpy="-1.5708 1.66607e-26 2.04457e-26"/>
-      <geometry>
-        <mesh filename="file://$(find plato2_description)/meshes/m4x10.stl"/>
-      </geometry>
-      <material name="m4x10_material">
-        <color rgba="0.752941 0.752941 0.752941 1"/>
-      </material>
-    </visual>
-    <collision>
-      <origin xyz="0.016 -0.005 0.01" rpy="-1.5708 1.66607e-26 2.04457e-26"/>
-      <geometry>
-        <mesh filename="file://$(find plato2_description)/meshes/m4x10.stl"/>
-      </geometry>
-    </collision>
-    <!-- Part index_driver_pulley_mount -->
-    <visual>
-      <origin xyz="0.038 -0.069 0.0145" rpy="-2.87681e-17 -1.0472 -1.5708"/>
-      <geometry>
-        <mesh filename="file://$(find plato2_description)/meshes/index_driver_pulley_mount.stl"/>
-      </geometry>
-      <material name="index_driver_pulley_mount_material">
-        <color rgba="0.8 0.8 0.8 1"/>
-      </material>
-    </visual>
-    <collision>
-      <origin xyz="0.038 -0.069 0.0145" rpy="-2.87681e-17 -1.0472 -1.5708"/>
-      <geometry>
-        <mesh filename="file://$(find plato2_description)/meshes/index_driver_pulley_mount.stl"/>
-      </geometry>
-    </collision>
-    <!-- Part m2_5x8_2 -->
-    <visual>
-      <origin xyz="-0.0160215 -0.039 -0.01925" rpy="1.5708 -1.5708 0"/>
-      <geometry>
-        <mesh filename="file://$(find plato2_description)/meshes/m2_5x8.stl"/>
-      </geometry>
-      <material name="m2_5x8_2_material">
-        <color rgba="0.752941 0.752941 0.752941 1"/>
-      </material>
-    </visual>
-    <collision>
-      <origin xyz="-0.0160215 -0.039 -0.01925" rpy="1.5708 -1.5708 0"/>
-      <geometry>
-        <mesh filename="file://$(find plato2_description)/meshes/m2_5x8.stl"/>
-      </geometry>
-    </collision>
-    <!-- Part tensioner_nut -->
-    <visual>
-      <origin xyz="0.0355 -0.0741962 0.0115" rpy="-3.01426e-17 -1.0472 -1.5708"/>
-      <geometry>
-        <mesh filename="file://$(find plato2_description)/meshes/tensioner_nut.stl"/>
-      </geometry>
-      <material name="tensioner_nut_material">
-        <color rgba="0.4 0.388235 0.34902 1"/>
-      </material>
-    </visual>
-    <collision>
-      <origin xyz="0.0355 -0.0741962 0.0115" rpy="-3.01426e-17 -1.0472 -1.5708"/>
-      <geometry>
-        <mesh filename="file://$(find plato2_description)/meshes/tensioner_nut.stl"/>
-      </geometry>
-    </collision>
-    <!-- Part m2_5x8_3 -->
-    <visual>
-      <origin xyz="4.45824e-16 -0.039 -0.047" rpy="1.5708 -1.5708 0"/>
-      <geometry>
-        <mesh filename="file://$(find plato2_description)/meshes/m2_5x8.stl"/>
-      </geometry>
-      <material name="m2_5x8_3_material">
-        <color rgba="0.752941 0.752941 0.752941 1"/>
-      </material>
-    </visual>
-    <collision>
-      <origin xyz="4.45824e-16 -0.039 -0.047" rpy="1.5708 -1.5708 0"/>
-      <geometry>
-        <mesh filename="file://$(find plato2_description)/meshes/m2_5x8.stl"/>
-      </geometry>
-    </collision>
-    <!-- Part m3x6 -->
-    <visual>
-      <origin xyz="0.0205 -0.0205 -0.011" rpy="1.5708 6.68702e-26 1.5708"/>
-      <geometry>
-        <mesh filename="file://$(find plato2_description)/meshes/m3x6.stl"/>
-      </geometry>
-      <material name="m3x6_material">
-        <color rgba="0.752941 0.752941 0.752941 1"/>
-      </material>
-    </visual>
-    <collision>
-      <origin xyz="0.0205 -0.0205 -0.011" rpy="1.5708 6.68702e-26 1.5708"/>
-      <geometry>
-        <mesh filename="file://$(find plato2_description)/meshes/m3x6.stl"/>
-      </geometry>
-    </collision>
-    <!-- Part tensioner -->
-    <visual>
-      <origin xyz="0.0355 -0.0741962 0.0115" rpy="7.51543e-17 -1.0472 -1.5708"/>
-      <geometry>
-        <mesh filename="file://$(find plato2_description)/meshes/tensioner.stl"/>
-      </geometry>
-      <material name="tensioner_material">
-        <color rgba="0.701961 0.682353 0.623529 1"/>
-      </material>
-    </visual>
-    <collision>
-      <origin xyz="0.0355 -0.0741962 0.0115" rpy="7.51543e-17 -1.0472 -1.5708"/>
-      <geometry>
-        <mesh filename="file://$(find plato2_description)/meshes/tensioner.stl"/>
-      </geometry>
-    </collision>
-    <!-- Part m2_5x8_4 -->
-    <visual>
-      <origin xyz="0.037 -0.0651 0.0145" rpy="-3.00419e-16 -0.523599 1.5708"/>
-      <geometry>
-        <mesh filename="file://$(find plato2_description)/meshes/m2_5x8__2.stl"/>
-      </geometry>
-      <material name="m2_5x8_4_material">
-        <color rgba="0.752941 0.752941 0.752941 1"/>
-      </material>
-    </visual>
-    <collision>
-      <origin xyz="0.037 -0.0651 0.0145" rpy="-3.00419e-16 -0.523599 1.5708"/>
-      <geometry>
-        <mesh filename="file://$(find plato2_description)/meshes/m2_5x8__2.stl"/>
-      </geometry>
-    </collision>
-    <!-- Part m2_5x6 -->
-    <visual>
-      <origin xyz="-0.0305 -0.0905 -0.01625" rpy="-3.14159 1.66607e-26 -2.31296e-16"/>
-      <geometry>
-        <mesh filename="file://$(find plato2_description)/meshes/m2_5x6.stl"/>
-      </geometry>
-      <material name="m2_5x6_material">
-        <color rgba="0.752941 0.752941 0.752941 1"/>
-      </material>
-    </visual>
-    <collision>
-      <origin xyz="-0.0305 -0.0905 -0.01625" rpy="-3.14159 1.66607e-26 -2.31296e-16"/>
-      <geometry>
-        <mesh filename="file://$(find plato2_description)/meshes/m2_5x6.stl"/>
-      </geometry>
-    </collision>
-    <!-- Part m2_5x8_5 -->
-    <visual>
-      <origin xyz="0.0305 -0.079 0.0145" rpy="-1.5708 0.523599 -1.5708"/>
-      <geometry>
-        <mesh filename="file://$(find plato2_description)/meshes/m2_5x8.stl"/>
-      </geometry>
-      <material name="m2_5x8_5_material">
-        <color rgba="0.752941 0.752941 0.752941 1"/>
-      </material>
-    </visual>
-    <collision>
-      <origin xyz="0.0305 -0.079 0.0145" rpy="-1.5708 0.523599 -1.5708"/>
-      <geometry>
-        <mesh filename="file://$(find plato2_description)/meshes/m2_5x8.stl"/>
-      </geometry>
-    </collision>
-    <!-- Part hand_palm -->
-    <visual>
-      <origin xyz="0.0295 -0.113 -0.01" rpy="1.66607e-26 -6.68575e-26 1.5708"/>
-      <geometry>
-        <mesh filename="file://$(find plato2_description)/meshes/hand_palm.stl"/>
-      </geometry>
-      <material name="hand_palm_material">
-        <color rgba="0.4 0.4 0.4 1"/>
-      </material>
-    </visual>
-    <collision>
-      <origin xyz="0.0295 -0.113 -0.01" rpy="1.66607e-26 -6.68575e-26 1.5708"/>
-      <geometry>
-        <mesh filename="file://$(find plato2_description)/meshes/hand_palm.stl"/>
-      </geometry>
-    </collision>
-    <!-- Part m3x6_2 -->
-    <visual>
-      <origin xyz="0.0205 -0.0385 -0.011" rpy="1.5708 6.68702e-26 1.5708"/>
-      <geometry>
-        <mesh filename="file://$(find plato2_description)/meshes/m3x6.stl"/>
-      </geometry>
-      <material name="m3x6_2_material">
-        <color rgba="0.752941 0.752941 0.752941 1"/>
-      </material>
-    </visual>
-    <collision>
-      <origin xyz="0.0205 -0.0385 -0.011" rpy="1.5708 6.68702e-26 1.5708"/>
-      <geometry>
-        <mesh filename="file://$(find plato2_description)/meshes/m3x6.stl"/>
-      </geometry>
-    </collision>
-    <!-- Part part_5_step -->
-    <visual>
-      <origin xyz="-1.21431e-17 -0.007 0.0214" rpy="1.5708 1.66481e-26 2.04457e-26"/>
-      <geometry>
-        <mesh filename="file://$(find plato2_description)/meshes/part_5_step.stl"/>
-      </geometry>
-      <material name="part_5_step_material">
-        <color rgba="0.282353 0.54902 0.160784 1"/>
-      </material>
-    </visual>
-    <collision>
-      <origin xyz="-1.21431e-17 -0.007 0.0214" rpy="1.5708 1.66481e-26 2.04457e-26"/>
-      <geometry>
-        <mesh filename="file://$(find plato2_description)/meshes/part_5_step.stl"/>
-      </geometry>
-    </collision>
-    <!-- Part middle_motor_mount -->
-    <visual>
-      <origin xyz="-0.0295 -0.0475 -0.0075" rpy="-3.31953e-27 -6.68575e-26 1.5708"/>
-      <geometry>
-        <mesh filename="file://$(find plato2_description)/meshes/middle_motor_mount.stl"/>
-      </geometry>
-      <material name="middle_motor_mount_material">
-        <color rgba="0.8 0.8 0.8 1"/>
-      </material>
-    </visual>
-    <collision>
-      <origin xyz="-0.0295 -0.0475 -0.0075" rpy="-3.31953e-27 -6.68575e-26 1.5708"/>
-      <geometry>
-        <mesh filename="file://$(find plato2_description)/meshes/middle_motor_mount.stl"/>
-      </geometry>
-    </collision>
-    <!-- Part tensioner_nut_2 -->
-    <visual>
-      <origin xyz="-0.0405 -0.069 0.0145" rpy="1.98406e-16 -1.0472 -1.5708"/>
-      <geometry>
-        <mesh filename="file://$(find plato2_description)/meshes/tensioner_nut.stl"/>
-      </geometry>
-      <material name="tensioner_nut_2_material">
-        <color rgba="0.4 0.388235 0.34902 1"/>
-      </material>
-    </visual>
-    <collision>
-      <origin xyz="-0.0405 -0.069 0.0145" rpy="1.98406e-16 -1.0472 -1.5708"/>
-      <geometry>
-        <mesh filename="file://$(find plato2_description)/meshes/tensioner_nut.stl"/>
-      </geometry>
-    </collision>
-    <!-- Part m2_5x8_6 -->
-    <visual>
-      <origin xyz="0.0255 -0.0868696 0.0192882" rpy="1.5708 -2.2463e-26 1.5708"/>
-      <geometry>
-        <mesh filename="file://$(find plato2_description)/meshes/m2_5x8.stl"/>
-      </geometry>
-      <material name="m2_5x8_6_material">
-        <color rgba="0.752941 0.752941 0.752941 1"/>
-      </material>
-    </visual>
-    <collision>
-      <origin xyz="0.0255 -0.0868696 0.0192882" rpy="1.5708 -2.2463e-26 1.5708"/>
-      <geometry>
-        <mesh filename="file://$(find plato2_description)/meshes/m2_5x8.stl"/>
-      </geometry>
-    </collision>
-    <!-- Part m2_5x8_7 -->
-    <visual>
-      <origin xyz="-0.0255 -0.0951304 0.00971185" rpy="-1.5708 -7.12247e-26 1.5708"/>
-      <geometry>
-        <mesh filename="file://$(find plato2_description)/meshes/m2_5x8.stl"/>
-      </geometry>
-      <material name="m2_5x8_7_material">
-        <color rgba="0.752941 0.752941 0.752941 1"/>
-      </material>
-    </visual>
-    <collision>
-      <origin xyz="-0.0255 -0.0951304 0.00971185" rpy="-1.5708 -7.12247e-26 1.5708"/>
-      <geometry>
-        <mesh filename="file://$(find plato2_description)/meshes/m2_5x8.stl"/>
-      </geometry>
-    </collision>
-    <!-- Part thumb_roll_mount -->
-    <visual>
-      <origin xyz="-0.023 -0.018 -0.008" rpy="-8.47805e-26 -1.94969e-25 -1.5708"/>
-      <geometry>
-        <mesh filename="file://$(find plato2_description)/meshes/thumb_roll_mount.stl"/>
-      </geometry>
-      <material name="thumb_roll_mount_material">
-        <color rgba="0.8 0.8 0.8 1"/>
-      </material>
-    </visual>
-    <collision>
-      <origin xyz="-0.023 -0.018 -0.008" rpy="-8.47805e-26 -1.94969e-25 -1.5708"/>
-      <geometry>
-        <mesh filename="file://$(find plato2_description)/meshes/thumb_roll_mount.stl"/>
-      </geometry>
-    </collision>
-    <!-- Part 2mm_dowel_x_4mm -->
-    <visual>
-      <origin xyz="-0.0205 -0.0255 -0.01" rpy="-1.5708 3.02039e-25 1.5708"/>
-      <geometry>
-        <mesh filename="file://$(find plato2_description)/meshes/2mm_dowel_x_4mm.stl"/>
-      </geometry>
-      <material name="2mm_dowel_x_4mm_material">
-        <color rgba="0.752941 0.752941 0.752941 1"/>
-      </material>
-    </visual>
-    <collision>
-      <origin xyz="-0.0205 -0.0255 -0.01" rpy="-1.5708 3.02039e-25 1.5708"/>
-      <geometry>
-        <mesh filename="file://$(find plato2_description)/meshes/2mm_dowel_x_4mm.stl"/>
-      </geometry>
-    </collision>
-    <!-- Part m2_5x8_8 -->
-    <visual>
-      <origin xyz="-0.037 -0.07095 0.0178775" rpy="3.14159 -0.523599 1.5708"/>
-      <geometry>
-        <mesh filename="file://$(find plato2_description)/meshes/m2_5x8__2.stl"/>
-      </geometry>
-      <material name="m2_5x8_8_material">
-        <color rgba="0.752941 0.752941 0.752941 1"/>
-      </material>
-    </visual>
-    <collision>
-      <origin xyz="-0.037 -0.07095 0.0178775" rpy="3.14159 -0.523599 1.5708"/>
-      <geometry>
-        <mesh filename="file://$(find plato2_description)/meshes/m2_5x8__2.stl"/>
-      </geometry>
-    </collision>
-    <!-- Part m3x6_3 -->
-    <visual>
-      <origin xyz="-0.0215 -0.0525 -0.011" rpy="3.14159 9.99645e-27 3.14159"/>
-      <geometry>
-        <mesh filename="file://$(find plato2_description)/meshes/m3x6__2.stl"/>
-      </geometry>
-      <material name="m3x6_3_material">
-        <color rgba="0.752941 0.752941 0.752941 1"/>
-      </material>
-    </visual>
-    <collision>
-      <origin xyz="-0.0215 -0.0525 -0.011" rpy="3.14159 9.99645e-27 3.14159"/>
-      <geometry>
-        <mesh filename="file://$(find plato2_description)/meshes/m3x6__2.stl"/>
-      </geometry>
-    </collision>
-    <!-- Part m2_5x8_9 -->
-    <visual>
-      <origin xyz="0.0255 -0.0511304 0.00971185" rpy="1.5708 -2.23147e-26 1.5708"/>
-      <geometry>
-        <mesh filename="file://$(find plato2_description)/meshes/m2_5x8.stl"/>
-      </geometry>
-      <material name="m2_5x8_9_material">
-        <color rgba="0.752941 0.752941 0.752941 1"/>
-      </material>
-    </visual>
-    <collision>
-      <origin xyz="0.0255 -0.0511304 0.00971185" rpy="1.5708 -2.23147e-26 1.5708"/>
-      <geometry>
-        <mesh filename="file://$(find plato2_description)/meshes/m2_5x8.stl"/>
-      </geometry>
-    </collision>
-    <!-- Part middle_thumb_driver_pulley -->
-    <visual>
-      <origin xyz="-0.038 -0.069 0.0145" rpy="3.32739e-16 -1.0472 -1.5708"/>
-      <geometry>
-        <mesh filename="file://$(find plato2_description)/meshes/middle_thumb_driver_pulley.stl"/>
-      </geometry>
-      <material name="middle_thumb_driver_pulley_material">
-        <color rgba="0.623529 0.666667 0.701961 1"/>
-      </material>
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