Commit message: revert back to p2 urdf

File: plato2_description/urdf/xacro/plato2_description.xacro (robot description, xacro)
@@ -1,285 +1,309 @@
-<?xml version="1.0" ?>
+<?xml version="1.0"?>
 <robot xmlns:xacro="http://www.ros.org/wiki/xacro">
 <xacro:macro name="plato2_description" params="connector_link  xyz:='0 0 0'  rpy:='0 0 0' ">
-  <!-- Link hand_base -->
-  <link name="hand_base">
-    <inertial>
-      <origin xyz="1.14624e-05 -0.0735402 0.00270001" rpy="0 0 0"/>
-      <mass value="0.739028"/>
-      <inertia ixx="0.00120378" ixy="-5.74097e-07" ixz="9.38706e-08" iyy="0.000581026" iyz="0.000226035" izz="0.00122618"/>
-    </inertial>
-    <!-- Part hand_base_parts -->
-    <visual>
-      <origin xyz="1.14624e-05 -0.0735402 0.00270001" rpy="0 -0 0"/>
-      <geometry>
-        <mesh filename="file://$(find plato2_description)/meshes/hand_base_visual.stl"/>
-      </geometry>
-      <material name="hand_base_parts_material">
-        <color rgba="0.582976 0.583383 0.583584 1"/>
-      </material>
-    </visual>
-    <collision>
-      <origin xyz="1.14624e-05 -0.0735402 0.00270001" rpy="0 -0 0"/>
-      <geometry>
-        <mesh filename="file://$(find plato2_description)/meshes/hand_base_collision.stl"/>
-      </geometry>
-    </collision>
-  </link>
-  <!-- Link thumb_metacarpal -->
-  <link name="thumb_metacarpal">
-    <inertial>
-      <origin xyz="5.08388e-05 0.0186588 -0.0228524" rpy="0 0 0"/>
-      <mass value="0.120521"/>
-      <inertia ixx="2.56992e-05" ixy="-5.49331e-08" ixz="4.85452e-08" iyy="3.3197e-05" iyz="2.03706e-06" izz="2.19064e-05"/>
-    </inertial>
-    <!-- Part thumb_metacarpal_parts -->
-    <visual>
-      <origin xyz="5.08388e-05 0.0186588 -0.0228524" rpy="1.5708 -2.31294e-16 -6.83582e-14"/>
-      <geometry>
-        <mesh filename="file://$(find plato2_description)/meshes/thumb_metacarpal_visual.stl"/>
-      </geometry>
-      <material name="thumb_metacarpal_parts_material">
-        <color rgba="0.55008 0.55008 0.55008 1"/>
-      </material>
-    </visual>
-    <collision>
-      <origin xyz="5.08388e-05 0.0186588 -0.0228524" rpy="1.5708 -2.31294e-16 -6.83582e-14"/>
-      <geometry>
-        <mesh filename="file://$(find plato2_description)/meshes/thumb_metacarpal_collision.stl"/>
-      </geometry>
-    </collision>
-  </link>
-  <!-- Link thumb_actuators -->
-  <link name="thumb_actuators">
-    <inertial>
-      <origin xyz="0.00119788 -0.0189545 -0.0225138" rpy="0 0 0"/>
-      <mass value="0.240831"/>
-      <inertia ixx="4.65934e-05" ixy="4.93309e-06" ixz="-5.99186e-07" iyy="0.00017164" iyz="-1.38804e-06" izz="0.000155026"/>
-    </inertial>
-    <!-- Part thumb_actuators_parts -->
-    <visual>
-      <origin xyz="0.00119788 -0.0189545 -0.0225138" rpy="-3.06645e-16 -6.82726e-14 -1.5708"/>
-      <geometry>
-        <mesh filename="file://$(find plato2_description)/meshes/thumb_actuators_visual.stl"/>
-      </geometry>
-      <material name="thumb_actuators_parts_material">
-        <color rgba="0.545814 0.546439 0.546747 1"/>
-      </material>
-    </visual>
-    <collision>
-      <origin xyz="0.00119788 -0.0189545 -0.0225138" rpy="-3.06645e-16 -6.82726e-14 -1.5708"/>
-      <geometry>
-        <mesh filename="file://$(find plato2_description)/meshes/thumb_actuators_collision.stl"/>
-      </geometry>
-    </collision>
-  </link>
-  <!-- Link thumb_proximal -->
-  <link name="thumb_proximal">
-    <inertial>
-      <origin xyz="0.0275353 -8.61887e-05 -0.00673205" rpy="0 0 0"/>
-      <mass value="0.0306406"/>
-      <inertia ixx="1.81672e-06" ixy="4.24383e-08" ixz="6.4245e-07" iyy="1.85497e-05" iyz="-2.07897e-09" izz="1.81545e-05"/>
-    </inertial>
-    <!-- Part thumb_proximal_parts -->
-    <visual>
-      <origin xyz="0.0275353 -8.61887e-05 -0.00673205" rpy="-1.5708 1.5708 0"/>
-      <geometry>
-        <mesh filename="file://$(find plato2_description)/meshes/thumb_proximal_visual.stl"/>
-      </geometry>
-      <material name="thumb_proximal_parts_material">
-        <color rgba="0.63463 0.635887 0.633109 1"/>
-      </material>
-    </visual>
-    <collision>
-      <origin xyz="0.0275353 -8.61887e-05 -0.00673205" rpy="-1.5708 1.5708 0"/>
-      <geometry>
-        <mesh filename="file://$(find plato2_description)/meshes/thumb_proximal_collision.stl"/>
-      </geometry>
-    </collision>
-  </link>
-  <!-- Link thumb_distal -->
-  <link name="thumb_distal">
-    <inertial>
-      <origin xyz="-0.03316 -0.000711768 -0.00300906" rpy="0 0 0"/>
-      <mass value="0.0219871"/>
-      <inertia ixx="1.20261e-06" ixy="-4.25688e-08" ixz="-2.6749e-09" iyy="9.76625e-06" iyz="1.45731e-10" izz="9.4432e-06"/>
-    </inertial>
-    <!-- Part thumb_distal_parts -->
-    <visual>
-      <origin xyz="-0.03316 -0.000711768 -0.00300906" rpy="-1.5708 -1.5708 0"/>
-      <geometry>
-        <mesh filename="file://$(find plato2_description)/meshes/thumb_distal_visual.stl"/>
-      </geometry>
-      <material name="thumb_distal_parts_material">
-        <color rgba="0.670015 0.670243 0.668779 1"/>
-      </material>
-    </visual>
-    <collision>
-      <origin xyz="-0.03316 -0.000711768 -0.00300906" rpy="-1.5708 -1.5708 0"/>
-      <geometry>
-        <mesh filename="file://$(find plato2_description)/meshes/thumb_distal_collision.stl"/>
-      </geometry>
-    </collision>
-  </link>
-  <!-- Joint from thumb_proximal to thumb_distal -->
-  <joint name="joint4" type="revolute">
-    <origin xyz="0.06 1.38778e-17 -0.0105" rpy="3.14159 4.87464e-15 3.14159"/>
-    <parent link="thumb_proximal"/>
-    <child link="thumb_distal"/>
-    <axis xyz="0 0 1"/>
-    <limit effort="10" velocity="10" lower="-2.0944" upper="1.0472"/>
-  </joint>
-  <!-- Joint from thumb_actuators to thumb_proximal -->
-  <joint name="joint3" type="revolute">
-    <origin xyz="-0.022 -0.0305 -0.0235" rpy="1.5708 -3.06645e-16 3.14159"/>
-    <parent link="thumb_actuators"/>
-    <child link="thumb_proximal"/>
-    <axis xyz="0 0 1"/>
-    <limit effort="10" velocity="10" lower="-1.0472" upper="1.0472"/>
-  </joint>
-  <!-- Joint from thumb_metacarpal to thumb_actuators -->
-  <joint name="joint2" type="revolute">
-    <origin xyz="-1.42383e-10 0.0315 -0.025" rpy="1.5708 -1.5708 0"/>
-    <parent link="thumb_metacarpal"/>
-    <child link="thumb_actuators"/>
-    <axis xyz="0 0 1"/>
-    <limit effort="10" velocity="10" lower="-1.5708" upper="1.5708"/>
-  </joint>
-  <!-- Joint from hand_base to thumb_metacarpal -->
-  <joint name="joint1" type="revolute">
-    <origin xyz="4.36425e-16 -0.044 -0.0285" rpy="-1.5708 6.83582e-14 -2.31294e-16"/>
-    <parent link="hand_base"/>
-    <child link="thumb_metacarpal"/>
-    <axis xyz="0 0 1"/>
-    <limit effort="10" velocity="10" lower="-0.785398" upper="0.785398"/>
-  </joint>
-  <!-- Link index_proximal -->
-  <link name="index_proximal">
-    <inertial>
-      <origin xyz="0.0275353 8.61566e-05 -0.00673211" rpy="0 0 0"/>
-      <mass value="0.0306406"/>
-      <inertia ixx="1.81666e-06" ixy="-4.24695e-08" ixz="6.42349e-07" iyy="1.85498e-05" iyz="1.97055e-09" izz="1.81546e-05"/>
-    </inertial>
-    <!-- Part index_proximal_parts -->
-    <visual>
-      <origin xyz="0.0275353 8.61566e-05 -0.00673211" rpy="-1.5708 1.5708 0"/>
-      <geometry>
-        <mesh filename="file://$(find plato2_description)/meshes/index_proximal_visual.stl"/>
-      </geometry>
-      <material name="index_proximal_parts_material">
-        <color rgba="0.63463 0.635887 0.633109 1"/>
-      </material>
-    </visual>
-    <collision>
-      <origin xyz="0.0275353 8.61566e-05 -0.00673211" rpy="-1.5708 1.5708 0"/>
-      <geometry>
-        <mesh filename="file://$(find plato2_description)/meshes/index_proximal_collision.stl"/>
-      </geometry>
-    </collision>
-  </link>
-  <!-- Link index_distal -->
-  <link name="index_distal">
-    <inertial>
-      <origin xyz="-0.03316 0.000711768 -0.00299094" rpy="0 0 0"/>
-      <mass value="0.0219871"/>
-      <inertia ixx="1.20261e-06" ixy="4.25688e-08" ixz="2.6749e-09" iyy="9.76625e-06" iyz="1.45731e-10" izz="9.4432e-06"/>
-    </inertial>
-    <!-- Part index_distal_parts -->
-    <visual>
-      <origin xyz="-0.03316 0.000711768 -0.00299094" rpy="-1.5708 -1.5708 0"/>
-      <geometry>
-        <mesh filename="file://$(find plato2_description)/meshes/index_distal_visual.stl"/>
-      </geometry>
-      <material name="index_distal_parts_material">
-        <color rgba="0.670015 0.670243 0.668779 1"/>
-      </material>
-    </visual>
-    <collision>
-      <origin xyz="-0.03316 0.000711768 -0.00299094" rpy="-1.5708 -1.5708 0"/>
-      <geometry>
-        <mesh filename="file://$(find plato2_description)/meshes/index_distal_collision.stl"/>
-      </geometry>
-    </collision>
-  </link>
-  <!-- Joint from index_proximal to index_distal -->
-  <joint name="joint6" type="revolute">
-    <origin xyz="0.06 5.20417e-18 -0.0105" rpy="-3.14159 6.12323e-17 -3.14159"/>
-    <parent link="index_proximal"/>
-    <child link="index_distal"/>
-    <axis xyz="0 0 1"/>
-    <limit effort="10" velocity="10" lower="-1.0472" upper="2.0944"/>
-  </joint>
-  <!-- Joint from hand_base to index_proximal -->
-  <joint name="joint5" type="revolute">
-    <origin xyz="0.0305 -0.113 0.0145" rpy="1.5708 1.58762e-14 -1.5708"/>
-    <parent link="hand_base"/>
-    <child link="index_proximal"/>
-    <axis xyz="0 0 1"/>
-    <limit effort="10" velocity="10" lower="-1.0472" upper="1.0472"/>
-  </joint>
-  <!-- Link middle_proximal -->
-  <link name="middle_proximal">
-    <inertial>
-      <origin xyz="0.0275353 -8.61887e-05 -0.00673205" rpy="0 0 0"/>
-      <mass value="0.0306406"/>
-      <inertia ixx="1.81672e-06" ixy="4.24383e-08" ixz="6.4245e-07" iyy="1.85497e-05" iyz="-2.07897e-09" izz="1.81545e-05"/>
-    </inertial>
-    <!-- Part middle_proximal_parts -->
-    <visual>
-      <origin xyz="0.0275353 -8.61887e-05 -0.00673205" rpy="1.5708 -1.5708 0"/>
-      <geometry>
-        <mesh filename="file://$(find plato2_description)/meshes/middle_proximal_visual.stl"/>
-      </geometry>
-      <material name="middle_proximal_parts_material">
-        <color rgba="0.63463 0.635887 0.633109 1"/>
-      </material>
-    </visual>
-    <collision>
-      <origin xyz="0.0275353 -8.61887e-05 -0.00673205" rpy="1.5708 -1.5708 0"/>
-      <geometry>
-        <mesh filename="file://$(find plato2_description)/meshes/middle_proximal_collision.stl"/>
-      </geometry>
-    </collision>
-  </link>
-  <!-- Link middle_distal -->
-  <link name="middle_distal">
-    <inertial>
-      <origin xyz="-0.03316 -0.000711768 -0.00300906" rpy="0 0 0"/>
-      <mass value="0.0219871"/>
-      <inertia ixx="1.20261e-06" ixy="-4.25688e-08" ixz="-2.6749e-09" iyy="9.76625e-06" iyz="1.45731e-10" izz="9.4432e-06"/>
-    </inertial>
-    <!-- Part middle_distal_parts -->
-    <visual>
-      <origin xyz="-0.03316 -0.000711768 -0.00300906" rpy="1.5708 1.5708 0"/>
-      <geometry>
-        <mesh filename="file://$(find plato2_description)/meshes/middle_distal_visual.stl"/>
-      </geometry>
-      <material name="middle_distal_parts_material">
-        <color rgba="0.670015 0.670243 0.668779 1"/>
-      </material>
-    </visual>
-    <collision>
-      <origin xyz="-0.03316 -0.000711768 -0.00300906" rpy="1.5708 1.5708 0"/>
-      <geometry>
-        <mesh filename="file://$(find plato2_description)/meshes/middle_distal_collision.stl"/>
-      </geometry>
-    </collision>
-  </link>
-  <!-- Joint from middle_proximal to middle_distal -->
-  <joint name="joint8" type="revolute">
-    <origin xyz="0.06 -4.51028e-17 -0.0105" rpy="3.14159 1.03954e-15 3.14159"/>
-    <parent link="middle_proximal"/>
-    <child link="middle_distal"/>
-    <axis xyz="0 0 1"/>
-    <limit effort="10" velocity="10" lower="-2.0944" upper="1.0472"/>
-  </joint>
-  <!-- Joint from hand_base to middle_proximal -->
-  <joint name="joint7" type="revolute">
-    <origin xyz="-0.0305 -0.113 0.0145" rpy="-1.5708 8.07687e-14 -1.5708"/>
-    <parent link="hand_base"/>
-    <child link="middle_proximal"/>
-    <axis xyz="0 0 1"/>
-    <limit effort="10" velocity="10" lower="-1.0472" upper="1.0472"/>
-  </joint>
+<!-- Connector Joint -->
+<!-- <joint name="connector_joint" type="fixed">
+    <parent link="${connector_link}"/>
+    <child link="base_link"/>
+    <origin xyz="${xyz}" rpy="${rpy}"/>
+</joint> -->
+<link name="base_link">
+<visual>
+<origin xyz="0 0 0" rpy="0 -0 0" />
+<geometry>
+<mesh filename="file://$(find plato2_description)/meshes/hand_base_visual.stl"/>
+</geometry>
+<material name="hand_base_material">
+<color rgba="0.62757649539087556612 0.63052391066502089245 0.63406435937041083495 1.0"/>
+</material>
+</visual>
+<collision>
+<origin xyz="0 0 0" rpy="0 -0 0" />
+<geometry>
+<mesh filename="file://$(find plato2_description)/meshes/hand_base_collision.stl"/>
+</geometry>
+</collision>
+<inertial>
+<origin xyz="0.071381088457538419134 0.0044411406143265753921 0.014775265975730310017" rpy="0 0 0"/>
+<mass value="0.76837978567269427099" />
+<inertia ixx="0.00085136196223773938103" ixy="0.00013892752211586731174"  ixz="-0.0002179020540203063913" iyy="0.0012036327317835073241" iyz="6.1825154819893692873e-05" izz="0.0016151849851495560934" />
+</inertial>
+</link>
+<link name="thumb_metacarpal">
+<visual>
+<origin xyz="0 0 0" rpy="0 -0 0" />
+<geometry>
+<mesh filename="file://$(find plato2_description)/meshes/thumb_metacarpal_visual.stl"/>
+</geometry>
+<material name="thumb_metacarpal_material">
+<color rgba="0.47481548487313229856 0.49707036313748559353 0.54567970250436259594 1.0"/>
+</material>
+</visual>
+<collision>
+<origin xyz="0 0 0" rpy="0 -0 0" />
+<geometry>
+<mesh filename="file://$(find plato2_description)/meshes/thumb_metacarpal_collision.stl"/>
+</geometry>
+</collision>
+<inertial>
+<origin xyz="0.036057066254829940599 -9.2990252935181391459e-07 0.020250212737826605441" rpy="0 0 0"/>
+<mass value="0.10438786966597224382" />
+<inertia ixx="2.8951316861868887426e-05" ixy="3.0994244419676533628e-10"  ixz="-4.800649674297535383e-07" iyy="3.8993260644122764531e-05" iyz="2.6529301795122234156e-10" izz="2.6615537505915890328e-05" />
+</inertial>
+</link>
+<link name="thumb_actuators">
+<visual>
+<origin xyz="0 0 0" rpy="0 -0 0" />
+<geometry>
+<mesh filename="file://$(find plato2_description)/meshes/thumb_actuators_visual.stl"/>
+</geometry>
+<material name="thumb_actuators_material">
+<color rgba="0.54936477010542306143 0.54936477010542306143 0.54936477010542306143 1.0"/>
+</material>
+</visual>
+<collision>
+<origin xyz="0 0 0" rpy="0 -0 0" />
+<geometry>
+<mesh filename="file://$(find plato2_description)/meshes/thumb_actuators_collision.stl"/>
+</geometry>
+</collision>
+<inertial>
+<origin xyz="-0.002512192597438537775 0.0011397629422540871483 -0.0230114785012479027" rpy="0 0 0"/>
+<mass value="0.22950045822102393966" />
+<inertia ixx="4.7745842527753026808e-05" ixy="2.3503025721242425626e-05"  ixz="-2.1890746820627907549e-06" iyy="0.00016677084855535142301" iyz="-6.3810307366217034236e-07" izz="0.00015370810388584102337" />
+</inertial>
+</link>
+<link name="thumb_proximal">
+<visual>
+<origin xyz="0 0 0" rpy="0 -0 0" />
+<geometry>
+<mesh filename="file://$(find plato2_description)/meshes/thumb_proximal_visual.stl"/>
+</geometry>
+<material name="thumb_proximal_material">
+<color rgba="0.85676347476547665138 0.85684628218728142723 0.85689596664036427054 1.0"/>
+</material>
+</visual>
+<collision>
+<origin xyz="0 0 0" rpy="0 -0 0" />
+<geometry>
+<mesh filename="file://$(find plato2_description)/meshes/thumb_proximal_collision.stl"/>
+</geometry>
+</collision>
+<inertial>
+<origin xyz="0.041723592555954480687 -0.00015325900345950071589 -0.0025347334070781532556" rpy="0 0 0"/>
+<mass value="0.046493308366953339794" />
+<inertia ixx="5.9693787373143358577e-06" ixy="3.1828148640339470878e-08"  ixz="-1.0284240810881167522e-08" iyy="2.0043167951845195001e-05" iyz="2.6933150996232134927e-10" izz="1.9050463454403359379e-05" />
+</inertial>
+</link>
+<link name="thumb_distal">
+<visual>
+<origin xyz="0 0 0" rpy="0 -0 0" />
+<geometry>
+<mesh filename="file://$(find plato2_description)/meshes/thumb_distal_visual.stl"/>
+</geometry>
+<material name="thumb_distal_material">
+<color rgba="0.91400085189828661481 0.91668729942166382596 0.91820961968491088268 1.0"/>
+</material>
+</visual>
+<collision>
+<origin xyz="0 0 0" rpy="0 -0 0" />
+<geometry>
+<mesh filename="file://$(find plato2_description)/meshes/thumb_distal_collision.stl"/>
+</geometry>
+</collision>
+<inertial>
+<origin xyz="-0.045658753506383910337 -0.0018551753759659538219 -0.0024988078851896785258" rpy="0 0 0"/>
+<mass value="0.043661202672803788027" />
+<inertia ixx="6.329463162449488319e-06" ixy="-4.2442099039110044596e-08"  ixz="-5.6685758581269062122e-09" iyy="1.633602004590589129e-05" iyz="1.4879017507959954281e-09" izz="1.5001660982685637597e-05" />
+</inertial>
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