Commit message: wip

File: plato2_description/urdf/xacro/aristo_description.xacro (robot description, xacro)
@@ -30,4 +30,14 @@
       </collision>
     </link>
+    <!-- thumb_distal_tactile: tactile sensor frame 4.73 cm distal of thumb_distal -->
+    <link name="thumb_distal_tactile" />
+    <joint name="thumb_distal_to_tactile" type="fixed">
+      <!-- translate 0.0473 m (4.73 cm) along the distal link local +x -->
+  <!-- orient tactile frame so Z+ points downward while keeping +X forward: rotate pi around X -->
+  <!-- keep thumb translation, mirror orientation of index (invert yaw) -->
+  <origin xyz="-0.0523 0.01 -0.0025" rpy="0 1.57 1.57"/>
+      <parent link="thumb_distal"/>
+      <child link="thumb_distal_tactile"/>
+    </joint>
     <!-- thumb_metacarpal -->
     <link name="thumb_metacarpal">
@@ -123,4 +133,25 @@
     </link>
     <!-- Thumb joints -->
+    <joint name="joint1" type="revolute">
+      <origin xyz="4.56293e-16 -0.044 -0.0285" rpy="1.5708 0 0"/>
+      <parent link="hand_base"/>
+      <child link="thumb_metacarpal"/>
+      <axis xyz="0 0 1"/>
+      <limit effort="10" velocity="10" lower="-0.785398" upper="0.785398"/>
+    </joint>
+    <joint name="joint2" type="revolute">
+      <origin xyz="-1.42383e-10 -0.0315 0.025" rpy="-1.5708 1.5708 0"/>
+      <parent link="thumb_metacarpal"/>
+      <child link="thumb_actuators"/>
+      <axis xyz="0 0 1"/>
+      <limit effort="10" velocity="10" lower="-1.5708" upper="1.5708"/>
+    </joint>
+    <joint name="joint3" type="revolute">
+      <origin xyz="-0.022 -0.0305 -0.0235" rpy="-1.5708 0 3.14159"/>
+      <parent link="thumb_actuators"/>
+      <child link="thumb_proximal"/>
+      <axis xyz="0 0 1"/>
+      <limit effort="10" velocity="10" lower="-1.0472" upper="1.0472"/>
+    </joint>
     <joint name="joint4" type="revolute">
       <origin xyz="0.06 0 0.0105" rpy="0 0 3.14159"/>
@@ -130,25 +161,4 @@
       <limit effort="10" velocity="10" lower="-2.0944" upper="1.0472"/>
     </joint>
-    <joint name="joint3" type="revolute">
-      <origin xyz="-0.022 -0.0305 -0.0235" rpy="-1.5708 0 3.14159"/>
-      <parent link="thumb_actuators"/>
-      <child link="thumb_proximal"/>
-      <axis xyz="0 0 1"/>
-      <limit effort="10" velocity="10" lower="-1.0472" upper="1.0472"/>
-    </joint>
-    <joint name="joint2" type="revolute">
-      <origin xyz="-1.42383e-10 -0.0315 0.025" rpy="-1.5708 1.5708 0"/>
-      <parent link="thumb_metacarpal"/>
-      <child link="thumb_actuators"/>
-      <axis xyz="0 0 1"/>
-      <limit effort="10" velocity="10" lower="-1.5708" upper="1.5708"/>
-    </joint>
-    <joint name="joint1" type="revolute">
-      <origin xyz="4.56293e-16 -0.044 -0.0285" rpy="1.5708 0 0"/>
-      <parent link="hand_base"/>
-      <child link="thumb_metacarpal"/>
-      <axis xyz="0 0 1"/>
-      <limit effort="10" velocity="10" lower="-0.785398" upper="0.785398"/>
-    </joint>
     <!-- index_proximal -->
     <link name="index_proximal">
@@ -198,4 +208,11 @@
     </link>
     <!-- Index joints -->
+    <joint name="joint5" type="revolute">
+      <origin xyz="0.0305 -0.113 0.0145" rpy="-1.5708 0 -1.5708"/>
+      <parent link="hand_base"/>
+      <child link="index_proximal"/>
+      <axis xyz="0 0 1"/>
+      <limit effort="10" velocity="10" lower="-1.0472" upper="1.0472"/>
+    </joint>
     <joint name="joint6" type="revolute">
       <origin xyz="0.06 0 0.0105" rpy="0 0 3.14159"/>
@@ -205,58 +222,21 @@
       <limit effort="10" velocity="10" lower="-1.0472" upper="2.0944"/>
     </joint>
-    <joint name="joint5" type="revolute">
-      <origin xyz="0.0305 -0.113 0.0145" rpy="-1.5708 0 -1.5708"/>
+    <!-- index_distal_tactile: tactile sensor frame 4.73 cm distal of index_distal -->
+    <link name="index_distal_tactile" />
+    <joint name="index_distal_to_tactile" type="fixed">
+      <!-- translate 0.0473 m (4.73 cm) along the distal link local +x -->
+  <!-- orient tactile frame so Z+ points downward while keeping +X forward: rotate pi around X -->
+  <origin xyz="-0.0523 -0.01 -0.0025" rpy="0 -1.57 1.57"/>
+      <parent link="index_distal"/>
+      <child link="index_distal_tactile"/>
+    </joint>
+      <!-- Middle joints -->
+    <joint name="joint7" type="revolute">
+      <origin xyz="-0.0305 -0.113 0.0145" rpy="-1.5708 0 -1.5708"/>
       <parent link="hand_base"/>
-      <child link="index_proximal"/>
+      <child link="middle_proximal"/>
       <axis xyz="0 0 1"/>
       <limit effort="10" velocity="10" lower="-1.0472" upper="1.0472"/>
     </joint>
-    <!-- middle_proximal -->
-    <link name="middle_proximal">
-      <inertial>
-        <origin xyz="0.0275353 -8.61887e-05 -0.00673205" rpy="0 0 0"/>
-        <mass value="0.0306406"/>
-        <inertia ixx="1.81672e-06" ixy="4.24383e-08" ixz="6.4245e-07" iyy="1.85497e-05" iyz="-2.07897e-09" izz="1.81545e-05"/>
-      </inertial>
-      <visual>
-        <origin xyz="0.0275353 -8.61887e-05 -0.00673205" rpy="1.5708 -1.5708 0"/>
-        <geometry>
-          <mesh filename="package://plato2_description/meshes/middle_proximal.stl"/>
-        </geometry>
-        <material name="middle_proximal_parts_material">
-          <color rgba="0.63463 0.635887 0.633109 1"/>
-        </material>
-      </visual>
-      <collision>
-        <origin xyz="0.0275353 -8.61887e-05 -0.00673205" rpy="1.5708 -1.5708 0"/>
-        <geometry>
-          <mesh filename="package://plato2_description/meshes/middle_proximal.stl"/>
-        </geometry>
-      </collision>
-    </link>
-    <!-- middle_distal -->
-    <link name="middle_distal">
-      <inertial>
-        <origin xyz="-0.0330685 0.00101822 0.00300906" rpy="0 0 0"/>
-        <mass value="0.0219871"/>
-        <inertia ixx="1.21431e-06" ixy="1.08631e-07" ixz="2.69395e-09" iyy="9.73575e-06" iyz="2.19882e-10" izz="9.42439e-06"/>
-      </inertial>
-      <visual>
-        <origin xyz="-0.0330685 0.00101822 0.00300906" rpy="-1.5708 -1.5708 0"/>
-        <geometry>
-          <mesh filename="package://plato2_description/meshes/middle_distal.stl"/>
-        </geometry>
-        <material name="middle_distal_parts_material">
-          <color rgba="0.670015 0.670243 0.668779 1"/>
-        </material>
-      </visual>
-      <collision>
-        <origin xyz="-0.0330685 0.00101822 0.00300906" rpy="-1.5708 -1.5708 0"/>
-        <geometry>
-          <mesh filename="package://plato2_description/meshes/middle_distal.stl"/>
-        </geometry>
-      </collision>
-    </link>
-    <!-- Middle joints -->
     <joint name="joint8" type="revolute">
       <origin xyz="0.06 0 -0.0105" rpy="0 0 -3.14159"/>
@@ -264,12 +244,60 @@
       <child link="middle_distal"/>
       <axis xyz="0 0 1"/>
-      <limit effort="10" velocity="10" lower="-2.0944" upper="1.0472"/>
-    </joint>
-    <joint name="joint7" type="revolute">
-      <origin xyz="-0.0305 -0.113 0.0145" rpy="-1.5708 0 -1.5708"/>
-      <parent link="hand_base"/>
-      <child link="middle_proximal"/>
-      <axis xyz="0 0 1"/>
-      <limit effort="10" velocity="10" lower="-1.0472" upper="1.0472"/>
+      <limit effort="10" velocity="10" lower="-1.0472" upper="2.0944"/>
+    </joint>
+    <!-- middle_proximal -->
+    <link name="middle_proximal">
+      <inertial>
+        <origin xyz="0.0275353 -8.61887e-05 -0.00673205" rpy="0 0 0"/>
+        <mass value="0.0306406"/>
+        <inertia ixx="1.81672e-06" ixy="4.24383e-08" ixz="6.4245e-07" iyy="1.85497e-05" iyz="-2.07897e-09" izz="1.81545e-05"/>
+      </inertial>
+      <visual>
+        <origin xyz="0.0275353 -8.61887e-05 -0.00673205" rpy="1.5708 -1.5708 0"/>
+        <geometry>
+          <mesh filename="package://plato2_description/meshes/middle_proximal.stl"/>
+        </geometry>
+        <material name="middle_proximal_parts_material">
+          <color rgba="0.63463 0.635887 0.633109 1"/>
+        </material>
+      </visual>
+      <collision>
+        <origin xyz="0.0275353 -8.61887e-05 -0.00673205" rpy="1.5708 -1.5708 0"/>
+        <geometry>
+          <mesh filename="package://plato2_description/meshes/middle_proximal.stl"/>
+        </geometry>
+      </collision>
+    </link>
+    <!-- middle_distal -->
+    <link name="middle_distal">
+      <inertial>
+        <origin xyz="-0.0330685 0.00101822 0.00300906" rpy="0 0 0"/>
+        <mass value="0.0219871"/>
+        <inertia ixx="1.21431e-06" ixy="1.08631e-07" ixz="2.69395e-09" iyy="9.73575e-06" iyz="2.19882e-10" izz="9.42439e-06"/>
+      </inertial>
+      <visual>
+        <origin xyz="-0.0330685 0.00101822 0.00300906" rpy="-1.5708 -1.5708 0"/>
+        <geometry>
+          <mesh filename="package://plato2_description/meshes/middle_distal.stl"/>
+        </geometry>
+        <material name="middle_distal_parts_material">
+          <color rgba="0.670015 0.670243 0.668779 1"/>
+        </material>
+      </visual>
+      <collision>
+        <origin xyz="-0.0330685 0.00101822 0.00300906" rpy="-1.5708 -1.5708 0"/>
+        <geometry>
+          <mesh filename="package://plato2_description/meshes/middle_distal.stl"/>
+        </geometry>
+      </collision>
+    </link>
+    <!-- middle_distal_tactile: tactile sensor frame 4.73 cm distal of middle_distal -->
+    <link name="middle_distal_tactile" />
+    <joint name="middle_distal_to_tactile" type="fixed">
+      <!-- translate 0.0473 m (4.73 cm) along the distal link local +x -->
+  <!-- orient tactile frame so Z+ points downward while keeping +X forward: rotate pi around X -->
+  <origin xyz="-0.0523 -0.01 -0.0025" rpy="0 -1.57 1.57"/>
+      <parent link="middle_distal"/>
+      <child link="middle_distal_tactile"/>
     </joint>
     <!-- Attach hand_base to the provided connector link -->

Commit message: fingertip frame

File: plato2_description/urdf/xacro/aristo_description.xacro (robot description, xacro)
@@ -7,4 +7,19 @@
   -->
   <xacro:macro name="aristo_description" params="connector_link xyz:='0 0 0' rpy:='0 0 0'">
+    <!-- Create hand_mount link as intermediate frame -->
+    <link name="hand_mount">
+    </link>
+    <!-- Attach hand_mount to the provided connector link -->
+    <joint name="connector_to_hand_mount" type="fixed">
+      <origin xyz="0 0 0" rpy="0 0 0"/>
+      <parent link="${connector_link}"/>
+      <child link="hand_mount"/>
+    </joint>
+    <!-- Rotate hand_base 90 degrees around Z to point in +X direction -->
+    <joint name="hand_mount_to_base" type="fixed">
+      <origin xyz="0 0 0" rpy="0 0 1.5708"/>
+      <parent link="hand_mount"/>
+      <child link="hand_base"/>
+    </joint>
     <!-- Base link of the hand -->
     <link name="hand_base">
@@ -40,4 +55,11 @@
       <child link="thumb_distal_tactile"/>
     </joint>
+    <!-- thumb_fingertip: fingertip frame at the end of thumb -->
+    <link name="thumb_fingertip" />
+    <joint name="thumb_distal_to_fingertip" type="fixed">
+      <origin xyz="-0.066 0 0" rpy="0 0 0"/>
+      <parent link="thumb_distal"/>
+      <child link="thumb_fingertip"/>
+    </joint>
     <!-- thumb_metacarpal -->
     <link name="thumb_metacarpal">
@@ -231,4 +253,11 @@
       <child link="index_distal_tactile"/>
     </joint>
+    <!-- index_fingertip: fingertip frame at the end of index finger -->
+    <link name="index_fingertip" />
+    <joint name="index_distal_to_fingertip" type="fixed">
+      <origin xyz="-0.066 0 0" rpy="0 0 0"/>
+      <parent link="index_distal"/>
+      <child link="index_fingertip"/>
+    </joint>
       <!-- Middle joints -->
     <joint name="joint7" type="revolute">
@@ -301,9 +330,10 @@
       <child link="middle_distal_tactile"/>
     </joint>
-    <!-- Attach hand_base to the provided connector link -->
-    <joint name="hand_mount" type="fixed">
-      <origin xyz="${xyz}" rpy="${rpy}"/>
-      <parent link="${connector_link}"/>
-      <child link="hand_base"/>
+    <!-- middle_fingertip: fingertip frame at the end of middle finger -->
+    <link name="middle_fingertip" />
+    <joint name="middle_distal_to_fingertip" type="fixed">
+      <origin xyz="-0.066 0 0" rpy="0 0 0"/>
+      <parent link="middle_distal"/>
+      <child link="middle_fingertip"/>
     </joint>
   </xacro:macro>
